File: hardware/MSD-1.0/_autosave-MSD-1.0.kicad_sch (KiCad schematic)
At the start: 19 parts, among them J1 Conn_01x05, J2 Conn_01x03, Q1 IRF840N, U1 NE555P, U2 PC817, U3 PC817

Commit message: modified:   hardware/MSD-1.0/_autosave-MSD-1.0.kicad_sch 	modified:   log.md
Parts:
- D2, D3: value D -> HER208
- L1: value L_Coupled -> Isolation Transformer (Custom)
- Q1: value IRF840N -> IRF840
- R4: value R -> 330Ω
Changed lines of the file:
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@@
 			)
 		)
-		(property "Value" "IRF840N"
+		(property "Value" "IRF840"
 			(at 124.46 55.88 0)
 			(effects
@@
 			)
 		)
-		(property "Value" "D"
+		(property "Value" "HER208"
 			(at 177.8 34.036 0)
 			(effects
@@
 					(size 1 1)
 				)
-				(hide yes)
 			)
 		)
@@
 				)
 				(justify left)
-				(hide yes)
 			)
 		)
@@
 			)
 		)
-		(property "Value" "D"
+		(property "Value" "HER208"
 			(at 177.8 99.314 0)
 			(effects
@@
 					(size 1 1)
 				)
-				(hide yes)
 			)
 		)
@@
 				)
 				(justify left)
-				(hide yes)
 			)
 		)
@@
 					(size 1 1)
 				)
-				(hide yes)
 			)
 		)
@@
 			)
 		)
-		(property "Value" "L_Coupled"
+		(property "Value" "Isolation Transformer (Custom)"
 			(at 137.414 44.958 90)
 			(effects
@@
 			)
 		)
-		(property "Value" "R"
+		(property "Value" "330Ω"
 			(at 165.1 103.886 90)
 			(effects
@@
 					(size 1 1)
 				)
-				(hide yes)
-			)
-		)
+			)
+		)
