File: hardware/MSD-1.0/MSD-1.0.kicad_sch (KiCad schematic)
At the start: 27 parts, among them J1 Conn_01x05, J2 Conn_01x03, Q1 IRF840, U1 NE555P, U2 PC817, U3 PC817

Commit message: modified:   .DS_Store 	modified:   README.md 	modified:   hardware/MSD-1.0/MSD-1.0-B_Cu.gbr 	modified:   hardware/MSD-1.0/MSD-1.0-B_Mask.gbr 	modified:   hardware/MSD-1.0/MSD-1.0-B_Paste.gbr 	modified:   hardware/MSD-1.0/MSD-1.0-B_Silkscreen.gbr 	modified:   hardware/MSD-1.0/MSD-1.0-Edge_Cuts.gbr 	modified:   hardware/MSD-1.0/MSD-1.0-F_Cu.gbr 	modified:   hardware/MSD-1.0/MSD-1.0-F_Mask.gbr 	modified:   hardware/MSD-1.0/MSD-1.0-F_Paste.gbr 	modified:   hardware/MSD-1.0/MSD-1.0-F_Silkscreen.gbr 	modified:   hardware/MSD-1.0/MSD-1.0-NPTH.drl 	modified:   hardware/MSD-1.0/MSD-1.0-PTH.drl 	deleted:    hardware/MSD-1.0/MSD-1.0-backups/MSD-1.0-2025-04-09_135836.zip 	deleted:    hardware/MSD-1.0/MSD-1.0-backups/MSD-1.0-2025-04-09_140350.zip 	new file:   hardware/MSD-1.0/MSD-1.0-backups/MSD-1.0-2025-05-08_171110.zip 	new file:   hardware/MSD-1.0/MSD-1.0-backups/MSD-1.0-2025-05-09_084805.zip 	modified:   hardware/MSD-1.0/MSD-1.0-job.gbrjob 	modified:   hardware/MSD-1.0/MSD-1.0.kicad_sch 	modified:   hardware/MSD-1.0/MSD-1.zip 	deleted:    hardware/MSD-1.0/~MSD-1.0.kicad_sch.lck 	modified:   hardware/PS-2.0/PS-2.0-B_Cu.gbr 	modified:   hardware/PS-2.0/PS-2.0-B_Mask.gbr 	modified:   hardware/PS-2.0/PS-2.0-B_Paste.gbr 	modified:   hardware/PS-2.0/PS-2.0-B_Silkscreen.gbr 	modified:   hardware/PS-2.0/PS-2.0-Edge_Cuts.gbr 	modified:   hardware/PS-2.0/PS-2.0-F_Cu.gbr 	modified:   hardware/PS-2.0/PS-2.0-F_Mask.gbr 	modified:   hardware/PS-2.0/PS-2.0-F_Paste.gbr 	modified:   hardware/PS-2.0/PS-2.0-F_Silkscreen.gbr 	modified:   hardware/PS-2.0/PS-2.0-NPTH.drl 	modified:   hardware/PS-2.0/PS-2.0-PTH.drl 	new file:   hardware/PS-2.0/PS-2.0-backups/PS-2.0-2025-05-09_084820.zip 	new file:   hardware/PS-2.0/PS-2.0-backups/PS-2.0-2025-05-09_090220.zip 	modified:   hardware/PS-2.0/PS-2.0-job.gbrjob 	modified:   hardware/PS-2.0/PS-2.0.kicad_pcb 	modified:   hardware/PS-2.0/PS-2.zip
Connections:
- net +12V renamed +5V
Other:
- moved on the sheet: J1, TP7
Changed lines of the file:
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@@
 	)
 	(junction
-		(at 57.15 57.15)
+		(at 54.61 57.15)
 		(diameter 0)
 		(color 0 0 0 0)
 	)
 	(junction
-		(at 52.07 38.1)
+		(at 49.53 38.1)
 		(diameter 0)
 		(color 0 0 0 0)
@@
 	(wire
 		(pts
-			(xy 52.07 91.44) (xy 52.07 59.69)
+			(xy 49.53 91.44) (xy 49.53 59.69)
 		)
 		(stroke
@@
 	(wire
 		(pts
-			(xy 46.99 102.87) (xy 46.99 62.23)
+			(xy 44.45 102.87) (xy 44.45 62.23)
 		)
 		(stroke
@@
 	(wire
 		(pts
-			(xy 52.07 35.56) (xy 52.07 38.1)
-		)
-		(stroke
-			(width 0)
-			(type default)
-		)
-	)
-	(wire
-		(pts
-			(xy 52.07 38.1) (xy 64.77 38.1)
+			(xy 49.53 35.56) (xy 49.53 38.1)
+		)
+		(stroke
+			(width 0)
+			(type default)
+		)
+	)
+	(wire
+		(pts
+			(xy 49.53 38.1) (xy 64.77 38.1)
 		)
 		(stroke
@@
 	(wire
 		(pts
-			(xy 166.37 91.44) (xy 52.07 91.44)
+			(xy 166.37 91.44) (xy 49.53 91.44)
 		)
 		(stroke
@@
 	(wire
 		(pts
-			(xy 46.99 62.23) (xy 41.91 62.23)
+			(xy 44.45 62.23) (xy 39.37 62.23)
 		)
 		(stroke
@@
 	(wire
 		(pts
-			(xy 57.15 57.15) (xy 57.15 83.82)
+			(xy 54.61 57.15) (xy 54.61 83.82)
 		)
 		(stroke
@@
 	(wire
 		(pts
-			(xy 41.91 57.15) (xy 57.15 57.15)
-		)
-		(stroke
-			(width 0)
-			(type default)
-		)
-	)
-	(wire
-		(pts
-			(xy 41.91 54.61) (xy 52.07 54.61)
+			(xy 39.37 57.15) (xy 54.61 57.15)
+		)
+		(stroke
+			(width 0)
+			(type default)
+		)
+	)
+	(wire
+		(pts
+			(xy 39.37 54.61) (xy 49.53 54.61)
 		)
 		(stroke
@@
 	(wire
 		(pts
-			(xy 166.37 102.87) (xy 46.99 102.87)
+			(xy 166.37 102.87) (xy 44.45 102.87)
 		)
 		(stroke
@@
 	(wire
 		(pts
-			(xy 57.15 83.82) (xy 64.77 83.82)
+			(xy 54.61 83.82) (xy 64.77 83.82)
 		)
 		(stroke
@@
 	(wire
 		(pts
-			(xy 52.07 38.1) (xy 52.07 54.61)
-		)
-		(stroke
-			(width 0)
-			(type default)
-		)
-	)
-	(wire
-		(pts
-			(xy 41.91 59.69) (xy 52.07 59.69)
+			(xy 49.53 38.1) (xy 49.53 54.61)
+		)
+		(stroke
+			(width 0)
+			(type default)
+		)
+	)
+	(wire
+		(pts
+			(xy 39.37 59.69) (xy 49.53 59.69)
 		)
 		(stroke
@@
 	(wire
 		(pts
-			(xy 57.15 35.56) (xy 57.15 57.15)
+			(xy 54.61 35.56) (xy 54.61 57.15)
 		)
 		(stroke
@@
 			(effects
 				(font
-					(size 1.27 1.27)
+					(size 1 1)
 				)
 				(justify left)
@@
 	(symbol
 		(lib_id "Connector:TestPoint")
-		(at 57.15 35.56 0)
+		(at 54.61 35.56 0)
 		(unit 1)
 		(exclude_from_sim no)
@@
 		(dnp no)
 		(property "Reference" "TP7"
-			(at 55.626 32.004 0)
+			(at 53.086 31.75 0)
 			(effects
 				(font
@@
 		)
 		(property "Value" "TestPoint"
-			(at 59.69 34.7979 0)
+			(at 57.15 34.7979 0)
 			(effects
 				(font
@@
 		)
 		(property "Footprint" "TestPoint:TestPoint_Bridge_Pitch2.54mm_Drill1.0mm"
-			(at 62.23 35.56 0)
+			(at 59.69 35.56 0)
 			(effects
 				(font
@@
 		)
 		(property "Datasheet" "~"
-			(at 62.23 35.56 0)
+			(at 59.69 35.56 0)
 			(effects
 				(font
@@
 		)
 		(property "Description" "test point"
-			(at 57.15 35.56 0)
+			(at 54.61 35.56 0)
 			(effects
 				(font
@@
 		)
 		(property "Value" "470µF 35V"
-			(at 65.024 71.882 0)
-			(effects
-				(font
-					(size 1 1)
-				)
-				(justify left)
-				(hide yes)
+			(at 61.214 69.85 90)
+			(effects
+				(font
+					(size 1 1)
+				)
 			)
 		)
@@
 			(effects
 				(font
-					(size 1.27 1.27)
+					(size 1 1)
 				)
 				(justify left)
@@
 		)
 		(property "Value" "2.2nF 100"
-			(at 85.598 71.882 0)
-			(effects
-				(font
-					(size 1 1)
-				)
-				(justify left)
+			(at 81.788 69.85 90)
+			(effects
+				(font
+					(size 1 1)
+				)
 			)
 		)
@@
 	(symbol
 		(lib_id "Connector_Generic:Conn_01x04")
-		(at 36.83 59.69 180)
+		(at 34.29 59.69 180)
 		(unit 1)
 		(exclude_from_sim no)
@@
 		(dnp no)
 		(property "Reference" "J1"
-			(at 36.83 52.07 0)
+			(at 34.29 52.07 0)
 			(effects
 				(font
@@
 		)
 		(property "Value" "Conn_01x05"
-			(at 36.83 50.8 0)
+			(at 34.29 50.8 0)
 			(effects
 				(font
@@
 		)
 		(property "Footprint" "Connector_PinHeader_2.54mm:PinHeader_1x04_P2.54mm_Horizontal_2"
-			(at 36.83 59.69 0)
+			(at 34.29 59.69 0)
 			(effects
 				(font
@@
 		)
 		(property "Datasheet" "~"
-			(at 36.83 59.69 0)
+			(at 34.29 59.69 0)
 			(effects
 				(font
@@
 		)
 		(property "Description" "Generic connector, single row, 01x04, script generated (kicad-library-utils/schlib/autogen/connector/)"
-			(at 36.83 59.69 0)
+			(at 34.29 59.69 0)
 			(effects
 				(font
@@
 		)
 		(property "Value" "100nF 100"
-			(at 75.438 71.882 0)
-			(effects
-				(font
-					(size 1 1)
-				)
-				(justify left)
+			(at 71.628 69.85 90)
+			(effects
+				(font
+					(size 1 1)
+				)
 			)
 		)
@@
 	(symbol
 		(lib_id "power:+12V")
-		(at 52.07 35.56 0)
+		(at 49.53 35.56 0)
 		(unit 1)
 		(exclude_from_sim no)
@@
 		(on_board yes)
 		(dnp no)
-		(fields_autoplaced yes)
 		(property "Reference" "#PWR01"
-			(at 52.07 39.37 0)
-			(effects
-				(font
-					(size 1.27 1.27)
-				)
-				(hide yes)
-			)
-		)
-		(property "Value" "+12V"
-			(at 52.07 30.48 0)
-			(effects
-				(font
-					(size 1.27 1.27)
-				)
+			(at 49.53 39.37 0)
+			(effects
+				(font
+					(size 1.27 1.27)
+				)
+				(hide yes)
+			)
+		)
+		(property "Value" "+5V"
+			(at 47.498 31.75 0)
+			(effects
+				(font
+					(size 1 1)
+				)
+				(justify left)
 			)
 		)
 		(property "Footprint" ""
-			(at 52.07 35.56 0)
+			(at 49.53 35.56 0)
 			(effects
 				(font
@@
 		)
 		(property "Datasheet" ""
-			(at 52.07 35.56 0)
+			(at 49.53 35.56 0)
 			(effects
 				(font
@@
 		)
 		(property "Description" "Power symbol creates a global label with name \"+12V\""
-			(at 52.07 35.56 0)
+			(at 49.53 35.56 0)
 			(effects
 				(font
@@
 		)
 		(property "Value" "10nF 63"
-			(at 95.758 71.882 0)
-			(effects
-				(font
-					(size 1 1)
-				)
-				(justify left)
-			)
-		)
+			(at 91.948 69.85 90)
+			(effects
+				(font
+					(size 1 1)
+				)
+			)
+		)
