File: hardware/REM-1.0/REM-1.0.kicad_sch (KiCad schematic)
At the start: 27 parts, among them J1 Conn_01x03, J2 Conn_01x03, Q1 BC327

Commit message: deleted:    hardware/MSD-1.0/#auto_saved_files# 	new file:   hardware/MSD-1.0/MSD-1.0 BoM.csv 	new file:   hardware/MSD-1.0/MSD-1.0-B_Cu.gbr 	new file:   hardware/MSD-1.0/MSD-1.0-B_Mask.gbr 	new file:   hardware/MSD-1.0/MSD-1.0-B_Paste.gbr 	new file:   hardware/MSD-1.0/MSD-1.0-B_Silkscreen.gbr 	new file:   hardware/MSD-1.0/MSD-1.0-Edge_Cuts.gbr 	new file:   hardware/MSD-1.0/MSD-1.0-F_Cu.gbr 	new file:   hardware/MSD-1.0/MSD-1.0-F_Mask.gbr 	new file:   hardware/MSD-1.0/MSD-1.0-F_Paste.gbr 	new file:   hardware/MSD-1.0/MSD-1.0-F_Silkscreen.gbr 	new file:   hardware/MSD-1.0/MSD-1.0-NPTH.drl 	new file:   hardware/MSD-1.0/MSD-1.0-PTH.drl 	deleted:    hardware/MSD-1.0/MSD-1.0-backups/MSD-1.0-2025-02-24_160102.zip 	deleted:    hardware/MSD-1.0/MSD-1.0-backups/MSD-1.0-2025-02-24_160721.zip 	deleted:    hardware/MSD-1.0/MSD-1.0-backups/MSD-1.0-2025-02-24_161316.zip 	deleted:    hardware/MSD-1.0/MSD-1.0-backups/MSD-1.0-2025-02-24_162407.zip 	deleted:    hardware/MSD-1.0/MSD-1.0-backups/MSD-1.0-2025-02-24_163137.zip 	deleted:    hardware/MSD-1.0/MSD-1.0-backups/MSD-1.0-2025-02-25_161045.zip 	deleted:    hardware/MSD-1.0/MSD-1.0-backups/MSD-1.0-2025-02-26_093224.zip 	deleted:    hardware/MSD-1.0/MSD-1.0-backups/MSD-1.0-2025-02-26_094218.zip 	new file:   hardware/MSD-1.0/MSD-1.0-backups/MSD-1.0-2025-02-26_163854.zip 	new file:   hardware/MSD-1.0/MSD-1.0-backups/MSD-1.0-2025-02-27_112851.zip 	new file:   hardware/MSD-1.0/MSD-1.0-backups/MSD-1.0-2025-02-27_114053.zip 	new file:   hardware/MSD-1.0/MSD-1.0-backups/MSD-1.0-2025-02-27_185834.zip 	new file:   hardware/MSD-1.0/MSD-1.0-backups/MSD-1.0-2025-02-27_190654.zip 	new file:   hardware/MSD-1.0/MSD-1.0-backups/MSD-1.0-2025-02-27_191228.zip 	new file:   hardware/MSD-1.0/MSD-1.0-backups/MSD-1.0-2025-02-28_140545.zip 	new file:   hardware/MSD-1.0/MSD-1.0-backups/MSD-1.0-2025-02-28_141533.zip 	new file:   hardware/MSD-1.0/MSD-1.0-backups/MSD-1.0-2025-02-28_142536.zip 	new file:   hardware/MSD-1.0/MSD-1.0-backups/MSD-1.0-2025-02-28_14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
Parts:
- L1: value L_Ferrite_Coupled -> Isolated Transformer (Custom)
- Q1: value BC327 -> 2N2222
- R5, R6: value R -> 33Ω
Changed lines of the file:
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@@
 			)
 		)
-		(property "Value" "BC327"
+		(property "Value" "2N2222"
 			(at 136.906 67.31 0)
 			(effects
@@
 			)
 		)
-		(property "Value" "R"
+		(property "Value" "33Ω"
 			(at 184.15 40.386 90)
 			(effects
@@
 			)
 		)
-		(property "Value" "R"
+		(property "Value" "33Ω"
 			(at 184.15 55.626 90)
 			(effects
@@
 			)
 		)
-		(property "Value" "L_Ferrite_Coupled"
+		(property "Value" "Isolated Transformer (Custom)"
 			(at 171.45 47.244 90)
 			(effects
