File: hardware/REM-2.0/REM-2.0.kicad_pcb (KiCad board)
At the start: 2 copper layers, 98.4 x 44.5 mm, 39 parts, among them J1 Conn_01x03, J2 Conn_01x03, Q1 IRF840, U1 NE555P, U2 NE5534

Commit message: modified:   .DS_Store 	deleted:    hardware/MSD-1.0/MSD-1.0-backups/MSD-1.0-2025-02-25_161819.zip 	deleted:    hardware/MSD-1.0/MSD-1.0-backups/MSD-1.0-2025-02-25_162448.zip 	deleted:    hardware/MSD-1.0/MSD-1.0-backups/MSD-1.0-2025-02-25_163016.zip 	deleted:    hardware/MSD-1.0/MSD-1.0-backups/MSD-1.0-2025-02-25_163954.zip 	deleted:    hardware/MSD-1.0/MSD-1.0-backups/MSD-1.0-2025-02-26_112856.zip 	deleted:    hardware/MSD-1.0/MSD-1.0-backups/MSD-1.0-2025-02-26_113923.zip 	deleted:    hardware/MSD-1.0/MSD-1.0-backups/MSD-1.0-2025-02-26_115654.zip 	deleted:    hardware/MSD-1.0/MSD-1.0-backups/MSD-1.0-2025-02-26_120757.zip 	deleted:    hardware/MSD-1.0/MSD-1.0-backups/MSD-1.0-2025-02-26_163854.zip 	deleted:    hardware/MSD-1.0/MSD-1.0-backups/MSD-1.0-2025-02-27_112851.zip 	deleted:    hardware/MSD-1.0/MSD-1.0-backups/MSD-1.0-2025-02-27_114053.zip 	deleted:    hardware/MSD-1.0/MSD-1.0-backups/MSD-1.0-2025-02-27_185834.zip 	deleted:    hardware/MSD-1.0/MSD-1.0-backups/MSD-1.0-2025-02-27_190654.zip 	deleted:    hardware/MSD-1.0/MSD-1.0-backups/MSD-1.0-2025-02-27_191228.zip 	deleted:    hardware/MSD-1.0/MSD-1.0-backups/MSD-1.0-2025-02-28_140545.zip 	deleted:    hardware/MSD-1.0/MSD-1.0-backups/MSD-1.0-2025-02-28_141533.zip 	deleted:    hardware/MSD-1.0/MSD-1.0-backups/MSD-1.0-2025-02-28_142536.zip 	deleted:    hardware/MSD-1.0/MSD-1.0-backups/MSD-1.0-2025-02-28_143342.zip 	deleted:    hardware/MSD-1.0/MSD-1.0-backups/MSD-1.0-2025-02-28_162722.zip 	deleted:    hardware/MSD-1.0/MSD-1.0-backups/MSD-1.0-2025-03-05_134102.zip 	deleted:    hardware/MSD-1.0/MSD-1.0-backups/MSD-1.0-2025-03-05_134620.zip 	new file:   hardware/MSD-1.0/MSD-1.0-backups/MSD-1.0-2025-03-24_113503.zip 	new file:   hardware/MSD-1.0/MSD-1.0-backups/MSD-1.0-2025-03-24_114029.zip 	new file:   hardware/MSD-1.0/MSD-1.0-backups/MSD-1.0-2025-03-24_132745.zip 	new file:   hardware/MSD-1.0/MSD-1.0-backups/MSD-1.0-2025-03-24_134332.zip 	new file:   hardware/MSD-1.0/MSD-1.0-backups/MSD-1.0-2025-03-25_144744.zip 	n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
Parts:
- D1: footprint Diode_THT:D_DO-34_SOD68_P7.62mm_Horizontal -> Diode_THT:D_DO-35_SOD27_P7.62mm_Horizontal
- J1: value Conn_01x03 -> Conn_01x04; footprint Connector_PinHeader_2.54mm:PinHeader_1x04_P2.54mm_Horizontal_Custom -> Connector_PinHeader_2.54mm:PinHeader_1x04_P2.54mm_Horizontal_2
- J2: footprint Connector_PinHeader_2.54mm:PinHeader_1x03_P5.08mm_Horizontal_Custom -> Connector_PinHeader_2.54mm:PinHeader_1x03_P5.08mm_Horizontal_2
- R4: value R -> 10k
- TP1, TP2, TP5, TP6, TP7: footprint TestPoint:TestPoint_Bridge_Pitch2.54mm_Drill0.7mm -> TestPoint:TestPoint_Bridge_Pitch2.54mm_Drill1.0mm
- moved J2 3.18 mm to (180.0, 101.3)
- moved J1 2.54 mm to (106.0, 101.3)
- moved TP7 0.64 mm to (98.4, 69.2)
Routing:
- net +5V: track 145.5 -> 154.3 mm
- net Net-(J2-Pin_1): track 12.9 -> 10.3 mm
- net Net-(J1-Pin_1): track 121.8 -> 123.7 mm
- net +12V: track 159.8 -> 161.1 mm
- net Net-(J2-Pin_3): track 28.3 -> 28.9 mm
- net Net-(J2-Pin_2): track 27.8 -> 28.5 mm
