File: hardware/REM-2.0/REM-2.0.kicad_sch (KiCad schematic)
At the start: 39 parts, among them J1 Conn_01x03, J2 Conn_01x03, Q1 IRF840, U1 NE555P, U2 NE5534

Commit message: modified:   .DS_Store 	deleted:    hardware/MSD-1.0/MSD-1.0-backups/MSD-1.0-2025-02-25_161819.zip 	deleted:    hardware/MSD-1.0/MSD-1.0-backups/MSD-1.0-2025-02-25_162448.zip 	deleted:    hardware/MSD-1.0/MSD-1.0-backups/MSD-1.0-2025-02-25_163016.zip 	deleted:    hardware/MSD-1.0/MSD-1.0-backups/MSD-1.0-2025-02-25_163954.zip 	deleted:    hardware/MSD-1.0/MSD-1.0-backups/MSD-1.0-2025-02-26_112856.zip 	deleted:    hardware/MSD-1.0/MSD-1.0-backups/MSD-1.0-2025-02-26_113923.zip 	deleted:    hardware/MSD-1.0/MSD-1.0-backups/MSD-1.0-2025-02-26_115654.zip 	deleted:    hardware/MSD-1.0/MSD-1.0-backups/MSD-1.0-2025-02-26_120757.zip 	deleted:    hardware/MSD-1.0/MSD-1.0-backups/MSD-1.0-2025-02-26_163854.zip 	deleted:    hardware/MSD-1.0/MSD-1.0-backups/MSD-1.0-2025-02-27_112851.zip 	deleted:    hardware/MSD-1.0/MSD-1.0-backups/MSD-1.0-2025-02-27_114053.zip 	deleted:    hardware/MSD-1.0/MSD-1.0-backups/MSD-1.0-2025-02-27_185834.zip 	deleted:    hardware/MSD-1.0/MSD-1.0-backups/MSD-1.0-2025-02-27_190654.zip 	deleted:    hardware/MSD-1.0/MSD-1.0-backups/MSD-1.0-2025-02-27_191228.zip 	deleted:    hardware/MSD-1.0/MSD-1.0-backups/MSD-1.0-2025-02-28_140545.zip 	deleted:    hardware/MSD-1.0/MSD-1.0-backups/MSD-1.0-2025-02-28_141533.zip 	deleted:    hardware/MSD-1.0/MSD-1.0-backups/MSD-1.0-2025-02-28_142536.zip 	deleted:    hardware/MSD-1.0/MSD-1.0-backups/MSD-1.0-2025-02-28_143342.zip 	deleted:    hardware/MSD-1.0/MSD-1.0-backups/MSD-1.0-2025-02-28_162722.zip 	deleted:    hardware/MSD-1.0/MSD-1.0-backups/MSD-1.0-2025-03-05_134102.zip 	deleted:    hardware/MSD-1.0/MSD-1.0-backups/MSD-1.0-2025-03-05_134620.zip 	new file:   hardware/MSD-1.0/MSD-1.0-backups/MSD-1.0-2025-03-24_113503.zip 	new file:   hardware/MSD-1.0/MSD-1.0-backups/MSD-1.0-2025-03-24_114029.zip 	new file:   hardware/MSD-1.0/MSD-1.0-backups/MSD-1.0-2025-03-24_132745.zip 	new file:   hardware/MSD-1.0/MSD-1.0-backups/MSD-1.0-2025-03-24_134332.zip 	new file:   hardware/MSD-1.0/MSD-1.0-backups/MSD-1.0-2025-03-25_144744.zip 	n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
Parts:
- added R10: 10kΩ, Resistor_THT:R_Axial_DIN0204_L3.6mm_D1.6mm_P7.62mm_Horizontal, symbol Device:R
- added R11: 10k, Resistor_THT:R_Axial_DIN0204_L3.6mm_D1.6mm_P7.62mm_Horizontal, symbol Device:R
- D1: footprint Diode_THT:D_DO-34_SOD68_P7.62mm_Horizontal -> Diode_THT:D_DO-35_SOD27_P7.62mm_Horizontal
- J1: value Conn_01x03 -> Conn_01x04; footprint Connector_PinHeader_2.54mm:PinHeader_1x04_P2.54mm_Horizontal_Custom -> Connector_PinHeader_2.54mm:PinHeader_1x04_P2.54mm_Horizontal_2
- J2: footprint Connector_PinHeader_2.54mm:PinHeader_1x03_P5.08mm_Horizontal_Custom -> Connector_PinHeader_2.54mm:PinHeader_1x03_P5.08mm_Horizontal_2
- R4: value R -> 10k
- TP1, TP2, TP5, TP6, TP7: footprint TestPoint:TestPoint_Bridge_Pitch2.54mm_Drill0.7mm -> TestPoint:TestPoint_Bridge_Pitch2.54mm_Drill1.0mm
Connections:
- net +12V: no longer RV2.3
- net GND: now also R6.1; no longer RV2.1
- net at RV2.2: no longer R6.1
Other:
- moved on the sheet: C10, C9, JP1, JP2, R6, R7, TP6, TP7, U2
