File: hardware/REM-3.0/REM-3.0.kicad_sch (KiCad schematic)
At the start: 56 parts, among them J1 Conn_01x04, J2 Conn_01x03, Q1 IRF840, U1 NE555P, U2 LM358

Commit message: deleted:    hardware/Gain/Gain-backups/Gain-2025-04-14_115147.zip 	new file:   hardware/Gain/Gain-backups/Gain-2025-04-15_120154.zip 	deleted:    hardware/MSD-1.0/MSD-1.0-backups/MSD-1.0-2025-03-24_134332.zip 	deleted:    hardware/MSD-1.0/MSD-1.0-backups/MSD-1.0-2025-03-25_144744.zip 	deleted:    hardware/MSD-1.0/MSD-1.0-backups/MSD-1.0-2025-03-25_145433.zip 	deleted:    hardware/MSD-1.0/MSD-1.0-backups/MSD-1.0-2025-03-25_150210.zip 	deleted:    hardware/MSD-1.0/MSD-1.0-backups/MSD-1.0-2025-03-25_150818.zip 	new file:   hardware/MSD-1.0/MSD-1.0-backups/MSD-1.0-2025-04-16_142822.zip 	new file:   hardware/MSD-1.0/MSD-1.0-backups/MSD-1.0-2025-04-16_143722.zip 	new file:   hardware/MSD-1.0/MSD-1.0-backups/MSD-1.0-2025-04-16_145208.zip 	new file:   hardware/MSD-1.0/MSD-1.0-backups/MSD-1.0-2025-04-16_150237.zip 	new file:   hardware/MSD-1.0/MSD-1.0-backups/MSD-1.0-2025-04-16_150829.zip 	modified:   hardware/MSD-1.0/MSD-1.0.kicad_pcb 	modified:   hardware/MSD-1.0/MSD-1.0.kicad_sch 	modified:   hardware/MSD-1.0/MSD-1.0.step 	new file:   hardware/MSD-2.0/MSD-2.0-backups/MSD-2.0-2025-04-16_090248.zip 	deleted:    hardware/PS-1.0/PS-1.0-backups/PS-1.0-2025-03-18_205016.zip 	deleted:    hardware/PS-1.0/PS-1.0-backups/PS-1.0-2025-03-18_205728.zip 	deleted:    hardware/PS-1.0/PS-1.0-backups/PS-1.0-2025-03-18_211157.zip 	deleted:    hardware/PS-1.0/PS-1.0-backups/PS-1.0-2025-03-18_213933.zip 	deleted:    hardware/PS-1.0/PS-1.0-backups/PS-1.0-2025-03-19_094557.zip 	deleted:    hardware/PS-1.0/PS-1.0-backups/PS-1.0-2025-03-19_101204.zip 	deleted:    hardware/PS-1.0/PS-1.0-backups/PS-1.0-2025-03-19_102323.zip 	new file:   hardware/PS-1.0/PS-1.0-backups/PS-1.0-2025-04-16_154157.zip 	new file:   hardware/PS-1.0/PS-1.0-backups/PS-1.0-2025-04-16_154838.zip 	new file:   hardware/PS-1.0/PS-1.0-backups/PS-1.0-2025-04-16_155906.zip 	new file:   hardware/PS-1.0/PS-1.0-backups/PS-1.0-2025-04-16_160456.zip 	new file:   hardware/PS-1.0/PS-1.0-backups/PS-1.0-2025-04-16_161300.zip 	new file:   har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
Parts:
- removed C9: 470uF 50V, Capacitor_THT:CP_Radial_D12.5mm_P5.00mm, symbol Device:C_Polarized
- removed JP10, JP5, JP6, JP9: TestPoint, TestPoint:TestPoint_THTPad_D1.5mm_Drill0.7mm, symbol Connector:TestPoint
Connections:
- net +12V is gone; now on net +5V: C3.1, C7.1, C8.1, J1.4 (Pin_4), JP1.1, JP2.1, JP7.1, JP8.1, L1.2, R1.1, TP1.1, U1.4 (R), U1.8 (VCC)
- net +5V: no longer J1.2 (Pin_2)
