File: hardware/REM-3.0/REM-3.0.kicad_pcb (KiCad board)
At the start: 2 copper layers, 98.4 x 50.8 mm, 56 parts, among them J1 Conn_01x04, J2 Conn_01x03, Q1 IRF840, U1 NE555P, U2 LM358

Commit message: deleted:    hardware/Gain/Gain-backups/Gain-2025-04-14_115147.zip 	new file:   hardware/Gain/Gain-backups/Gain-2025-04-15_120154.zip 	deleted:    hardware/MSD-1.0/MSD-1.0-backups/MSD-1.0-2025-03-24_134332.zip 	deleted:    hardware/MSD-1.0/MSD-1.0-backups/MSD-1.0-2025-03-25_144744.zip 	deleted:    hardware/MSD-1.0/MSD-1.0-backups/MSD-1.0-2025-03-25_145433.zip 	deleted:    hardware/MSD-1.0/MSD-1.0-backups/MSD-1.0-2025-03-25_150210.zip 	deleted:    hardware/MSD-1.0/MSD-1.0-backups/MSD-1.0-2025-03-25_150818.zip 	new file:   hardware/MSD-1.0/MSD-1.0-backups/MSD-1.0-2025-04-16_142822.zip 	new file:   hardware/MSD-1.0/MSD-1.0-backups/MSD-1.0-2025-04-16_143722.zip 	new file:   hardware/MSD-1.0/MSD-1.0-backups/MSD-1.0-2025-04-16_145208.zip 	new file:   hardware/MSD-1.0/MSD-1.0-backups/MSD-1.0-2025-04-16_150237.zip 	new file:   hardware/MSD-1.0/MSD-1.0-backups/MSD-1.0-2025-04-16_150829.zip 	modified:   hardware/MSD-1.0/MSD-1.0.kicad_pcb 	modified:   hardware/MSD-1.0/MSD-1.0.kicad_sch 	modified:   hardware/MSD-1.0/MSD-1.0.step 	new file:   hardware/MSD-2.0/MSD-2.0-backups/MSD-2.0-2025-04-16_090248.zip 	deleted:    hardware/PS-1.0/PS-1.0-backups/PS-1.0-2025-03-18_205016.zip 	deleted:    hardware/PS-1.0/PS-1.0-backups/PS-1.0-2025-03-18_205728.zip 	deleted:    hardware/PS-1.0/PS-1.0-backups/PS-1.0-2025-03-18_211157.zip 	deleted:    hardware/PS-1.0/PS-1.0-backups/PS-1.0-2025-03-18_213933.zip 	deleted:    hardware/PS-1.0/PS-1.0-backups/PS-1.0-2025-03-19_094557.zip 	deleted:    hardware/PS-1.0/PS-1.0-backups/PS-1.0-2025-03-19_101204.zip 	deleted:    hardware/PS-1.0/PS-1.0-backups/PS-1.0-2025-03-19_102323.zip 	new file:   hardware/PS-1.0/PS-1.0-backups/PS-1.0-2025-04-16_154157.zip 	new file:   hardware/PS-1.0/PS-1.0-backups/PS-1.0-2025-04-16_154838.zip 	new file:   hardware/PS-1.0/PS-1.0-backups/PS-1.0-2025-04-16_155906.zip 	new file:   hardware/PS-1.0/PS-1.0-backups/PS-1.0-2025-04-16_160456.zip 	new file:   hardware/PS-1.0/PS-1.0-backups/PS-1.0-2025-04-16_161300.zip 	new file:   har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
Parts:
- removed C9: 470uF 50V, Capacitor_THT:CP_Radial_D12.5mm_P5.00mm
- removed JP10, JP5, JP6, JP9: TestPoint, TestPoint:TestPoint_THTPad_D1.5mm_Drill0.7mm
- moved C7 13.3 mm to (116.2, 101.6)
Connections:
- C3 pad 1: +12V -> +5V
- C7 pad 1: +12V -> +5V
- C8 pad 1: +12V -> +5V
- J1 pad 2: +5V -> unconnected-(J1-Pin_2-Pad2)
- J1 pad 4: +12V -> +5V
- JP1 pad 1: +12V -> +5V
- JP2 pad 1: +12V -> +5V
- JP7 pad 1: +12V -> +5V
- JP8 pad 1: +12V -> +5V
- L1 pad 2: +12V -> +5V
- R1 pad 1: +12V -> +5V
- TP1 pad 1: +12V -> +5V
- U1 pad 4: +12V -> +5V
- U1 pad 8: +12V -> +5V
Routing:
- net +12V: track 126.1 -> 0.00 mm
- net +5V: track 157.7 -> 210.7 mm
- net GND: track 7.62 -> 0.00 mm
