File: hardware/REM-4.0/REM-4.0.kicad_sch (KiCad schematic)
At the start: 35 parts, among them J1 Conn_01x04, J2 Conn_01x03, Q1 IRF840, U1 NE555P

Commit message: new file:   .~BoM.xlsx 	new file:   BoM.xlsx 	new file:   hardware/BoM.xlsx 	deleted:    hardware/MSD-1.0/MSD-1.0-backups/MSD-1.0-2025-03-26_092035.zip 	deleted:    hardware/MSD-1.0/MSD-1.0-backups/MSD-1.0-2025-03-26_092834.zip 	deleted:    hardware/MSD-1.0/MSD-1.0-backups/MSD-1.0-2025-03-27_092014.zip 	new file:   hardware/MSD-1.0/MSD-1.0-backups/MSD-1.0-2025-04-28_130614.zip 	new file:   hardware/MSD-1.0/MSD-1.0-backups/MSD-1.0-2025-04-28_131128.zip 	new file:   hardware/MSD-1.0/MSD-1.0-backups/MSD-1.0-2025-04-28_132753.zip 	new file:   hardware/MSD-1.0/MSD-1.0.csv 	modified:   hardware/MSD-1.0/MSD-1.0.kicad_pcb 	modified:   hardware/MSD-1.0/MSD-1.0.kicad_sch 	deleted:    hardware/PS-1.0/PS-1.0-backups/PS-1.0-2025-03-24_111800.zip 	deleted:    hardware/PS-1.0/PS-1.0-backups/PS-1.0-2025-03-24_112738.zip 	deleted:    hardware/PS-1.0/PS-1.0-backups/PS-1.0-2025-03-25_152833.zip 	deleted:    hardware/PS-1.0/PS-1.0-backups/PS-1.0-2025-03-25_154601.zip 	deleted:    hardware/PS-1.0/PS-1.0-backups/PS-1.0-2025-03-25_155821.zip 	deleted:    hardware/PS-1.0/PS-1.0-backups/PS-1.0-2025-04-11_101418.zip 	deleted:    hardware/PS-1.0/PS-1.0-backups/PS-1.0-2025-04-11_110528.zip 	deleted:    hardware/PS-1.0/PS-1.0-backups/PS-1.0-2025-04-11_111527.zip 	deleted:    hardware/PS-1.0/PS-1.0-backups/PS-1.0-2025-04-11_114252.zip 	deleted:    hardware/PS-1.0/PS-1.0-backups/PS-1.0-2025-04-17_105409.zip 	new file:   hardware/PS-1.0/PS-1.0-backups/PS-1.0-2025-04-19_071925.zip 	new file:   hardware/PS-1.0/PS-1.0-backups/PS-1.0-2025-04-27_222808.zip 	new file:   hardware/PS-1.0/PS-1.0-backups/PS-1.0-2025-04-27_223939.zip 	new file:   hardware/PS-1.0/PS-1.0-backups/PS-1.0-2025-04-27_224445.zip 	new file:   hardware/PS-1.0/PS-1.0-backups/PS-1.0-2025-04-27_225206.zip 	new file:   hardware/PS-1.0/PS-1.0-backups/PS-1.0-2025-04-27_230217.zip 	new file:   hardware/PS-1.0/PS-1.0-backups/PS-1.0-2025-04-28_083014.zip 	new file:   hardware/PS-1.0/PS-1.0-backups/PS-1.0-2025-04-28_112951.zip 	new file:   har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
Parts:
- C1: value 2.2nF -> 2.2nF 100
- C11, C12: value C -> 0.01µF 1000
- C2: value 10nF -> 10nF 63
- C3: value 0.022uF 400V MKP -> 0.022µF 400V
- C4: value 22nF -> 22nF 100
- C5, C6, C8: value 100nF -> 100nF 100
- J1: value Conn_01x04 -> PinHeader_2.54mm 02x04 Horizontal
- J2: value Conn_01x03 -> PinHeader_2.54mm 02x05 Horizontal
- R8, R9: value 33Ω -> 33Ω 2W
- RV1: value 1kΩ -> 5kΩ
Changed lines of the file:
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@@
 			)
 		)
-		(property "Value" "2.2nF"
+		(property "Value" "2.2nF 100"
 			(at 152.908 121.412 0)
 			(effects
@@
 			)
 		)
-		(property "Value" "33Ω"
+		(property "Value" "33Ω 2W"
 			(at 247.65 89.916 90)
 			(effects
@@
 			)
 		)
-		(property "Value" "100nF"
+		(property "Value" "100nF 100"
 			(at 145.288 121.92 0)
 			(effects
@@
 			)
 		)
-		(property "Value" "Conn_01x04"
+		(property "Value" "PinHeader_2.54mm 02x04 Horizontal"
 			(at 90.17 31.75 0)
 			(effects
@@
 			)
 		)
-		(property "Value" "10nF"
+		(property "Value" "10nF 63"
 			(at 160.528 121.412 0)
 			(effects
@@
 			)
 		)
-		(property "Value" "100nF"
+		(property "Value" "100nF 100"
 			(at 178.308 57.15 0)
 			(effects
@@
 			)
 		)
-		(property "Value" "33Ω"
+		(property "Value" "33Ω 2W"
 			(at 247.65 102.616 90)
 			(effects
@@
 			)
 		)
-		(property "Value" "C"
+		(property "Value" "0.01µF 1000"
 			(at 262.128 109.22 0)
 			(effects
@@
 			)
 		)
-		(property "Value" "100nF"
+		(property "Value" "100nF 100"
 			(at 165.608 57.15 0)
 			(effects
@@
 			)
 		)
-		(property "Value" "1kΩ"
+		(property "Value" "5kΩ"
 			(at 153.416 53.34 0)
 			(effects
@@
 			)
 		)
-		(property "Value" "Conn_01x03"
+		(property "Value" "PinHeader_2.54mm 02x05 Horizontal"
 			(at 279.4 86.3601 0)
 			(effects
@@
 			)
 		)
-		(property "Value" "22nF"
+		(property "Value" "22nF 100"
 			(at 218.948 57.15 0)
 			(effects
@@
 			)
 		)
-		(property "Value" "C"
+		(property "Value" "0.01µF 1000"
 			(at 254.508 109.22 0)
 			(effects
@@
 			)
 		)
-		(property "Value" "0.022uF 400V MKP"
+		(property "Value" "0.022µF 400V"
 			(at 224.028 96.012 0)
 			(effects
