File: hardware/REM-4.0/REM-4.0.kicad_sch (KiCad schematic)
At the start: 35 parts, among them J1 PinHeader_2.54mm 02x04 Horizo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, J2 PinHeader_2.54mm 02x05 Horizo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, Q1 IRF840, U1 NE555P

Commit message: modified:   .DS_Store 	new file:   CAD/FR_TEST.dxf 	modified:   Ferrite Transformer Calculation.xlsx 	new file:   archive/PR_ 0201_2026.docx 	modified:   archive/Purchase 20260105.xlsx 	new file:   archive/Purchase 20260209.zip 	new file:   archive/Purchase 20260209/Invoice | Tokopedia 1.pdf 	new file:   archive/Purchase 20260209/Invoice | Tokopedia 2.pdf 	new file:   archive/Purchase 20260209/Invoice | Tokopedia 3.pdf 	new file:   archive/Purchase 20260209/Invoice | Tokopedia 4.pdf 	new file:   archive/Purchase 20260209/Invoice | Tokopedia 5.pdf 	new file:   archive/Purchase_20260109_0924.jpg 	new file:   archive/Purchase_20260209_0924.xlsx 	new file:   archive/R parallel.xlsx 	modified:   firmware/ESP32-S3 PWM/include/config.h 	modified:   firmware/ESP32-S3 PWM/include/hardware_control.h 	modified:   firmware/ESP32-S3 PWM/platformio.ini 	modified:   firmware/ESP32-S3 PWM/src/hardware_control.cpp 	modified:   firmware/ESP32-S3 PWM/src/main.cpp 	new file:   hardware/CTL-4.3/CTL-4.3-backups/CTL-4.3-2026-02-11_163805.zip 	new file:   hardware/CTL-4.3/CTL-4.3-backups/CTL-4.3-2026-02-13_145455.zip 	new file:   hardware/CTL-4.3/CTL-4.3-backups/CTL-4.3-2026-02-13_163249.zip 	new file:   hardware/CTL-4.3/CTL-4.3-backups/CTL-4.3-2026-02-18_163417.zip 	new file:   hardware/CTL-4.3/CTL-4.3-backups/CTL-4.3-2026-02-19_083102.zip 	new file:   hardware/CTL-4.3/CTL-4.3-backups/CTL-4.3-2026-03-04_102408.zip 	modified:   hardware/CTL-4.3/fp-info-cache 	new file:   hardware/CTL-5.0/CTL-4.3-backups/CTL-4.3-2026-01-19_105947.zip 	new file:   hardware/CTL-5.0/CTL-4.3-backups/CTL-4.3-2026-01-19_110601.zip 	new file:   hardware/CTL-5.0/CTL-4.3-backups/CTL-4.3-2026-01-19_111804.zip 	new file:   hardware/CTL-5.0/CTL-4.3-backups/CTL-4.3-2026-01-19_113721.zip 	new file:   hardware/CTL-5.0/CTL-4.3-backups/CTL-4.3-2026-01-19_164107.zip 	new file:   hardware/CTL-5.0/CTL-4.3-backups/CTL-4.3-2026-01-20_112913.zip 	new file:   hardware/CTL-5.0/CTL-4.3-backups/CTL-4.3-2026-02-11_163805.zip 	new file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
Parts:
- removed JP1, JP2: TestPoint, TestPoint:TestPoint_THTPad_2.0x2.0mm_Drill1.0mm_NoSilkscreen, symbol Connector:TestPoint
- removed JP7, JP8: TestPoint, TestPoint:TestPoint_THTPad_D1.5mm_Drill0.7mm, symbol Connector:TestPoint
- removed TP6: ~, TestPoint:TestPoint_Bridge_Pitch2.54mm_Drill1.0mm, symbol Connector:TestPoint
- added D4: BAT54S, Package_TO_SOT_SMD:SOT-23, symbol Diode:BAT54S
- added R6: 120Ω 2W, Resistor_THT:R_Axial_DIN0414_L11.9mm_D4.5mm_P20.32mm_Horizontal, symbol Device:R
- added TP3: ~, TestPoint:TestPoint_Bridge_Pitch2.54mm_Drill1.0mm, symbol Connector:TestPoint
- D2, D3: value 1N4148 -> BAT85
- Q1: value IRF840 -> IRLB3034PbF
Connections:
- net GND: now also D4.1 (A), TP3.1
- net at C5.1, D3.1 (K), R5.1: now also D4.2 (K)
- net at C4.1, D2.1 (K), D3.2 (A)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: now also D4.3 (COM)
- net at L1.3, R9.2: now also R6.2
- net at L1.4, R8.2: now also R6.1
Other:
- moved on the sheet: C1, C11, C12, C2, C3, C4, C5, C6, C7, C8, D1, D2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

Commit message: modified:   .DS_Store 	modified:   Ferrite Transformer Calculation.xlsx 	new file:   archive/REM - Vsense.xlsx 	new file:   hardware/INA-1.0/#auto_saved_files# 	new file:   hardware/INA-1.0/INA-1.0-backups/INA-1.0-2026-04-10_134714.zip 	new file:   hardware/INA-1.0/INA-1.0-backups/INA-1.0-2026-04-10_141544.zip 	new file:   hardware/INA-1.0/INA-1.0-backups/INA-1.0-2026-04-10_154242.zip 	new file:   hardware/INA-1.0/INA-1.0-backups/INA-1.0-2026-04-10_161020.zip 	new file:   hardware/INA-1.0/INA-1.0-backups/INA-1.0-2026-04-10_163134.zip 	new file:   hardware/INA-1.0/INA-1.0-backups/INA-1.0-2026-04-12_233203.zip 	new file:   hardware/INA-1.0/INA-1.0-backups/INA-1.0-2026-04-12_234518.zip 	new file:   hardware/INA-1.0/INA-1.0-backups/INA-1.0-2026-04-13_105232.zip 	new file:   hardware/INA-1.0/INA-1.0-backups/INA-1.0-2026-04-13_105845.zip 	new file:   hardware/INA-1.0/INA-1.0-backups/INA-1.0-2026-04-13_110346.zip 	new file:   hardware/INA-1.0/INA-1.0-backups/INA-1.0-2026-04-13_112014.zip 	new file:   hardware/INA-1.0/INA-1.0-backups/INA-1.0-2026-04-13_112658.zip 	new file:   hardware/INA-1.0/INA-1.0-backups/INA-1.0-2026-04-13_114201.zip 	new file:   hardware/INA-1.0/INA-1.0.kicad_pcb 	new file:   hardware/INA-1.0/INA-1.0.kicad_prl 	new file:   hardware/INA-1.0/INA-1.0.kicad_pro 	new file:   hardware/INA-1.0/INA-1.0.kicad_sch 	new file:   hardware/INA-1.0/_autosave-INA-1.0.kicad_pcb 	new file:   hardware/INA-1.0/_autosave-INA-1.0.kicad_sch 	new file:   hardware/INA-1.0/fabrication-outputs/INA-1.0-F_Cu.dxf 	new file:   hardware/INA-1.0/fabrication-outputs/INA-1.0-F_Mask.dxf 	new file:   hardware/INA-1.0/fabrication-outputs/INA-1.0-NPTH-drl_map.dxf 	new file:   hardware/INA-1.0/fabrication-outputs/INA-1.0-PTH-drl_map.dxf 	new file:   hardware/INA-1.0/fabrication-outputs/TRACE.dxf 	new file:   hardware/INA-1.0/fp-info-cache 	renamed:    hardware/REM-4.0/~REM-4.0.kicad_pcb.lck -> hardware/INA-1.0/~INA-1.0.kicad_sch.lck 	new file:   hardware/INA-1.0/~_autosave-INA-1.0.kicad_pcb.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
Parts:
- added C9: 100nF 100, Capacitor_THT:C_Rect_L7.0mm_W3.5mm_P5.00mm, symbol Device:C
- added R7: 4.7kΩ, Resistor_THT:R_Axial_DIN0204_L3.6mm_D1.6mm_P7.62mm_Horizontal, symbol Device:R
Connections:
- net GND: now also C9.2
- net at C6.1, R5.2, RV1.3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: now also R7.1; no longer J1.1 (Pin_1)
- new net: C9.1, J1.1 (Pin_1), R7.2
Other:
- moved on the sheet: C4, C5, C6, D2, D3, D4, J1, R4, R5, RV1, TP3, TP5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
