File: hardware/XF-1.0/XF-1.0.kicad_pcb (KiCad board)
At the start: 2 copper layers, 100.3 x 111.8 mm, 23 parts, among them CN1 Conn_01x02, CN2 Conn_01x02, CN3 Conn_01x03, CN4 Conn_01x03, CN5 Conn_01x02, CN6 Conn_01x03, CN7 Conn_01x02

Commit message: modified:   .DS_Store 	new file:   hardware/.~Request PO 20250807.xlsx 	new file:   hardware/CTL-3.0/.~BoM.xlsx 	modified:   hardware/CTL-3.0/BoM.xlsx 	deleted:    hardware/PS-2.0/PS-2.0-backups/PS-2.0-2025-07-26_112315.zip 	deleted:    hardware/PS-2.0/PS-2.0-backups/PS-2.0-2025-07-26_113619.zip 	deleted:    hardware/PS-2.0/PS-2.0-backups/PS-2.0-2025-07-26_114654.zip 	deleted:    hardware/PS-2.0/PS-2.0-backups/PS-2.0-2025-08-06_121001.zip 	new file:   hardware/PS-2.0/PS-2.0-backups/PS-2.0-2025-08-07_142024.zip 	new file:   hardware/PS-2.0/PS-2.0-backups/PS-2.0-2025-08-07_143133.zip 	new file:   hardware/PS-2.0/PS-2.0-backups/PS-2.0-2025-08-07_145326.zip 	new file:   hardware/PS-2.0/PS-2.0-backups/PS-2.0-2025-08-07_160132.zip 	new file:   hardware/PS-2.0/PS-2.0-backups/PS-2.0-2025-08-07_161316.zip 	new file:   hardware/PS-2.0/_autosave-PS-2.0.kicad_pcb 	new file:   hardware/PS-2.0/~_autosave-PS-2.0.kicad_pcb.lck 	new file:   hardware/Request PO 20250807 1029.xlsx 	deleted:    hardware/XF-1.0/XF-1.0-backups/XF-1.0-2025-07-15_152320.zip 	deleted:    hardware/XF-1.0/XF-1.0-backups/XF-1.0-2025-07-15_154638.zip 	deleted:    hardware/XF-1.0/XF-1.0-backups/XF-1.0-2025-07-16_140719.zip 	deleted:    hardware/XF-1.0/XF-1.0-backups/XF-1.0-2025-07-17_145542.zip 	deleted:    hardware/XF-1.0/XF-1.0-backups/XF-1.0-2025-07-17_150101.zip 	deleted:    hardware/XF-1.0/XF-1.0-backups/XF-1.0-2025-07-17_150621.zip 	deleted:    hardware/XF-1.0/XF-1.0-backups/XF-1.0-2025-07-17_151256.zip 	new file:   hardware/XF-1.0/XF-1.0-backups/XF-1.0-2025-08-07_145812.zip 	new file:   hardware/XF-1.0/XF-1.0-backups/XF-1.0-2025-08-07_150444.zip 	new file:   hardware/XF-1.0/XF-1.0-backups/XF-1.0-2025-08-07_151358.zip 	new file:   hardware/XF-1.0/XF-1.0-backups/XF-1.0-2025-08-07_152043.zip 	new file:   hardware/XF-1.0/XF-1.0-backups/XF-1.0-2025-08-07_153427.zip 	new file:   hardware/XF-1.0/XF-1.0-backups/XF-1.0-2025-08-07_155906.zip 	modified:   hardware/XF-1.0/XF-1.0.kicad_pcb 	modified:   hardware/XF-1.0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
Parts:
- C1, C4: footprint Capacitor_THT:C_Rect_L13.0mm_W8.0mm_P10.00mm_FKS3_FKP3_MKS4 -> Capacitor_THT:C_Axial_L12.0mm_D6.5mm_P20.00mm_Horizontal
- moved H1 89.2 mm to (120.7, 52.4), turned to -90 degrees
- moved H2 88.9 mm to (31.1, 52.4), turned to -90 degrees
- moved H4 80.6 mm to (120.7, 131.8), turned to -90 degrees
- moved H3 80.3 mm to (31.1, 131.8), turned to -90 degrees
- moved C6 76.5 mm to (39.1, 60.9), turned to 90 degrees
- moved CN5 75.7 mm to (105.9, 54.4), turned to 180 degrees
- moved CN2 75.3 mm to (45.9, 140.6), turned to 0 degrees
- moved CN1 71.6 mm to (98.0, 140.6), turned to 0 degrees
- moved CN7 70.0 mm to (53.8, 54.4), turned to 180 degrees
- moved C2 69.7 mm to (112.7, 60.9)
- moved C1 68.9 mm to (111.9, 68.6), turned to 180 degrees
- moved CN6 63.0 mm to (83.8, 54.4), turned to 180 degrees
- moved CN3 58.1 mm to (68.0, 140.6), turned to 0 degrees
- moved L1 58.0 mm to (112.1, 81.9), turned to 90 degrees
- moved CN4 57.9 mm to (68.0, 68.8), turned to 0 degrees
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Routing:
- net Net-(CN4-Pin_2): track 101.2 -> 14.4 mm
- net Net-(CN4-Pin_1): track 96.7 -> 14.4 mm
- net Net-(CN4-Pin_3): track 105.1 -> 44.7 mm
- net Net-(C1-Pad1): track 15.4 -> 30.1 mm, vias 2 -> 3
- net Net-(CN5-Pin_2): track 26.5 -> 14.4 mm
- net Net-(CN5-Pin_1): track 26.5 -> 14.4 mm
- net Net-(C4-Pad1): track 15.4 -> 26.3 mm, vias 2 -> 3
- net Net-(C1-Pad2): track 15.4 -> 26.3 mm, vias 2 -> 3
- net Net-(C4-Pad2): track 15.4 -> 26.3 mm, vias 2 -> 3
- net Net-(CN3-Pin_1): track 112.9 -> 115.5 mm
- net Net-(CN2-Pin_1): track 11.3 -> 10.1 mm
- net Net-(CN1-Pin_1): track 11.3 -> 10.1 mm
- net Net-(CN2-Pin_2): track 11.3 -> 10.1 mm
- net Net-(CN1-Pin_2): track 11.3 -> 10.1 mm
- net Net-(CN3-Pin_3): track 100.3 -> 100.8 mm
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Other:
- board size 100.3 x 111.8 mm -> 99.1 x 99.7 mm

Commit message: modified:   .DS_Store 	modified:   README.md 	new file:   hardware/CTL-3.0/CTL-3.0-backups/CTL-3.0-2025-08-08_093936.zip 	new file:   hardware/CTL-3.0/CTL-3.0-backups/CTL-3.0-2025-08-08_103359.zip 	new file:   hardware/CTL-3.0/CTL-3.0-backups/CTL-3.0-2025-08-08_104842.zip 	new file:   hardware/CTL-3.0/CTL-3.0-backups/CTL-3.0-2025-08-08_105743.zip 	modified:   hardware/CTL-3.0/CTL-3.0.kicad_pcb 	modified:   hardware/CTL-3.0/CTL-3.0.kicad_sch 	modified:   hardware/CTL-3.0/CTL-3.0.step 	modified:   hardware/CTL-3.0/fp-info-cache 	modified:   hardware/MSD-1.0/MSD-1.0.step 	deleted:    hardware/PS-2.0/PS-2.0-backups/PS-2.0-2025-07-28_091511.zip 	deleted:    hardware/PS-2.0/PS-2.0-backups/PS-2.0-2025-07-28_120953.zip 	deleted:    hardware/PS-2.0/PS-2.0-backups/PS-2.0-2025-07-29_151613.zip 	deleted:    hardware/PS-2.0/PS-2.0-backups/PS-2.0-2025-07-30_104542.zip 	deleted:    hardware/PS-2.0/PS-2.0-backups/PS-2.0-2025-08-07_142024.zip 	new file:   hardware/PS-2.0/PS-2.0-backups/PS-2.0-2025-08-08_083444.zip 	new file:   hardware/PS-2.0/PS-2.0-backups/PS-2.0-2025-08-08_093021.zip 	new file:   hardware/PS-2.0/PS-2.0-backups/PS-2.0-2025-08-08_095017.zip 	new file:   hardware/PS-2.0/PS-2.0-backups/PS-2.0-2025-08-08_101231.zip 	new file:   hardware/PS-2.0/PS-2.0-backups/PS-2.0-2025-08-08_102520.zip 	modified:   hardware/PS-2.0/PS-2.0.kicad_pcb 	modified:   hardware/PS-2.0/PS-2.0.kicad_prl 	new file:   hardware/PS-2.0/~PS-2.0.kicad_pcb.lck 	modified:   hardware/REM-4.0/REM-4.0.step 	deleted:    hardware/XF-1.0/XF-1.0-backups/XF-1.0-2025-07-17_151907.zip 	deleted:    hardware/XF-1.0/XF-1.0-backups/XF-1.0-2025-08-07_145812.zip 	new file:   hardware/XF-1.0/XF-1.0-backups/XF-1.0-2025-08-08_083643.zip 	new file:   hardware/XF-1.0/XF-1.0-backups/XF-1.0-2025-08-08_100854.zip 	new file:   hardware/XF-1.0/XF-1.0-backups/XF-1.0-2025-08-08_101915.zip 	modified:   hardware/XF-1.0/XF-1.0.kicad_pcb 	modified:   hardware/XF-1.0/XF-1.0.step 	modified:   hardware/XF-1.0/fp-info-cache 	modified:   l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
Changed lines of the file:
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@@
 		)
 		(fp_text user "${REFERENCE}"
-			(at 3.96 -4.9 360)
+			(at 3.96 -4.9 0)
 			(layer "F.Fab")
 			(effects
@@
 			(pintype "passive")
 		)
-		(pad "2" thru_hole circle
+		(pad "2" thru_hole oval
 			(at 7.92 0)
-			(size 3.5 3.5)
+			(size 3.16 4.2)
 			(drill 1.8)
 			(layers "*.Cu" "*.Mask")
@@
 			(pinfunction "Pin_2")
 			(pintype "passive")
-			(thermal_bridge_angle 90)
+		)
+		(model "/Users/margabudi/Documents/KiCad/8.0/3dmodels/JST 3.96/JST-CH-Thru(V)-3Pin-3.96-2.step"
+			(offset
+				(xyz 3.96 0 0)
+			)
+			(scale
+				(xyz 1 1 1)
+			)
+			(rotate
+				(xyz 0 0 180)
+			)
 		)
 	)
@@
 		)
 		(fp_text user "${REFERENCE}"
-			(at 3.96 -4.9 360)
+			(at 3.96 -4.9 0)
 			(layer "F.Fab")
 			(effects
@@
 			(pintype "passive")
 		)
-		(pad "2" thru_hole circle
+		(pad "2" thru_hole oval
 			(at 7.92 0)
-			(size 3.5 3.5)
+			(size 3.16 4.2)
 			(drill 1.8)
 			(layers "*.Cu" "*.Mask")
@@
 			(pinfunction "Pin_2")
 			(pintype "passive")
-			(thermal_bridge_angle 90)
+		)
+		(model "/Users/margabudi/Documents/KiCad/8.0/3dmodels/JST 3.96/JST-CH-Thru(V)-3Pin-3.96-2.step"
+			(offset
+				(xyz 3.96 0 0)
+			)
+			(scale
+				(xyz 1 1 1)
+			)
+			(rotate
+				(xyz 0 0 180)
+			)
 		)
 	)
@@
 		(tags "connector Molex KK-396 vertical")
 		(property "Reference" "CN3"
-			(at 7.92 -3.81 360)
+			(at 7.92 -3.81 0)
 			(layer "F.SilkS")
 			(effects
@@
 		)
 		(property "Value" "Conn_01x03"
-			(at 7.92 6.35 360)
+			(at 7.92 6.35 0)
 			(layer "F.Fab")
 			(effects
@@
 		)
 		(fp_text user "${REFERENCE}"
-			(at 7.92 -4.9 360)
+			(at 7.92 -4.9 0)
 			(layer "F.Fab")
 			(effects
@@
 			)
 		)
-		(pad "1" thru_hole circle
+		(pad "1" thru_hole roundrect
 			(at 0 0)
-			(size 3.5 3.5)
+			(size 3.16 4.2)
 			(drill 1.8)
 			(layers "*.Cu" "*.Mask")
 			(remove_unused_layers no)
+			(roundrect_rratio 0.079114)
 			(net 22 "Net-(CN3-Pin_1)")
 			(pinfunction "Pin_1")
 			(pintype "passive")
-			(thermal_bridge_angle 90)
 		)
-		(pad "2" thru_hole circle
+		(pad "2" thru_hole oval
 			(at 7.92 0)
-			(size 3.5 3.5)
+			(size 3.16 4.2)
 			(drill 1.8)
 			(layers "*.Cu" "*.Mask")
@@
 			(pinfunction "Pin_2")
 			(pintype "passive")
-			(thermal_bridge_angle 90)
 		)
-		(pad "3" thru_hole circle
+		(pad "3" thru_hole oval
 			(at 15.84 0)
-			(size 3.5 3.5)
+			(size 3.16 4.2)
 			(drill 1.8)
 			(layers "*.Cu" "*.Mask")
@@
 			(pinfunction "Pin_3")
 			(pintype "passive")
-			(thermal_bridge_angle 90)
 		)
-		(model "${KICAD8_3DMODEL_DIR}/Connector_Molex.3dshapes/Molex_KK-396_5273-05A_1x05_P3.96mm_Vertical.wrl"
+		(model "/Users/margabudi/Documents/KiCad/8.0/3dmodels/JST 3.96/JST-CH-Thru(V)-5Pin-3.96-2.step"
 			(offset
-				(xyz 0 0 0)
+				(xyz 7.92 0 0)
 			)
 			(scale
@@
 			)
 			(rotate
-				(xyz 0 0 0)
+				(xyz 0 0 180)
 			)
 		)
@@
 		(tags "connector Molex KK-396 vertical")
 		(property "Reference" "CN6"
-			(at 7.92 -4.035 360)
+			(at 7.92 -4.035 0)
 			(layer "F.SilkS")
 			(effects
@@
 		)
 		(property "Value" "Conn_01x03"
-			(at 7.92 6.35 360)
+			(at 7.92 6.35 0)
 			(layer "F.Fab")
 			(effects
@@
 		)
 		(fp_text user "${REFERENCE}"
-			(at 7.92 -4.9 360)
+			(at 7.92 -4.9 0)
 			(layer "F.Fab")
 			(effects
@@
 			)
 		)
-		(pad "1" thru_hole circle
+		(pad "1" thru_hole roundrect
 			(at 0 0 180)
-			(size 3.5 3.5)
+			(size 3.16 4.2)
 			(drill 1.8)
 			(layers "*.Cu" "*.Mask")
 			(remove_unused_layers no)
+			(roundrect_rratio 0.079114)
 			(net 20 "Net-(CN4-Pin_3)")
 			(pinfunction "Pin_1")
 			(pintype "passive")
-			(thermal_bridge_angle 90)
 		)
-		(pad "2" thru_hole circle
+		(pad "2" thru_hole oval
 			(at 7.92 0 180)
-			(size 3.5 3.5)
+			(size 3.16 4.2)
 			(drill 1.8)
 			(layers "*.Cu" "*.Mask")
@@
 			(pinfunction "Pin_2")
 			(pintype "passive")
-			(thermal_bridge_angle 90)
 		)
-		(pad "3" thru_hole circle
+		(pad "3" thru_hole oval
 			(at 15.84 0 180)
-			(size 3.5 3.5)
+			(size 3.16 4.2)
 			(drill 1.8)
 			(layers "*.Cu" "*.Mask")
@@
 			(pinfunction "Pin_3")
 			(pintype "passive")
-			(thermal_bridge_angle 90)
 		)
-		(model "${KICAD8_3DMODEL_DIR}/Connector_Molex.3dshapes/Molex_KK-396_5273-05A_1x05_P3.96mm_Vertical.wrl"
+		(model "/Users/margabudi/Documents/KiCad/8.0/3dmodels/JST 3.96/JST-CH-Thru(V)-5Pin-3.96-2.step"
 			(offset
-				(xyz 0 0 0)
+				(xyz 7.92 0 0)
 			)
 			(scale
@@
 			)
 			(rotate
-				(xyz 0 0 0)
+				(xyz 0 0 180)
 			)
 		)
@@
 		(tags "Transformer Toroid horizontal laying Diameter 9mm Amidon T30 ")
 		(property "Reference" "XF2"
-			(at 0 0 360)
+			(at 0 0 0)
 			(layer "F.SilkS")
 			(effects
@@
 		)
 		(property "Value" "~"
-			(at 0 1.5875 360)
+			(at 0 1.5875 0)
 			(layer "F.Fab")
 			(effects
@@
 		)
 		(fp_text user "${REFERENCE}"
-			(at 0 0 360)
+			(at 0 0 0)
 			(layer "F.Fab")
 			(effects
@@
 		)
 		(fp_text user "${REFERENCE}"
-			(at 3.96 -4.9 360)
+			(at 3.96 -4.9 0)
 			(layer "F.Fab")
 			(effects
@@
 			)
 		)
-		(pad "1" thru_hole circle
+		(pad "1" thru_hole roundrect
 			(at 0 0 180)
-			(size 3.5 3.5)
+			(size 3.16 4.2)
 			(drill 1.8)
 			(layers "*.Cu" "*.Mask")
 			(remove_unused_layers no)
+			(roundrect_rratio 0.079114)
 			(net 12 "Net-(CN3-Pin_3)")
 			(pinfunction "Pin_1")
 			(pintype "passive")
-			(thermal_bridge_angle 90)
 		)
-		(pad "2" thru_hole circle
+		(pad "2" thru_hole oval
 			(at 7.92 0 180)
-			(size 3.5 3.5)
+			(size 3.16 4.2)
 			(drill 1.8)
 			(layers "*.Cu" "*.Mask")
@@
 			(pinfunction "Pin_2")
 			(pintype "passive")
-			(thermal_bridge_angle 90)
+		)
+		(model "/Users/margabudi/Documents/KiCad/8.0/3dmodels/JST 3.96/JST-CH-Thru(V)-3Pin-3.96-2.step"
+			(offset
+				(xyz 3.96 0 0)
+			)
+			(scale
+				(xyz 1 1 1)
+			)
+			(rotate
+				(xyz 0 0 180)
+			)
 		)
 	)
@@
 		(tags "C Axial series Axial Horizontal pin pitch 20mm  length 12mm diameter 6.5mm")
 		(property "Reference" "C4"
-			(at 10 0 360)
+			(at 10 0 0)
 			(layer "F.SilkS")
 			(effects
@@
 		)
 		(property "Value" "2.7nF"
-			(at 10 4.37 360)
+			(at 10 4.37 0)
 			(layer "F.Fab")
 			(effects
@@
 		)
 		(fp_text user "${REFERENCE}"
-			(at 10 0 360)
+			(at 10 0 0)
 			(layer "F.Fab")
 			(effects
@@
 		(tags "C Axial series Axial Horizontal pin pitch 20mm  length 12mm diameter 6.5mm")
 		(property "Reference" "C1"
-			(at 10 0 360)
+			(at 10 0 0)
 			(layer "F.SilkS")
 			(effects
@@
 		)
 		(property "Value" "2.7nF"
-			(at 10 4.37 360)
+			(at 10 4.37 0)
 			(layer "F.Fab")
 			(effects
@@
 		)
 		(fp_text user "${REFERENCE}"
-			(at 10 0 360)
+			(at 10 0 0)
 			(layer "F.Fab")
 			(effects
@@
 		(tags "connector Molex KK-396 vertical")
 		(property "Reference" "CN4"
-			(at 7.92 -3.81 360)
+			(at 7.92 -3.81 0)
 			(layer "F.SilkS")
 			(effects
@@
 		)
 		(property "Value" "Conn_01x03"
-			(at 7.92 6.35 360)
+			(at 7.92 6.35 0)
 			(layer "F.Fab")
 			(effects
@@
 		)
 		(fp_text user "${REFERENCE}"
-			(at 7.92 -4.9 360)
+			(at 7.92 -4.9 0)
 			(layer "F.Fab")
 			(effects
@@
 			(pintype "passive")
 		)
-		(pad "2" thru_hole circle
+		(pad "2" thru_hole oval
 			(at 7.92 0)
-			(size 3.5 3.5)
+			(size 3.16 4.2)
 			(drill 1.8)
 			(layers "*.Cu" "*.Mask")
@@
 			(pinfunction "Pin_2")
 			(pintype "passive")
-			(thermal_bridge_angle 90)
 		)
-		(pad "3" thru_hole circle
+		(pad "3" thru_hole oval
 			(at 15.84 0)
-			(size 3.5 3.5)
+			(size 3.16 4.2)
 			(drill 1.8)
 			(layers "*.Cu" "*.Mask")
@@
 			(pinfunction "Pin_3")
 			(pintype "passive")
-			(thermal_bridge_angle 90)
 		)
-		(model "${KICAD8_3DMODEL_DIR}/Connector_Molex.3dshapes/Molex_KK-396_5273-05A_1x05_P3.96mm_Vertical.wrl"
+		(model "/Users/margabudi/Documents/KiCad/8.0/3dmodels/JST 3.96/JST-CH-Thru(V)-5Pin-3.96-2.step"
 			(offset
-				(xyz 0 0 0)
+				(xyz 7.92 0 0)
 			)
 			(scale
@@
 			)
 			(rotate
-				(xyz 0 0 0)
+				(xyz 0 0 180)
 			)
 		)
@@
 		(tags "Transformer Toroid horizontal laying Diameter 9mm Amidon T30 ")
 		(property "Reference" "XF1"
-			(at 0 0 360)
+			(at 0 0 0)
 			(layer "F.SilkS")
 			(effects
@@
 		)
 		(property "Value" "~"
-			(at 0 1.5875 360)
+			(at 0 1.5875 0)
 			(layer "F.Fab")
 			(effects
@@
 		)
 		(fp_text user "${REFERENCE}"
-			(at 0 0 360)
+			(at 0 0 0)
 			(layer "F.Fab")
 			(effects
@@
 		)
 		(fp_text user "${REFERENCE}"
-			(at 3.96 -4.9 360)
+			(at 3.96 -4.9 0)
 			(layer "F.Fab")
 			(effects
@@
 			)
 		)
-		(pad "1" thru_hole circle
+		(pad "1" thru_hole roundrect
 			(at 0 0 180)
-			(size 3.5 3.5)
+			(size 3.16 4.2)
 			(drill 1.8)
 			(layers "*.Cu" "*.Mask")
 			(remove_unused_layers no)
+			(roundrect_rratio 0.079114)
 			(net 9 "Net-(CN5-Pin_1)")
 			(pinfunction "Pin_1")
 			(pintype "passive")
-			(thermal_bridge_angle 90)
 		)
-		(pad "2" thru_hole circle
+		(pad "2" thru_hole oval
 			(at 7.92 0 180)
-			(size 3.5 3.5)
+			(size 3.16 4.2)
 			(drill 1.8)
 			(layers "*.Cu" "*.Mask")
@@
 			(pinfunction "Pin_2")
 			(pintype "passive")
-			(thermal_bridge_angle 90)
+		)
+		(model "/Users/margabudi/Documents/KiCad/8.0/3dmodels/JST 3.96/JST-CH-Thru(V)-3Pin-3.96-2.step"
+			(offset
+				(xyz 3.96 0 0)
+			)
+			(scale
+				(xyz 1 1 1)
+			)
+			(rotate
+				(xyz 0 0 180)
+			)
 		)
 	)

Commit message: modified:   .DS_Store 	modified:   README.md 	deleted:    hardware/PS-2.0/PS-2.0-backups/PS-2.0-2025-08-12_110109.zip 	deleted:    hardware/PS-2.0/PS-2.0-backups/PS-2.0-2025-08-12_110823.zip 	new file:   hardware/PS-2.0/PS-2.0-backups/PS-2.0-2025-08-12_131017.zip 	new file:   hardware/PS-2.0/PS-2.0-backups/PS-2.0-2025-08-12_194453.zip 	modified:   hardware/PS-2.0/PS-2.0.kicad_sch 	deleted:    hardware/PS-2.0/~PS-2.0.kicad_pcb.lck 	deleted:    hardware/PS-2.0/~PS-2.0.kicad_sch.lck 	modified:   hardware/Request PO 20250807 1029.xlsx 	new file:   hardware/XF-1.0/XF-1.0-B_Cu.gbr 	new file:   hardware/XF-1.0/XF-1.0-B_Mask.gbr 	new file:   hardware/XF-1.0/XF-1.0-B_Paste.gbr 	new file:   hardware/XF-1.0/XF-1.0-B_Silkscreen.gbr 	new file:   hardware/XF-1.0/XF-1.0-Edge_Cuts.gbr 	new file:   hardware/XF-1.0/XF-1.0-F_Cu.gbr 	new file:   hardware/XF-1.0/XF-1.0-F_Mask.gbr 	new file:   hardware/XF-1.0/XF-1.0-F_Paste.gbr 	new file:   hardware/XF-1.0/XF-1.0-F_Silkscreen.gbr 	new file:   hardware/XF-1.0/XF-1.0-NPTH.drl 	new file:   hardware/XF-1.0/XF-1.0-PTH.drl 	deleted:    hardware/XF-1.0/XF-1.0-backups/XF-1.0-2025-07-24_195648.zip 	deleted:    hardware/XF-1.0/XF-1.0-backups/XF-1.0-2025-07-24_200323.zip 	deleted:    hardware/XF-1.0/XF-1.0-backups/XF-1.0-2025-07-24_200926.zip 	new file:   hardware/XF-1.0/XF-1.0-backups/XF-1.0-2025-08-12_131501.zip 	new file:   hardware/XF-1.0/XF-1.0-backups/XF-1.0-2025-08-12_133029.zip 	new file:   hardware/XF-1.0/XF-1.0-backups/XF-1.0-2025-08-12_151757.zip 	new file:   hardware/XF-1.0/XF-1.0-job.gbrjob 	modified:   hardware/XF-1.0/XF-1.0.kicad_pcb 	modified:   pic/.DS_Store 	new file:   pic/PS/400kHz/1/400kHz-1-comparison.png 	deleted:    pic/PS/400kHz/1/LC-29u-3n3/PS2.0.png 	new file:   pic/PS/400kHz/1/LC-29u-3n3/comparison.drawio 	new file:   pic/PS/400kHz/3/LC-47u-3n3/comparison.drawio 	modified:   pic/Reverse Engineering/.DS_Store 	new file:   pic/Reverse Engineering/20kHz/RigolDS0.png 	new file:   pic/Reverse Engineering/20kHz/RigolDS1.png 	n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
Changed lines of the file:
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@@
 			(outputformat 1)
 			(mirror no)
-			(drillshape 1)
+			(drillshape 0)
 			(scaleselection 1)
 			(outputdirectory "")
@@
 		(tags "connector Molex KK-396 vertical")
 		(property "Reference" "CN3"
-			(at 7.92 -3.81 0)
+			(at 7.92 -7.21 0)
 			(layer "F.SilkS")
 			(effects
@@
 		(tags "connector Molex KK-396 vertical")
 		(property "Reference" "CN6"
-			(at 7.92 -4.035 0)
+			(at 7.92 -7.21 0)
 			(layer "F.SilkS")
 			(effects
@@
 		(at 53.8075 54.385 180)
 		(property "Reference" "CN7"
-			(at 3.96 -3.4 180)
+			(at 3.96 -7.21 180)
 			(unlocked yes)
 			(layer "F.SilkS")
@@
 		(tags "connector Molex KK-396 vertical")
 		(property "Reference" "CN4"
-			(at 7.92 -3.81 0)
+			(at 7.92 7.0775 0)
 			(layer "F.SilkS")
 			(effects
@@
 		(at 105.8775 54.385 180)
 		(property "Reference" "CN5"
-			(at 3.96 -3.4 180)
+			(at 3.96 -7.21 180)
 			(unlocked yes)
 			(layer "F.SilkS")
