File: hardware/CTL-4.0/CTL-4.0.kicad_pcb (KiCad board)
At the start: 2 copper layers, 198.2 x 45.1 mm, 67 parts, among them J1 Conn_02x16_Top_Bottom, J3 Conn_01x03, J4 Conn_01x02, J5 Conn_02x06_Odd_Even, J6 Conn_01x04, J7 Conn_01x04, J8 Conn_01x04, K1 G5V-1, Q1 BCX56, Q2 BCX56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

Commit message: modified:   firmware/ESP32-S3 PWM/src/main.cpp 	new file:   hardware/CTL-4.0/CTL-4.0-backups/CTL-4.0-2025-09-30_152410.zip 	new file:   hardware/CTL-4.0/CTL-4.0-backups/CTL-4.0-2025-09-30_153003.zip 	new file:   hardware/CTL-4.0/CTL-4.0-backups/CTL-4.0-2025-09-30_153714.zip 	new file:   hardware/CTL-4.0/CTL-4.0-backups/CTL-4.0-2025-09-30_154923.zip 	new file:   hardware/CTL-4.0/CTL-4.0-backups/CTL-4.0-2025-09-30_155511.zip 	modified:   hardware/CTL-4.0/CTL-4.0.kicad_pcb 	modified:   hardware/CTL-4.0/CTL-4.0.kicad_sch 	modified:   hardware/CTL-4.0/fp-info-cache 	new file:   hardware/CTL-4.1/BoM.xlsx 	new file:   hardware/CTL-4.1/CTL-4.1-backups/CTL-4.1-2025-09-30_155705.zip 	new file:   hardware/CTL-4.1/CTL-4.1-backups/CTL-4.1-2025-09-30_160713.zip 	new file:   hardware/CTL-4.1/CTL-4.1-backups/CTL-4.1-2025-09-30_161258.zip 	new file:   hardware/CTL-4.1/CTL-4.1-backups/CTL-4.1-2025-09-30_161801.zip 	new file:   hardware/CTL-4.1/CTL-4.1-backups/CTL-4.1-2025-09-30_162354.zip 	new file:   hardware/CTL-4.1/CTL-4.1-backups/CTL-4.1-2025-09-30_163220.zip 	new file:   hardware/CTL-4.1/CTL-4.1.FCStd 	new file:   hardware/CTL-4.1/CTL-4.1.iges 	new file:   hardware/CTL-4.1/CTL-4.1.kicad_pcb 	new file:   hardware/CTL-4.1/CTL-4.1.kicad_prl 	new file:   hardware/CTL-4.1/CTL-4.1.kicad_pro 	new file:   hardware/CTL-4.1/CTL-4.1.kicad_sch 	new file:   hardware/CTL-4.1/CTL-4.1.png 	new file:   hardware/CTL-4.1/CTL-4.1.step 	new file:   hardware/CTL-4.1/fp-info-cache
Parts:
- added J2: ~, Connector_FFC-FPC:TE_1-84952-0_1x10-1MP_P1.0mm_Horizontal, F.Cu at (76.2, 108.6)
