File: hardware/PS-4.0/PS-4.0.kicad_pcb (KiCad board)
At the start: 2 copper layers, 227.3 x 199.4 mm, 71 parts, among them CN1 Conn_01x02, CN5 Conn_01x02, CN6 Conn_01x03, J1 PinSocket_02x16_P2.54mm_Verti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, K1 RAYEX-L90, K2 RAYEX-L90, K3 G2RL-2, K4 G2RL-2, Q1 IRFPE50, Q2 IRFPE50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

Commit message: modified:   .DS_Store 	new file:   CAD/enclosure.dwg 	new file:   CAD/front-panel.dwg 	new file:   CAD/socket-bipolar-v1.dwg 	new file:   CAD/socket-monopolar-v1.dwg 	new file:   CAD/socket-re-v1.dwg 	new file:   CAD/test-probe.dwg 	modified:   Ferrite Transformer Calculation.xlsx 	new file:   archive/Purchase 20260105.xlsx 	modified:   firmware/ESP32-S3 PWM/src/buzzer.cpp 	new file:   hardware/CTL-4.1/CTL-4.1-backups/CTL-4.1-2025-10-23_132246.zip 	new file:   hardware/CTL-4.1/CTL-4.1-backups/CTL-4.1-2025-11-21_160148.zip 	new file:   hardware/CTL-4.1/CTL-4.1-backups/CTL-4.1-2025-11-21_161233.zip 	new file:   hardware/CTL-4.1/CTL-4.1-backups/CTL-4.1-2025-11-21_161917.zip 	new file:   hardware/CTL-4.1/CTL-4.1-backups/CTL-4.1-2025-11-21_162924.zip 	new file:   hardware/CTL-4.1/CTL-4.1-backups/CTL-4.1-2025-11-21_163425.zip 	new file:   hardware/CTL-4.1/CTL-4.1-backups/CTL-4.1-2025-11-24_100545.zip 	new file:   hardware/CTL-4.1/CTL-4.1-backups/CTL-4.1-2026-01-01_173613.zip 	new file:   hardware/CTL-4.1/CTL-4.1-backups/CTL-4.1-2026-01-01_174207.zip 	new file:   hardware/CTL-4.1/CTL-4.1-backups/CTL-4.1-2026-01-01_174749.zip 	new file:   hardware/CTL-4.1/CTL-4.1-backups/CTL-4.1-2026-01-02_130920.zip 	new file:   hardware/CTL-4.1/CTL-4.1-backups/CTL-4.1-2026-01-06_145810.zip 	new file:   hardware/CTL-4.1/CTL-4.1-backups/CTL-4.1-2026-01-06_164111.zip 	modified:   hardware/CTL-4.1/CTL-4.1.kicad_pcb 	modified:   hardware/CTL-4.1/CTL-4.1.kicad_prl 	modified:   hardware/CTL-4.1/CTL-4.1.kicad_pro 	new file:   hardware/CTL-4.1/bom/ibom.html 	modified:   hardware/CTL-4.1/fp-info-cache 	new file:   hardware/PS-3.0/PS-3.0-backups/PS-3.0-2025-10-23_133252.zip 	new file:   hardware/PS-3.0/PS-3.0-backups/PS-3.0-2025-11-20_095956.zip 	new file:   hardware/PS-3.0/PS-3.0-backups/PS-3.0-2025-11-20_100505.zip 	deleted:    hardware/PS-4.0/PS-4.0-backups/PS-4.0-2025-10-01_154815.zip 	new file:   hardware/PS-4.0/PS-4.0-backups/PS-4.0-2025-10-23_133027.zip 	new file:   hardware/PS-4.0/PS-4.0-bac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
Parts:
- added C13: 2.7nF, Capacitor_THT:C_Rect_L18.0mm_W7.0mm_P15.00mm_FKS3_FKP3, F.Cu at (149.2, 176.2)
- added C14: 4.7nF, Capacitor_THT:C_Rect_L18.0mm_W7.0mm_P15.00mm_FKS3_FKP3, F.Cu at (149.2, 161.0)
- added C15: 4.7nF, Capacitor_THT:C_Rect_L18.0mm_W7.0mm_P15.00mm_FKS3_FKP3, F.Cu at (149.2, 191.5)
- added L12: 29µH, Inductor_THT:L_Radial_Multilayer_D8.0mm_P12.70mm, F.Cu at (170.2, 161.0)
- added L13: 29µH, Inductor_THT:L_Radial_Multilayer_D8.0mm_P12.70mm, F.Cu at (170.2, 191.5)
- C10, C7: footprint Capacitor_THT:C_Axial_L12.0mm_D6.5mm_P15.00mm_Horizontal -> Capacitor_THT:C_Rect_L18.0mm_W7.0mm_P15.00mm_FKS3_FKP3
- C11, C12, C8, C9: footprint Capacitor_THT:C_Rect_L13.0mm_W8.0mm_P10.00mm_FKS3_FKP3_MKS4 -> Capacitor_THT:C_Rect_L18.0mm_W7.0mm_P15.00mm_FKS3_FKP3
- moved L10 94.0 mm to (170.2, 100.6)
- moved C12 88.6 mm to (149.2, 131.1)
- moved C11 87.3 mm to (149.2, 100.6)
- moved L11 82.6 mm to (170.2, 131.1)
- moved C10 80.7 mm to (149.2, 115.9), turned to 90 degrees
- moved XF2 50.5 mm to (201.6, 115.9)
- moved D11 31.2 mm to (167.3, 142.2), turned to -90 degrees
- moved K3 25.2 mm to (236.5, 114.6), turned to 0 degrees
- moved XF3 20.7 mm to (201.6, 176.2)
- moved K4 20.6 mm to (162.2, 146.1), turned to -90 degrees
- moved D10 15.1 mm to (232.7, 109.5), turned to 0 degrees
- moved C7 14.0 mm to (149.5, 58.7)
- moved L9 13.3 mm to (170.2, 74.0)
- moved CN6 8.55 mm to (126.8, 168.3)
- moved L8 8.31 mm to (170.2, 43.5)
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- renumbered XF3 to XF2, XF2 to XF3
Connections:
- C11 pad 1: Net-(C10-Pad1) -> Net-(C10-Pad2)
- C11 pad 2: /ACTIVE_MN1 -> Net-(C11-Pad2)
- C12 pad 1: Net-(C10-Pad2) -> Net-(C10-Pad1)
- C12 pad 2: /ACTIVE_MN2 -> Net-(C12-Pad2)
- CN6 pad 1: /BTN_CUT -> /ACTIVE_MN1
- CN6 pad 2: /BTN_COAG -> /BTN_CUT
- CN6 pad 3: /ACTIVE_MN1 -> /BTN_COAG
- K3 pad 12: /XF2-2 -> Net-(K3-Pad12)
- K3 pad 14: /XF3-2 -> Net-(K3-Pad14)
- K3 pad 22: /XF2-1 -> Net-(K3-Pad22)
- K3 pad 24: /XF3-1 -> Net-(K3-Pad24)
- K4 pad 11: /MNo-1 -> /ACTIVE_MN1
- K4 pad 12: /XF2-4 -> Net-(C12-Pad2)
- K4 pad 14: /XF3-4 -> Net-(C15-Pad2)
- K4 pad 21: /MNo-2 -> /ACTIVE_MN2
- K4 pad 22: /XF2-3 -> Net-(C11-Pad2)
- K4 pad 24: /XF3-3 -> Net-(C14-Pad2)
- L10 pad 1: /MNo-1 -> Net-(L10-Pad1)
- L10 pad 2: Net-(C10-Pad1) -> Net-(C10-Pad2)
- L11 pad 1: /MNo-2 -> Net-(L11-Pad1)
- L11 pad 2: Net-(C10-Pad2) -> Net-(C10-Pad1)
- XF2 pad 1: /XF3-1 -> Net-(K3-Pad22)
- XF2 pad 2: /XF3-2 -> Net-(K3-Pad12)
- XF2 pad 3: /XF3-4 -> Net-(L11-Pad1)
- XF2 pad 4: /XF3-3 -> Net-(L10-Pad1)
- XF3 pad 1: /XF2-1 -> Net-(K3-Pad24)
- XF3 pad 2: /XF2-2 -> Net-(K3-Pad14)
- XF3 pad 3: /XF2-4 -> Net-(L13-Pad1)
- XF3 pad 4: /XF2-3 -> Net-(L12-Pad1)
Routing:
- net /BTN_CUT: track 173.7 -> 29.2 mm
- net /BTN_COAG: track 172.5 -> 33.8 mm
- net /XF3-3: track 101.5 -> 0.00 mm
- net /ACTIVE_MN1: track 181.2 -> 83.1 mm, vias 1 -> 0
- net /MNo-2: track 79.6 -> 0.00 mm, vias 2 -> 0
- net /XF3-4: track 68.8 -> 0.00 mm
- net /XF2-1: track 62.7 -> 0.00 mm
- net Net-(C11-Pad2): track 0.00 -> 55.8 mm
- net Net-(C15-Pad2): track 0.00 -> 55.5 mm
- net /XF2-2: track 54.5 -> 0.00 mm
- net Net-(K3-Pad24): track 0.00 -> 52.3 mm
- net /XF2-4: track 45.7 -> 0.00 mm
- net /XF2-3: track 45.7 -> 0.00 mm
- net /MNi-2: track 86.3 -> 42.7 mm
- net Net-(K3-Pad12): track 0.00 -> 40.4 mm
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