File: hardware/CTL-4.1/CTL-4.1.kicad_pcb (KiCad board)
At the start: 2 copper layers, 198.2 x 45.1 mm, 68 parts, among them J1 Conn_02x16_Top_Bottom, J3 Conn_01x03, J4 Conn_01x02, J5 Conn_02x06_Odd_Even, J6 Conn_01x04, J7 Conn_01x04, J8 Conn_01x04, K1 G5V-1, Q1 BCX56, Q2 BCX56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

Commit message: modified:   .DS_Store 	modified:   firmware/ESP32-S3 PWM/include/config.h 	modified:   firmware/ESP32-S3 PWM/src/display_comm.cpp 	modified:   firmware/ESP32-S3 PWM/src/main.cpp 	deleted:    hardware/CTL-4.1/CTL-4.1-backups/CTL-4.1-2025-09-30_155705.zip 	new file:   hardware/CTL-4.1/CTL-4.1-backups/CTL-4.1-2025-10-01_120127.zip 	new file:   hardware/CTL-4.1/CTL-4.1-backups/CTL-4.1-2025-10-01_132128.zip 	new file:   hardware/CTL-4.1/CTL-4.1-backups/CTL-4.1-2025-10-01_132655.zip 	new file:   hardware/CTL-4.1/CTL-4.1-backups/CTL-4.1-2025-10-01_140704.zip 	new file:   hardware/CTL-4.1/CTL-4.1-backups/CTL-4.1-2025-10-01_143344.zip 	new file:   hardware/CTL-4.1/CTL-4.1-backups/CTL-4.1-2025-10-01_163205.zip 	modified:   hardware/CTL-4.1/CTL-4.1.kicad_pcb 	modified:   hardware/CTL-4.1/CTL-4.1.kicad_prl 	modified:   hardware/CTL-4.1/CTL-4.1.kicad_pro 	new file:   hardware/PS-3.0/PS-3.0-backups/PS-3.0-2025-10-01_133217.zip 	new file:   hardware/PS-3.0/PS-3.0-backups/PS-3.0-2025-10-01_134157.zip 	new file:   hardware/PS-3.0/PS-3.0-backups/PS-3.0-2025-10-01_143300.zip 	modified:   hardware/PS-3.0/PS-3.0.kicad_prl 	new file:   hardware/PS-3.0/bom/ibom.html 	modified:   hardware/PS-3.0/fp-info-cache 	new file:   hardware/PS-4.0/CTL-4.0.step 	new file:   hardware/PS-4.0/ERC.rpt 	new file:   hardware/PS-4.0/MSD-1.0.step 	new file:   hardware/PS-4.0/PS-3.0-backups/PS-3.0-2025-08-19_144351.zip 	new file:   hardware/PS-4.0/PS-3.0-backups/PS-3.0-2025-08-20_200710.zip 	new file:   hardware/PS-4.0/PS-3.0-backups/PS-3.0-2025-08-20_201526.zip 	new file:   hardware/PS-4.0/PS-3.0-backups/PS-3.0-2025-08-20_202132.zip 	new file:   hardware/PS-4.0/PS-3.0-backups/PS-3.0-2025-08-20_202750.zip 	new file:   hardware/PS-4.0/PS-3.0-backups/PS-3.0-2025-08-20_203343.zip 	new file:   hardware/PS-4.0/PS-3.0-backups/PS-3.0-2025-08-21_144605.zip 	new file:   hardware/PS-4.0/PS-3.0-backups/PS-3.0-2025-08-21_145115.zip 	new file:   hardware/PS-4.0/PS-3.0-backups/PS-3.0-2025-08-22_134708.zip 	new file:   hard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
Parts:
- removed J8: Conn_01x04, Connector_PinHeader_2.54mm:PinHeader_1x04_P2.54mm_Vertical
- moved C10 11.3 mm to (86.4, 116.5)
- moved C11 10.4 mm to (89.5, 116.5)
- moved R16 5.21 mm to (80.0, 116.5), turned to -90 degrees
- moved C9 3.31 mm to (83.2, 116.5)
- moved C1 1.27 mm to (152.5, 119.4)
- moved C2 1.27 mm to (152.5, 147.3)
- moved C3 1.27 mm to (184.9, 119.4)
- moved C4 1.27 mm to (184.9, 147.3)
- moved D3 1.27 mm to (218.3, 127.6)
- moved D4 1.27 mm to (142.6, 150.5)
- moved D5 1.27 mm to (175.0, 150.5)
- moved L3 1.27 mm to (204.3, 135.6)
- moved Q3 1.27 mm to (79.4, 143.8)
- moved Q4 1.27 mm to (79.4, 137.5)
- moved Q6 1.27 mm to (97.8, 137.5)
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Routing:
- net +5V: track 185.3 -> 266.0 mm, vias 0 -> 2
- net /SW-COAG: track 6.80 -> 23.8 mm
- net /TXD.1: track 28.7 -> 45.1 mm, vias 1 -> 3
- net Net-(Q5-C): track 35.3 -> 51.5 mm, vias 1 -> 2
- net +3.3V: track 235.6 -> 251.0 mm, vias 4 -> 5
- net /RXD.1: track 31.3 -> 45.9 mm, vias 1 -> 3
- net /SEN-COAG: track 38.6 -> 48.8 mm
- net +12V: track 219.0 -> 228.8 mm
- net /PWM-EN: track 27.1 -> 35.0 mm
- net /CTL-BUZZ: track 52.5 -> 60.2 mm
- net /EN: track 68.6 -> 75.7 mm
- net /SEN-CUT: track 33.0 -> 39.8 mm
- net /D+: track 70.3 -> 65.1 mm
- net /D-: track 65.8 -> 61.8 mm
- net /REM: track 87.1 -> 89.6 mm
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
Commit message: modified:   .DS_Store 	new file:   CAD/enclosure.dwg 	new file:   CAD/front-panel.dwg 	new file:   CAD/socket-bipolar-v1.dwg 	new file:   CAD/socket-monopolar-v1.dwg 	new file:   CAD/socket-re-v1.dwg 	new file:   CAD/test-probe.dwg 	modified:   Ferrite Transformer Calculation.xlsx 	new file:   archive/Purchase 20260105.xlsx 	modified:   firmware/ESP32-S3 PWM/src/buzzer.cpp 	new file:   hardware/CTL-4.1/CTL-4.1-backups/CTL-4.1-2025-10-23_132246.zip 	new file:   hardware/CTL-4.1/CTL-4.1-backups/CTL-4.1-2025-11-21_160148.zip 	new file:   hardware/CTL-4.1/CTL-4.1-backups/CTL-4.1-2025-11-21_161233.zip 	new file:   hardware/CTL-4.1/CTL-4.1-backups/CTL-4.1-2025-11-21_161917.zip 	new file:   hardware/CTL-4.1/CTL-4.1-backups/CTL-4.1-2025-11-21_162924.zip 	new file:   hardware/CTL-4.1/CTL-4.1-backups/CTL-4.1-2025-11-21_163425.zip 	new file:   hardware/CTL-4.1/CTL-4.1-backups/CTL-4.1-2025-11-24_100545.zip 	new file:   hardware/CTL-4.1/CTL-4.1-backups/CTL-4.1-2026-01-01_173613.zip 	new file:   hardware/CTL-4.1/CTL-4.1-backups/CTL-4.1-2026-01-01_174207.zip 	new file:   hardware/CTL-4.1/CTL-4.1-backups/CTL-4.1-2026-01-01_174749.zip 	new file:   hardware/CTL-4.1/CTL-4.1-backups/CTL-4.1-2026-01-02_130920.zip 	new file:   hardware/CTL-4.1/CTL-4.1-backups/CTL-4.1-2026-01-06_145810.zip 	new file:   hardware/CTL-4.1/CTL-4.1-backups/CTL-4.1-2026-01-06_164111.zip 	modified:   hardware/CTL-4.1/CTL-4.1.kicad_pcb 	modified:   hardware/CTL-4.1/CTL-4.1.kicad_prl 	modified:   hardware/CTL-4.1/CTL-4.1.kicad_pro 	new file:   hardware/CTL-4.1/bom/ibom.html 	modified:   hardware/CTL-4.1/fp-info-cache 	new file:   hardware/PS-3.0/PS-3.0-backups/PS-3.0-2025-10-23_133252.zip 	new file:   hardware/PS-3.0/PS-3.0-backups/PS-3.0-2025-11-20_095956.zip 	new file:   hardware/PS-3.0/PS-3.0-backups/PS-3.0-2025-11-20_100505.zip 	deleted:    hardware/PS-4.0/PS-4.0-backups/PS-4.0-2025-10-01_154815.zip 	new file:   hardware/PS-4.0/PS-4.0-backups/PS-4.0-2025-10-23_133027.zip 	new file:   hardware/PS-4.0/PS-4.0-bac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
Parts:
- moved D1 1.21 mm to (154.6, 127.6)
- moved D2 1.15 mm to (187.0, 127.6)
- moved D3 1.09 mm to (219.4, 127.6)
- moved TP1 0.64 mm to (137.8, 150.2)
- moved D4 0.32 mm to (142.9, 150.5)
- moved R9 0.32 mm to (142.9, 147.3)
- moved C1 0.26 mm to (152.7, 119.4)
- moved C2 0.26 mm to (152.7, 147.3)
- moved D5 0.26 mm to (175.3, 150.5)
- moved R10 0.26 mm to (175.3, 147.3)
- moved D6 0.20 mm to (207.6, 150.5)
- moved R11 0.20 mm to (207.6, 147.3)
- moved C3 0.20 mm to (185.1, 119.4)
- moved C4 0.20 mm to (185.1, 147.3)
- moved U3 0.15 mm to (222.2, 135.6)
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Connections:
- J2 pad MP: unconnected-(J2-MountPin-PadMP) -> (no net)
Routing:
- net +24V: track 297.9 -> 176.2 mm, vias 5 -> 20
- net +5V: track 266.0 -> 220.1 mm
- net +12V: track 228.8 -> 183.4 mm
- net +3.3V: track 251.0 -> 209.6 mm
- net Net-(D2-K): track 21.2 -> 19.7 mm
- net Net-(D1-K): track 21.2 -> 19.7 mm
- net Net-(D3-K): track 21.2 -> 19.8 mm
- net /BUZZ: track 51.6 -> 52.6 mm, vias 1 -> 2
- net /RXD.1: track 45.9 -> 46.5 mm
- net /PWM.00: track 25.9 -> 25.3 mm
- net Net-(Q5-C): track 51.5 -> 50.9 mm, vias 2 -> 1
- net /CTL-BUZZ: track 60.2 -> 59.6 mm
- net /REM: track 89.6 -> 89.1 mm
- net GND: vias 39 -> 111
- added copper zone on F.Cu, net +12V
- added copper zone on B.Cu, net +24V
- added copper zone on F.Cu, net +24V
- added copper zone on F.Cu, net +3.3V
- added copper zone on F.Cu, net +5V
Other:
- board text added: "+3.3V"
- board text added: "+5V"
- board text added: "CN1"
- board text added: "CN2"
- board text added: "CN3"
- board text added: "CN4"
- board text added: "CN5"
- board text added: "DTR"
- board text added: "GND"
- board text added: "RTS"
- board text added: "RX.0"
- board text added: "RX.1"
- board text added: "TCK"
- board text added: "TDI"
- board text added: "TDO"
- board text added: "TMS"
- board text added: "TX.0"
- board text added: "TX.1"
