File: hardware/CTL-4.1/CTL-4.1.kicad_sch (KiCad schematic)
At the start: 68 parts, among them J1 Conn_02x16_Top_Bottom, J3 Conn_01x03, J4 Conn_01x02, J5 Conn_02x06_Odd_Even, J6 Conn_01x04, J7 Conn_01x04, J8 Conn_01x04, K1 G5V-1, Q1 BCX56, Q2 BCX56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

Commit message: modified:   .DS_Store 	modified:   archive/Purchase 20260105.xlsx 	deleted:    hardware/CTL-4.1/BoM.xlsx 	new file:   hardware/CTL-4.1/CTL-4.1-backups/CTL-4.1-2026-01-07_112112.zip 	new file:   hardware/CTL-4.1/CTL-4.1-backups/CTL-4.1-2026-01-07_112720.zip 	modified:   hardware/CTL-4.1/CTL-4.1.kicad_pcb 	modified:   hardware/CTL-4.1/CTL-4.1.kicad_sch 	new file:   hardware/CTL-4.1/CTL-4.1.xlsx 	new file:   hardware/CTL-4.2/CTL-4.1-backups/CTL-4.1-2025-09-30_160713.zip 	new file:   hardware/CTL-4.2/CTL-4.1-backups/CTL-4.1-2025-09-30_161258.zip 	new file:   hardware/CTL-4.2/CTL-4.1-backups/CTL-4.1-2025-09-30_161801.zip 	new file:   hardware/CTL-4.2/CTL-4.1-backups/CTL-4.1-2025-09-30_162354.zip 	new file:   hardware/CTL-4.2/CTL-4.1-backups/CTL-4.1-2025-09-30_163220.zip 	new file:   hardware/CTL-4.2/CTL-4.1-backups/CTL-4.1-2025-10-01_132128.zip 	new file:   hardware/CTL-4.2/CTL-4.1-backups/CTL-4.1-2025-10-01_132655.zip 	new file:   hardware/CTL-4.2/CTL-4.1-backups/CTL-4.1-2025-10-01_140704.zip 	new file:   hardware/CTL-4.2/CTL-4.1-backups/CTL-4.1-2025-10-01_143344.zip 	new file:   hardware/CTL-4.2/CTL-4.1-backups/CTL-4.1-2025-10-01_163205.zip 	new file:   hardware/CTL-4.2/CTL-4.1-backups/CTL-4.1-2025-10-03_094957.zip 	new file:   hardware/CTL-4.2/CTL-4.1-backups/CTL-4.1-2025-10-23_132246.zip 	new file:   hardware/CTL-4.2/CTL-4.1-backups/CTL-4.1-2025-11-21_160148.zip 	new file:   hardware/CTL-4.2/CTL-4.1-backups/CTL-4.1-2025-11-21_161233.zip 	new file:   hardware/CTL-4.2/CTL-4.1-backups/CTL-4.1-2025-11-21_161917.zip 	new file:   hardware/CTL-4.2/CTL-4.1-backups/CTL-4.1-2025-11-21_162924.zip 	new file:   hardware/CTL-4.2/CTL-4.1-backups/CTL-4.1-2025-11-21_163425.zip 	new file:   hardware/CTL-4.2/CTL-4.1-backups/CTL-4.1-2025-11-24_100545.zip 	new file:   hardware/CTL-4.2/CTL-4.1-backups/CTL-4.1-2026-01-01_173613.zip 	new file:   hardware/CTL-4.2/CTL-4.1-backups/CTL-4.1-2026-01-01_174207.zip 	new file:   hardware/CTL-4.2/CTL-4.1-backups/CTL-4.1-2026-01-01_174749.zip 	new fil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
Connections:
- net +12V: no longer J4.1 (Pin_1)
- net +5V: now also J4.1 (Pin_1)
Changed lines of the file:
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@@
 		)
 	)
-	(label "+12V"
+	(label "+5V"
 		(at 354.33 83.82 0)
 		(fields_autoplaced yes)
