File: hardware/CTL-4.2/CTL-4.2.kicad_pcb (KiCad board)
At the start: 2 copper layers, 198.2 x 45.1 mm, 72 parts, among them J1 Conn_02x16_Top_Bottom, J3 Conn_01x03, J4 Conn_01x03, J5 Conn_02x06_Odd_Even, J6 Conn_01x04, J7 Conn_01x04, K1 G5V-1, Q1 BCX56, Q2 BCX56, Q3 BCX56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

Commit message: modified:   .DS_Store 	modified:   archive/Purchase 20260105.xlsx 	deleted:    hardware/CTL-4.2/CTL-4.2-backups/CTL-4.2-2026-01-07_141653.zip 	deleted:    hardware/CTL-4.2/CTL-4.2-backups/CTL-4.2-2026-01-07_142924.zip 	deleted:    hardware/CTL-4.2/CTL-4.2-backups/CTL-4.2-2026-01-07_143704.zip 	deleted:    hardware/CTL-4.2/CTL-4.2-backups/CTL-4.2-2026-01-07_144240.zip 	deleted:    hardware/CTL-4.2/CTL-4.2-backups/CTL-4.2-2026-01-07_172928.zip 	deleted:    hardware/CTL-4.2/CTL-4.2-backups/CTL-4.2-2026-01-08_104233.zip 	deleted:    hardware/CTL-4.2/CTL-4.2-backups/CTL-4.2-2026-01-08_105414.zip 	deleted:    hardware/CTL-4.2/CTL-4.2-backups/CTL-4.2-2026-01-08_110821.zip 	deleted:    hardware/CTL-4.2/CTL-4.2-backups/CTL-4.2-2026-01-08_113902.zip 	new file:   hardware/CTL-4.2/CTL-4.2-backups/CTL-4.2-2026-01-09_161105.zip 	new file:   hardware/CTL-4.2/CTL-4.2-backups/CTL-4.2-2026-01-09_161607.zip 	new file:   hardware/CTL-4.2/CTL-4.2-backups/CTL-4.2-2026-01-09_162214.zip 	new file:   hardware/CTL-4.2/CTL-4.2-backups/CTL-4.2-2026-01-09_162911.zip 	new file:   hardware/CTL-4.2/CTL-4.2-backups/CTL-4.2-2026-01-09_163538.zip 	new file:   hardware/CTL-4.2/CTL-4.2-backups/CTL-4.2-2026-01-10_175837.zip 	new file:   hardware/CTL-4.2/CTL-4.2-backups/CTL-4.2-2026-01-12_160020.zip 	new file:   hardware/CTL-4.2/CTL-4.2-backups/CTL-4.2-2026-01-12_160649.zip 	new file:   hardware/CTL-4.2/CTL-4.2-backups/CTL-4.2-2026-01-12_161345.zip 	new file:   hardware/CTL-4.2/CTL-4.2-backups/CTL-4.2-2026-01-12_162048.zip 	new file:   hardware/CTL-4.2/CTL-4.2-backups/CTL-4.2-2026-01-12_165205.zip 	new file:   hardware/CTL-4.2/CTL-4.2-backups/CTL-4.2-2026-01-13_144014.zip 	new file:   hardware/CTL-4.2/CTL-4.2-backups/CTL-4.2-2026-01-13_150252.zip 	new file:   hardware/CTL-4.2/CTL-4.2-backups/CTL-4.2-2026-01-13_151249.zip 	new file:   hardware/CTL-4.2/CTL-4.2-backups/CTL-4.2-2026-01-13_151858.zip 	new file:   hardware/CTL-4.2/CTL-4.2-backups/CTL-4.2-2026-01-13_163249.zip 	new file:   hardware/CTL-4.2/CTL-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
Parts:
- C10: value 22µF 10V -> 10µF 10V; footprint Capacitor_Tantalum_SMD:CP_EIA-3528-12_Kemet-T_Pad1.50x2.35mm_HandSolder -> Capacitor_Tantalum_SMD:CP_EIA-3216-18_Kemet-A_Pad1.58x1.35mm_HandSolder
- C11, C7, C8, C9: footprint Capacitor_SMD:C_1206_3216Metric_Pad1.33x1.80mm_HandSolder -> Capacitor_SMD:C_0805_2012Metric_Pad1.18x1.45mm_HandSolder
- D7: value BAT60A -> SS32; footprint Diode_SMD:D_SMB_Handsoldering -> Diode_SMD:D_SMA
- R1, R12, R13, R15, R16, R17, R18, R19, R2, R20, R3, R4, R5, R6, R7, R8: footprint Resistor_SMD:R_1206_3216Metric_Pad1.30x1.75mm_HandSolder -> Resistor_SMD:R_0805_2012Metric_Pad1.20x1.40mm_HandSolder
- moved Q6 18.9 mm to (79.4, 143.8)
- moved R20 18.9 mm to (83.2, 143.8)
- moved R16 8.94 mm to (88.7, 118.4)
- moved C9 7.70 mm to (90.6, 118.4)
- moved Q3 6.35 mm to (79.4, 137.5)
- moved Q4 6.35 mm to (79.4, 131.1)
- moved R3 6.35 mm to (83.2, 137.5)
- moved R4 6.35 mm to (83.2, 131.1)
- moved R15 5.05 mm to (81.1, 125.3)
- moved R18 4.67 mm to (79.2, 125.3)
- moved R17 4.63 mm to (77.3, 125.3)
- moved R21 4.13 mm to (87.6, 131.1)
- moved R22 4.13 mm to (89.9, 131.1)
- moved C11 3.30 mm to (86.8, 118.4), turned to 90 degrees
- moved C10 2.64 mm to (88.6, 115.1), turned to 180 degrees
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Connections:
- net +24V renamed +36V
Routing:
- net /RLY-A.2: track 38.1 -> 15.3 mm
- net /CTL-RLY-A.2: track 30.9 -> 52.2 mm
- net /EN: track 74.5 -> 54.6 mm
- net +3.3V: track 209.6 -> 198.9 mm
- net /BUZZ: track 52.6 -> 58.4 mm
- net +5V: track 223.8 -> 229.4 mm
- net /RLY-A.1: track 18.2 -> 23.1 mm
- net /MSD1: track 69.7 -> 73.8 mm
- net +36V: track 176.2 -> 173.5 mm, vias 20 -> 15
- net /DTR: track 62.2 -> 59.8 mm
- net /RTS: track 66.9 -> 64.7 mm
- net /MSD2: track 70.7 -> 72.3 mm
- net /REM: track 90.4 -> 88.9 mm
- net /RXD.1: track 44.3 -> 42.8 mm
- net /CTL-RLY-A.1: track 30.6 -> 29.2 mm
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- added copper zone on B.Cu, net Net-(Q5-C)
Other:
- board text added: "CN6"
- board text added: "CN7"
