File: hardware/CTL-4.3/CTL-4.3.kicad_pcb (KiCad board)
At the start: 2 copper layers, 198.2 x 45.1 mm, 72 parts, among them J1 Conn_02x16_Top_Bottom, J3 Conn_01x03, J4 Conn_01x03, J5 Conn_02x06_Odd_Even, J6 Conn_01x04, J7 Conn_01x04, K1 G5V-1, Q1 BCX56, Q2 BCX56, Q3 BCX56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

Commit message: modified:   .DS_Store 	modified:   archive/Purchase 20260105.xlsx 	deleted:    hardware/CTL-4.3/CTL-4.3-backups/CTL-4.3-2026-01-19_090613.zip 	renamed:    hardware/CTL-4.3/CTL-4.3-backups/CTL-4.3-2026-01-19_091818.zip -> hardware/CTL-4.3/CTL-4.3-backups/CTL-4.3-2026-01-19_105947.zip 	new file:   hardware/CTL-4.3/CTL-4.3-backups/CTL-4.3-2026-01-19_110601.zip 	new file:   hardware/CTL-4.3/CTL-4.3-backups/CTL-4.3-2026-01-19_111804.zip 	new file:   hardware/CTL-4.3/CTL-4.3-backups/CTL-4.3-2026-01-19_113721.zip 	new file:   hardware/CTL-4.3/CTL-4.3-backups/CTL-4.3-2026-01-19_164107.zip 	new file:   hardware/CTL-4.3/CTL-4.3-backups/CTL-4.3-2026-01-20_112913.zip 	modified:   hardware/CTL-4.3/CTL-4.3.kicad_pcb 	modified:   hardware/CTL-4.3/CTL-4.3.kicad_sch 	modified:   hardware/CTL-4.3/bom/ibom.html 	modified:   hardware/CTL-4.3/fp-info-cache 	new file:   hardware/PS-5.1/PS-5.1-backups/PS-5.1-2026-01-19_103049.zip
Parts:
- C10: value 10µF 10V -> 22µF 10V
- D4, D5, D6: footprint LED_SMD:LED_1206_3216Metric_Pad1.42x1.75mm_HandSolder -> LED_SMD:LED_0805_2012Metric_Pad1.15x1.40mm_HandSolder
- R10, R11, R9: footprint Resistor_SMD:R_1206_3216Metric_Pad1.30x1.75mm_HandSolder -> Resistor_SMD:R_0805_2012Metric_Pad1.20x1.40mm_HandSolder
- moved D5 0.71 mm to (155.6, 50.2)
- moved R10 0.71 mm to (155.6, 47.6)
- moved D4 0.71 mm to (123.2, 50.2)
- moved R9 0.71 mm to (123.2, 47.6)
- moved D6 0.71 mm to (188.0, 50.2)
- moved R11 0.71 mm to (188.0, 47.6)
Routing:
- net Net-(D6-A): track 3.18 -> 2.54 mm
- net Net-(D5-A): track 3.18 -> 2.54 mm
- net Net-(D4-A): track 3.18 -> 2.54 mm
