File: hardware/CTL-4.3/CTL-4.3.kicad_sch (KiCad schematic)
At the start: 73 parts, among them J1 Conn_02x16_Top_Bottom, J3 Conn_01x03, J4 Conn_01x03, J5 Conn_02x06_Odd_Even, J6 Conn_01x04, J7 Conn_01x04, J8 Conn_01x04, K1 G5V-1, Q1 BCX56, Q2 BCX56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

Commit message: modified:   .DS_Store 	modified:   archive/Purchase 20260105.xlsx 	deleted:    hardware/CTL-4.3/CTL-4.3-backups/CTL-4.3-2026-01-19_090613.zip 	renamed:    hardware/CTL-4.3/CTL-4.3-backups/CTL-4.3-2026-01-19_091818.zip -> hardware/CTL-4.3/CTL-4.3-backups/CTL-4.3-2026-01-19_105947.zip 	new file:   hardware/CTL-4.3/CTL-4.3-backups/CTL-4.3-2026-01-19_110601.zip 	new file:   hardware/CTL-4.3/CTL-4.3-backups/CTL-4.3-2026-01-19_111804.zip 	new file:   hardware/CTL-4.3/CTL-4.3-backups/CTL-4.3-2026-01-19_113721.zip 	new file:   hardware/CTL-4.3/CTL-4.3-backups/CTL-4.3-2026-01-19_164107.zip 	new file:   hardware/CTL-4.3/CTL-4.3-backups/CTL-4.3-2026-01-20_112913.zip 	modified:   hardware/CTL-4.3/CTL-4.3.kicad_pcb 	modified:   hardware/CTL-4.3/CTL-4.3.kicad_sch 	modified:   hardware/CTL-4.3/bom/ibom.html 	modified:   hardware/CTL-4.3/fp-info-cache 	new file:   hardware/PS-5.1/PS-5.1-backups/PS-5.1-2026-01-19_103049.zip
Parts:
- C10: value 10µF 10V -> 22µF 10V
- D4, D5, D6: footprint LED_SMD:LED_1206_3216Metric_Pad1.42x1.75mm_HandSolder -> LED_SMD:LED_0805_2012Metric_Pad1.15x1.40mm_HandSolder
- R10, R11, R9: footprint Resistor_SMD:R_1206_3216Metric_Pad1.30x1.75mm_HandSolder -> Resistor_SMD:R_0805_2012Metric_Pad1.20x1.40mm_HandSolder
Changed lines of the file:
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@@
 			)
 		)
-		(property "Footprint" "LED_SMD:LED_1206_3216Metric_Pad1.42x1.75mm_HandSolder"
+		(property "Footprint" "LED_SMD:LED_0805_2012Metric_Pad1.15x1.40mm_HandSolder"
 			(at 111.76 67.31 0)
 			(effects
@@
 			)
 		)
-		(property "Footprint" "LED_SMD:LED_1206_3216Metric_Pad1.42x1.75mm_HandSolder"
+		(property "Footprint" "LED_SMD:LED_0805_2012Metric_Pad1.15x1.40mm_HandSolder"
 			(at 111.76 34.29 0)
 			(effects
@@
 			)
 		)
-		(property "Footprint" "Resistor_SMD:R_1206_3216Metric_Pad1.30x1.75mm_HandSolder"
+		(property "Footprint" "Resistor_SMD:R_0805_2012Metric_Pad1.20x1.40mm_HandSolder"
 			(at 105.41 62.738 90)
 			(effects
@@
 			)
 		)
-		(property "Value" "10µF 10V"
+		(property "Value" "22µF 10V"
 			(at 103.124 167.64 90)
 			(effects
@@
 			)
 		)
-		(property "Footprint" "LED_SMD:LED_1206_3216Metric_Pad1.42x1.75mm_HandSolder"
+		(property "Footprint" "LED_SMD:LED_0805_2012Metric_Pad1.15x1.40mm_HandSolder"
 			(at 111.76 100.33 0)
 			(effects
@@
 			)
 		)
-		(property "Footprint" "Resistor_SMD:R_1206_3216Metric_Pad1.30x1.75mm_HandSolder"
+		(property "Footprint" "Resistor_SMD:R_0805_2012Metric_Pad1.20x1.40mm_HandSolder"
 			(at 105.41 95.758 90)
 			(effects
@@
 			)
 		)
-		(property "Footprint" "Resistor_SMD:R_1206_3216Metric_Pad1.30x1.75mm_HandSolder"
+		(property "Footprint" "Resistor_SMD:R_0805_2012Metric_Pad1.20x1.40mm_HandSolder"
 			(at 105.41 29.718 90)
 			(effects
