File: hardware/PS-5.1/PS-5.1.kicad_sch (KiCad schematic)
At the start: 67 parts, among them CN5 Conn_01x02, CN6 Conn_01x03, J1 PinSocket_02x16_P2.54mm_Verti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, K1 RAYEX-L90, K2 RAYEX-L90, Q1 IRFPE50, Q2 IRFPE50, Q3 IRFPE50, U1 TC4422/ TC4420, U4 PC817

Commit message: modified:   .DS_Store 	new file:   CAD/FR_TEST.dxf 	modified:   Ferrite Transformer Calculation.xlsx 	new file:   archive/PR_ 0201_2026.docx 	modified:   archive/Purchase 20260105.xlsx 	new file:   archive/Purchase 20260209.zip 	new file:   archive/Purchase 20260209/Invoice | Tokopedia 1.pdf 	new file:   archive/Purchase 20260209/Invoice | Tokopedia 2.pdf 	new file:   archive/Purchase 20260209/Invoice | Tokopedia 3.pdf 	new file:   archive/Purchase 20260209/Invoice | Tokopedia 4.pdf 	new file:   archive/Purchase 20260209/Invoice | Tokopedia 5.pdf 	new file:   archive/Purchase_20260109_0924.jpg 	new file:   archive/Purchase_20260209_0924.xlsx 	new file:   archive/R parallel.xlsx 	modified:   firmware/ESP32-S3 PWM/include/config.h 	modified:   firmware/ESP32-S3 PWM/include/hardware_control.h 	modified:   firmware/ESP32-S3 PWM/platformio.ini 	modified:   firmware/ESP32-S3 PWM/src/hardware_control.cpp 	modified:   firmware/ESP32-S3 PWM/src/main.cpp 	new file:   hardware/CTL-4.3/CTL-4.3-backups/CTL-4.3-2026-02-11_163805.zip 	new file:   hardware/CTL-4.3/CTL-4.3-backups/CTL-4.3-2026-02-13_145455.zip 	new file:   hardware/CTL-4.3/CTL-4.3-backups/CTL-4.3-2026-02-13_163249.zip 	new file:   hardware/CTL-4.3/CTL-4.3-backups/CTL-4.3-2026-02-18_163417.zip 	new file:   hardware/CTL-4.3/CTL-4.3-backups/CTL-4.3-2026-02-19_083102.zip 	new file:   hardware/CTL-4.3/CTL-4.3-backups/CTL-4.3-2026-03-04_102408.zip 	modified:   hardware/CTL-4.3/fp-info-cache 	new file:   hardware/CTL-5.0/CTL-4.3-backups/CTL-4.3-2026-01-19_105947.zip 	new file:   hardware/CTL-5.0/CTL-4.3-backups/CTL-4.3-2026-01-19_110601.zip 	new file:   hardware/CTL-5.0/CTL-4.3-backups/CTL-4.3-2026-01-19_111804.zip 	new file:   hardware/CTL-5.0/CTL-4.3-backups/CTL-4.3-2026-01-19_113721.zip 	new file:   hardware/CTL-5.0/CTL-4.3-backups/CTL-4.3-2026-01-19_164107.zip 	new file:   hardware/CTL-5.0/CTL-4.3-backups/CTL-4.3-2026-01-20_112913.zip 	new file:   hardware/CTL-5.0/CTL-4.3-backups/CTL-4.3-2026-02-11_163805.zip 	new file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
Parts:
- U3: footprint Custom:ESU-MSD-1.0 -> Custom:ESU-REM-4.0
Connections:
- net RLY-K renamed +12V
Changed lines of the file:
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@@
 		)
 	)
-	(label "RLY-K"
+	(label "+12V"
 		(at 24.13 50.8 0)
 		(fields_autoplaced yes)
@@
 			)
 		)
-		(property "Footprint" "Custom:ESU-MSD-1.0"
+		(property "Footprint" "Custom:ESU-REM-4.0"
 			(at 83.82 214.63 0)
 			(effects
