File: hardware/INA-1.0/INA-1.0.kicad_sch (KiCad schematic)
At the start: 10 parts, among them J1 Conn_01x04, U1 AD623, U2 MCP1501-12xSN

Commit message: deleted:    hardware/INA-1.0/#auto_saved_files# 	deleted:    hardware/INA-1.0/INA-1.0-backups/INA-1.0-2026-04-13_105232.zip 	deleted:    hardware/INA-1.0/INA-1.0-backups/INA-1.0-2026-04-13_105845.zip 	deleted:    hardware/INA-1.0/INA-1.0-backups/INA-1.0-2026-04-13_110346.zip 	deleted:    hardware/INA-1.0/INA-1.0-backups/INA-1.0-2026-04-13_112014.zip 	new file:   hardware/INA-1.0/INA-1.0-backups/INA-1.0-2026-04-13_141241.zip 	new file:   hardware/INA-1.0/INA-1.0-backups/INA-1.0-2026-04-13_161543.zip 	new file:   hardware/INA-1.0/INA-1.0-backups/INA-1.0-2026-04-13_162052.zip 	new file:   hardware/INA-1.0/INA-1.0-backups/INA-1.0-2026-04-13_162733.zip 	modified:   hardware/INA-1.0/INA-1.0.kicad_pcb 	modified:   hardware/INA-1.0/INA-1.0.kicad_pro 	modified:   hardware/INA-1.0/INA-1.0.kicad_sch 	deleted:    hardware/INA-1.0/_autosave-INA-1.0.kicad_pcb 	deleted:    hardware/INA-1.0/_autosave-INA-1.0.kicad_sch 	deleted:    hardware/INA-1.0/~INA-1.0.kicad_sch.lck 	deleted:    hardware/INA-1.0/~_autosave-INA-1.0.kicad_pcb.lck
Connections:
- net +5V: now also J1.4 (Pin_4); no longer J1.1 (Pin_1)
- net GND: now also J1.3 (Pin_3); no longer J1.2 (Pin_2)
- net INPUT: now also J1.2 (Pin_2); no longer J1.3 (Pin_3)
- net OUTPUT: now also J1.1 (Pin_1); no longer J1.4 (Pin_4)
Other:
- moved on the sheet: C1, C2, C3, R1, R2, U1

Commit message: new file:   hardware/CTL-5.0/CTL-5.0-backups/CTL-5.0-2026-04-14_112836.zip 	new file:   hardware/CTL-5.0/CTL-5.0-backups/CTL-5.0-2026-04-14_114223.zip 	deleted:    hardware/INA-1.0/INA-1.0-backups/INA-1.0-2026-04-13_112658.zip 	new file:   hardware/INA-1.0/INA-1.0-backups/INA-1.0-2026-04-14_092403.zip 	new file:   hardware/INA-1.0/INA-1.0-backups/INA-1.0-2026-04-14_112617.zip 	new file:   hardware/INA-1.0/INA-1.0-backups/INA-1.0-2026-04-15_103830.zip 	new file:   hardware/INA-1.0/INA-1.0-backups/INA-1.0-2026-04-15_105330.zip 	new file:   hardware/INA-1.0/INA-1.0-backups/INA-1.0-2026-04-15_110411.zip 	new file:   hardware/INA-1.0/INA-1.0-backups/INA-1.0-2026-04-15_111143.zip 	new file:   hardware/INA-1.0/INA-1.0-backups/INA-1.0-2026-04-15_111849.zip 	new file:   hardware/INA-1.0/INA-1.0-backups/INA-1.0-2026-04-15_113315.zip 	modified:   hardware/INA-1.0/INA-1.0.kicad_pcb 	modified:   hardware/INA-1.0/INA-1.0.kicad_pro 	modified:   hardware/INA-1.0/INA-1.0.kicad_sch 	new file:   hardware/INA-1.0/_autosave-INA-1.0.kicad_pcb 	modified:   hardware/INA-1.0/fabrication-outputs/INA-1.0-F_Cu.dxf 	modified:   hardware/INA-1.0/fabrication-outputs/INA-1.0-F_Mask.dxf 	new file:   hardware/INA-1.0/fabrication-outputs/TRACE-2.dwg 	new file:   hardware/INA-1.0/fabrication-outputs/TRACE-2.dxf 	new file:   hardware/INA-1.0/~INA-1.0.kicad_sch.lck 	new file:   hardware/INA-1.0/~_autosave-INA-1.0.kicad_pcb.lck 	new file:   hardware/PSU-1.0/CTL-4.3-backups/CTL-4.3-2026-01-19_105947.zip 	new file:   hardware/PSU-1.0/CTL-4.3-backups/CTL-4.3-2026-01-19_110601.zip 	new file:   hardware/PSU-1.0/CTL-4.3-backups/CTL-4.3-2026-01-19_111804.zip 	new file:   hardware/PSU-1.0/CTL-4.3-backups/CTL-4.3-2026-01-19_113721.zip 	new file:   hardware/PSU-1.0/CTL-4.3-backups/CTL-4.3-2026-01-19_164107.zip 	new file:   hardware/PSU-1.0/CTL-4.3-backups/CTL-4.3-2026-01-20_112913.zip 	new file:   hardware/PSU-1.0/CTL-4.3-backups/CTL-4.3-2026-02-11_163805.zip 	new file:   hardware/PSU-1.0/CTL-4.3-backups/CTL-4.3-2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
Parts:
- R1: value R -> 20kΩ
Changed lines of the file:
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@@
 			)
 		)
-		(property "Value" "R"
+		(property "Value" "20kΩ"
 			(at 93.472 80.01 0)
 			(effects
