File: hardware/INA-4.0/INA-4.0.kicad_pcb (KiCad board)
At the start: 2 copper layers, 36.8 x 38.1 mm, 18 parts, among them J1 Conn_01x05, U1 LM358, U2 LM358, U3 AMS1117-1.8

Commit message: deleted:    hardware/INA-4.0/INA-4.0-backups/INA-4.0-2026-04-23_100333.zip 	new file:   hardware/INA-4.0/INA-4.0-backups/INA-4.0-2026-04-23_155429.zip 	modified:   hardware/INA-4.0/INA-4.0.kicad_pcb 	modified:   hardware/INA-4.0/INA-4.0.kicad_prl 	modified:   hardware/INA-4.0/INA-4.0.kicad_pro 	deleted:    hardware/INA-4.0/_autosave-INA-4.0.kicad_pcb 	modified:   hardware/INA-4.0/fp-info-cache 	renamed:    hardware/INA-4.0/~INA-4.0.kicad_sch.lck -> hardware/INA-4.0/~INA-4.0.kicad_pcb.lck 	deleted:    hardware/INA-4.0/~_autosave-INA-4.0.kicad_pcb.lck
Routing:
- net +5V: track 55.1 -> 60.1 mm
Changed lines of the file:
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@@
 		(allow_soldermask_bridges_in_footprints no)
 		(pcbplotparams
-			(layerselection 0x00010fc_ffffffff)
-			(plot_on_all_layers_selection 0x0000000_00000000)
+			(layerselection 0x0000000_fffffffe)
+			(plot_on_all_layers_selection 0x0001000_00000000)
 			(disableapertmacros no)
 			(usegerberextensions no)
@@
 			(svgprecision 4)
 			(plotframeref no)
-			(viasonmask no)
+			(viasonmask yes)
 			(mode 1)
 			(useauxorigin no)
@@
 			(pdf_back_fp_property_popups yes)
 			(dxfpolygonmode yes)
-			(dxfimperialunits yes)
+			(dxfimperialunits no)
 			(dxfusepcbnewfont yes)
 			(psnegative no)
@@
 			(sketchpadsonfab no)
 			(subtractmaskfromsilk no)
-			(outputformat 1)
+			(outputformat 3)
 			(mirror no)
 			(drillshape 1)
 			(scaleselection 1)
-			(outputdirectory "")
+			(outputdirectory "fabrication-outputs/")
 		)
 	)
@@
 		(end 70.1675 82.55)
 		(stroke
-			(width 0.05)
+			(width 0)
 			(type default)
 		)
@@
 		(end 70.1675 82.55)
 		(stroke
-			(width 0.05)
+			(width 0)
 			(type default)
 		)
@@
 		(end 33.3375 82.55)
 		(stroke
-			(width 0.05)
+			(width 0)
 			(type default)
 		)
@@
 		(end 70.1675 44.45)
 		(stroke
-			(width 0.05)
+			(width 0)
 			(type default)
 		)
@@
 		(net 10)
 	)
+	(segment
+		(start 56.8325 55.245)
+		(end 61.9125 55.245)
+		(width 0.6)
+		(layer "F.Cu")
+		(net 12)
+	)
 	(via
