File: hardware/CTL-5.0/CTL-5.0.kicad_sch (KiCad schematic)
At the start: 73 parts, among them J1 Conn_02x16_Top_Bottom, J3 Conn_01x03, J4 Conn_01x03, J5 Conn_02x06_Odd_Even, J6 Conn_01x04, J7 Conn_01x04, J8 Conn_01x04, K1 G5V-1, Q1 BCX56, Q2 BCX56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

Commit message: modified:   .DS_Store 	new file:   archive/Payment 20260424.pdf 	new file:   archive/Purchase 20260424.docx 	new file:   archive/REM_OUTPUT.xlsx 	modified:   firmware/ESP32-S3 PWM/include/config.h 	modified:   firmware/ESP32-S3 PWM/src/hardware_control.cpp 	deleted:    hardware/CTL-5.0/CTL-5.0-backups/CTL-5.0-2026-02-20_154251.zip 	deleted:    hardware/CTL-5.0/CTL-5.0-backups/CTL-5.0-2026-02-20_184343.zip 	deleted:    hardware/CTL-5.0/CTL-5.0-backups/CTL-5.0-2026-02-26_100701.zip 	deleted:    hardware/CTL-5.0/CTL-5.0-backups/CTL-5.0-2026-02-26_102054.zip 	deleted:    hardware/CTL-5.0/CTL-5.0-backups/CTL-5.0-2026-02-26_102605.zip 	deleted:    hardware/CTL-5.0/CTL-5.0-backups/CTL-5.0-2026-02-26_103340.zip 	deleted:    hardware/CTL-5.0/CTL-5.0-backups/CTL-5.0-2026-02-26_153650.zip 	new file:   hardware/CTL-5.0/CTL-5.0-backups/CTL-5.0-2026-04-30_153803.zip 	new file:   hardware/CTL-5.0/CTL-5.0-backups/CTL-5.0-2026-04-30_154828.zip 	new file:   hardware/CTL-5.0/CTL-5.0-backups/CTL-5.0-2026-04-30_160225.zip 	new file:   hardware/CTL-5.0/CTL-5.0-backups/CTL-5.0-2026-04-30_161241.zip 	new file:   hardware/CTL-5.0/CTL-5.0-backups/CTL-5.0-2026-04-30_162225.zip 	new file:   hardware/CTL-5.0/CTL-5.0-backups/CTL-5.0-2026-04-30_162925.zip 	modified:   hardware/CTL-5.0/CTL-5.0.kicad_pcb 	modified:   hardware/CTL-5.0/CTL-5.0.kicad_sch 	modified:   hardware/CTL-5.0/fp-info-cache 	deleted:    hardware/INA-3.1/INA-3.1-backups/INA-3.1-2026-04-21_104126.zip 	new file:   hardware/INA-3.1/INA-3.1-backups/INA-3.1-2026-04-29_085310.zip 	new file:   hardware/INA-3.1/INA-3.1-backups/INA-3.1-2026-04-30_110843.zip 	new file:   hardware/INA-3.1/INA-3.1-backups/INA-3.1-2026-04-30_111401.zip 	new file:   hardware/INA-3.1/INA-3.1-backups/INA-3.1-2026-04-30_111913.zip 	new file:   hardware/INA-3.1/INA-3.1-backups/INA-3.1-2026-04-30_112649.zip 	new file:   hardware/INA-3.1/INA-3.1-backups/INA-3.1-2026-04-30_113258.zip 	modified:   hardware/INA-3.1/INA-3.1.kicad_pcb 	modified:   hardware/INA-3.1/INA-3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
Parts:
- removed U5: 4071, Package_SO:SOIC-14_3.9x8.7mm_P1.27mm, symbol 4xxx:4071
- added U5: 74LVC1G32, Package_TO_SOT_SMD:SOT-23-5_HandSoldering, symbol 74xGxx:74LVC1G32
- R19, R20, R3, R4: value 10k -> 1k
Connections:
- net +3.3V: now also U5.5 (VCC)
- net GND: now also U5.3 (GND)
- net PWM: now also U5.4
- net PWM.00: now also U5.1
- net PWM.01: now also U5.2
