File: hardware/CTL-5.0/CTL-5.0.kicad_pcb (KiCad board)
At the start: 2 copper layers, 198.2 x 45.1 mm, 72 parts, among them J1 Conn_02x16_Top_Bottom, J3 Conn_01x03, J4 Conn_01x03, J5 Conn_02x06_Odd_Even, J6 Conn_01x04, J7 Conn_01x04, K1 G5V-1, Q1 BCX56, Q2 BCX56, Q3 BCX56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

Commit message: modified:   .DS_Store 	new file:   archive/Payment 20260424.pdf 	new file:   archive/Purchase 20260424.docx 	new file:   archive/REM_OUTPUT.xlsx 	modified:   firmware/ESP32-S3 PWM/include/config.h 	modified:   firmware/ESP32-S3 PWM/src/hardware_control.cpp 	deleted:    hardware/CTL-5.0/CTL-5.0-backups/CTL-5.0-2026-02-20_154251.zip 	deleted:    hardware/CTL-5.0/CTL-5.0-backups/CTL-5.0-2026-02-20_184343.zip 	deleted:    hardware/CTL-5.0/CTL-5.0-backups/CTL-5.0-2026-02-26_100701.zip 	deleted:    hardware/CTL-5.0/CTL-5.0-backups/CTL-5.0-2026-02-26_102054.zip 	deleted:    hardware/CTL-5.0/CTL-5.0-backups/CTL-5.0-2026-02-26_102605.zip 	deleted:    hardware/CTL-5.0/CTL-5.0-backups/CTL-5.0-2026-02-26_103340.zip 	deleted:    hardware/CTL-5.0/CTL-5.0-backups/CTL-5.0-2026-02-26_153650.zip 	new file:   hardware/CTL-5.0/CTL-5.0-backups/CTL-5.0-2026-04-30_153803.zip 	new file:   hardware/CTL-5.0/CTL-5.0-backups/CTL-5.0-2026-04-30_154828.zip 	new file:   hardware/CTL-5.0/CTL-5.0-backups/CTL-5.0-2026-04-30_160225.zip 	new file:   hardware/CTL-5.0/CTL-5.0-backups/CTL-5.0-2026-04-30_161241.zip 	new file:   hardware/CTL-5.0/CTL-5.0-backups/CTL-5.0-2026-04-30_162225.zip 	new file:   hardware/CTL-5.0/CTL-5.0-backups/CTL-5.0-2026-04-30_162925.zip 	modified:   hardware/CTL-5.0/CTL-5.0.kicad_pcb 	modified:   hardware/CTL-5.0/CTL-5.0.kicad_sch 	modified:   hardware/CTL-5.0/fp-info-cache 	deleted:    hardware/INA-3.1/INA-3.1-backups/INA-3.1-2026-04-21_104126.zip 	new file:   hardware/INA-3.1/INA-3.1-backups/INA-3.1-2026-04-29_085310.zip 	new file:   hardware/INA-3.1/INA-3.1-backups/INA-3.1-2026-04-30_110843.zip 	new file:   hardware/INA-3.1/INA-3.1-backups/INA-3.1-2026-04-30_111401.zip 	new file:   hardware/INA-3.1/INA-3.1-backups/INA-3.1-2026-04-30_111913.zip 	new file:   hardware/INA-3.1/INA-3.1-backups/INA-3.1-2026-04-30_112649.zip 	new file:   hardware/INA-3.1/INA-3.1-backups/INA-3.1-2026-04-30_113258.zip 	modified:   hardware/INA-3.1/INA-3.1.kicad_pcb 	modified:   hardware/INA-3.1/INA-3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
Parts:
- R19, R20, R3, R4: value 10k -> 1k
- U5: value 4071 -> 74LVC1G32; footprint Package_SO:SOIC-14_3.9x8.7mm_P1.27mm -> Package_TO_SOT_SMD:SOT-23-5_HandSoldering
- moved U5 6.13 mm to (100.0, 29.4), turned to -90 degrees
- moved C7 1.37 mm to (89.4, 52.2)
- moved C8 1.37 mm to (79.5, 52.2)
- moved Q1 1.11 mm to (79.2, 48.3)
- moved Q2 1.11 mm to (89.7, 48.3)
- moved SW1 0.90 mm to (96.5, 48.3)
- moved SW2 0.90 mm to (72.4, 48.3)
Connections:
- U5 pad 3: /PWM -> GND
- U5 pad 4: (no net) -> /PWM
- U5 pad 5: (no net) -> +3.3V
Routing:
- net +3.3V: track 213.4 -> 180.1 mm, vias 5 -> 6
- net /IO.00: track 33.2 -> 12.9 mm
- net /EN: track 54.6 -> 34.2 mm
- net /DTR: track 59.2 -> 52.7 mm
- net /PWM: track 76.2 -> 71.7 mm
- net /PWM.01: track 27.6 -> 23.7 mm
- net /PWM.00: track 27.3 -> 25.7 mm
- net Net-(Q2-B): track 3.25 -> 1.83 mm
- net Net-(Q1-B): track 2.70 -> 1.83 mm
- net /RTS: track 55.0 -> 54.3 mm

Commit message: modified:   .DS_Store 	modified:   firmware/ESP32-S3 PWM/src/hardware_control.cpp 	deleted:    hardware/CTL-5.0/CTL-4.3-backups/CTL-4.3-2026-01-19_105947.zip 	deleted:    hardware/CTL-5.0/CTL-4.3-backups/CTL-4.3-2026-01-19_110601.zip 	deleted:    hardware/CTL-5.0/CTL-4.3-backups/CTL-4.3-2026-01-19_111804.zip 	deleted:    hardware/CTL-5.0/CTL-4.3-backups/CTL-4.3-2026-01-19_113721.zip 	deleted:    hardware/CTL-5.0/CTL-4.3-backups/CTL-4.3-2026-01-19_164107.zip 	deleted:    hardware/CTL-5.0/CTL-4.3-backups/CTL-4.3-2026-01-20_112913.zip 	deleted:    hardware/CTL-5.0/CTL-4.3-backups/CTL-4.3-2026-02-11_163805.zip 	deleted:    hardware/CTL-5.0/CTL-4.3-backups/CTL-4.3-2026-02-13_145455.zip 	deleted:    hardware/CTL-5.0/CTL-4.3-backups/CTL-4.3-2026-02-13_163249.zip 	deleted:    hardware/CTL-5.0/CTL-4.3-backups/CTL-4.3-2026-02-18_163417.zip 	deleted:    hardware/CTL-5.0/CTL-4.zip 	deleted:    hardware/CTL-5.0/CTL-5.0-backups/CTL-5.0-2026-02-27_095759.zip 	deleted:    hardware/CTL-5.0/CTL-5.0-backups/CTL-5.0-2026-02-27_101209.zip 	deleted:    hardware/CTL-5.0/CTL-5.0-backups/CTL-5.0-2026-03-02_113302.zip 	deleted:    hardware/CTL-5.0/CTL-5.0-backups/CTL-5.0-2026-04-30_153803.zip 	deleted:    hardware/CTL-5.0/CTL-5.0-backups/CTL-5.0-2026-04-30_154828.zip 	new file:   hardware/CTL-5.0/CTL-5.0-backups/CTL-5.0-2026-04-30_163534.zip 	new file:   hardware/CTL-5.0/CTL-5.0-backups/CTL-5.0-2026-05-01_164305.zip 	new file:   hardware/CTL-5.0/CTL-5.0-backups/CTL-5.0-2026-05-04_084718.zip 	new file:   hardware/CTL-5.0/CTL-5.0-backups/CTL-5.0-2026-05-04_085459.zip 	new file:   hardware/CTL-5.0/CTL-5.0-backups/CTL-5.0-2026-05-04_090501.zip 	new file:   hardware/CTL-5.0/CTL-5.0-backups/CTL-5.0-2026-05-04_091505.zip 	modified:   hardware/CTL-5.0/CTL-5.0.kicad_pcb 	modified:   hardware/CTL-5.0/CTL-5.0.kicad_prl 	new file:   hardware/CTL-6.0/CTL-6.0-backups/CTL-6.0-2026-05-04_160013.zip 	new file:   hardware/CTL-6.0/CTL-6.0-backups/CTL-6.0-2026-05-04_160854.zip 	new file:   hardware/CTL-6.0/CTL-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
Parts:
- moved C7 57.3 mm to (121.1, 99.9)
- moved C8 57.3 mm to (111.3, 99.9)
- moved C14 57.2 mm to (144.1, 89.5)
- moved C15 57.2 mm to (144.1, 84.5)
- moved D4 57.2 mm to (151.9, 95.1)
- moved J6 57.2 mm to (134.0, 63.5)
- moved J7 57.2 mm to (134.0, 68.3)
- moved SW1 57.2 mm to (128.3, 95.9)
- moved C1 57.2 mm to (154.9, 89.5)
- moved C10 57.2 mm to (101.4, 62.9)
- moved C12 57.2 mm to (100.3, 85.1)
- moved C2 57.2 mm to (154.9, 84.5)
- moved C3 57.2 mm to (180.0, 67.6)
- moved C5 57.2 mm to (212.4, 67.6)
- moved D2 57.2 mm to (181.9, 75.2)
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Routing:
- net /EN: track 34.2 -> 55.0 mm
- net /IO.00: track 12.9 -> 33.5 mm
- net /DTR: track 52.7 -> 64.5 mm, vias 2 -> 0
- net /RTS: track 54.3 -> 54.8 mm, vias 1 -> 0
- net GND: vias 181 -> 183
- net +36V: vias 10 -> 11
