File: hardware/INA-3.1/INA-3.1.kicad_pcb (KiCad board)
At the start: 2 copper layers, 28.4 x 24.4 mm, 20 parts, among them J1 Conn_01x05, U1 OPA365, U2 OPA365, U3 OPA365, U4 AMS1117-1.8

Commit message: modified:   .DS_Store 	new file:   archive/Payment 20260424.pdf 	new file:   archive/Purchase 20260424.docx 	new file:   archive/REM_OUTPUT.xlsx 	modified:   firmware/ESP32-S3 PWM/include/config.h 	modified:   firmware/ESP32-S3 PWM/src/hardware_control.cpp 	deleted:    hardware/CTL-5.0/CTL-5.0-backups/CTL-5.0-2026-02-20_154251.zip 	deleted:    hardware/CTL-5.0/CTL-5.0-backups/CTL-5.0-2026-02-20_184343.zip 	deleted:    hardware/CTL-5.0/CTL-5.0-backups/CTL-5.0-2026-02-26_100701.zip 	deleted:    hardware/CTL-5.0/CTL-5.0-backups/CTL-5.0-2026-02-26_102054.zip 	deleted:    hardware/CTL-5.0/CTL-5.0-backups/CTL-5.0-2026-02-26_102605.zip 	deleted:    hardware/CTL-5.0/CTL-5.0-backups/CTL-5.0-2026-02-26_103340.zip 	deleted:    hardware/CTL-5.0/CTL-5.0-backups/CTL-5.0-2026-02-26_153650.zip 	new file:   hardware/CTL-5.0/CTL-5.0-backups/CTL-5.0-2026-04-30_153803.zip 	new file:   hardware/CTL-5.0/CTL-5.0-backups/CTL-5.0-2026-04-30_154828.zip 	new file:   hardware/CTL-5.0/CTL-5.0-backups/CTL-5.0-2026-04-30_160225.zip 	new file:   hardware/CTL-5.0/CTL-5.0-backups/CTL-5.0-2026-04-30_161241.zip 	new file:   hardware/CTL-5.0/CTL-5.0-backups/CTL-5.0-2026-04-30_162225.zip 	new file:   hardware/CTL-5.0/CTL-5.0-backups/CTL-5.0-2026-04-30_162925.zip 	modified:   hardware/CTL-5.0/CTL-5.0.kicad_pcb 	modified:   hardware/CTL-5.0/CTL-5.0.kicad_sch 	modified:   hardware/CTL-5.0/fp-info-cache 	deleted:    hardware/INA-3.1/INA-3.1-backups/INA-3.1-2026-04-21_104126.zip 	new file:   hardware/INA-3.1/INA-3.1-backups/INA-3.1-2026-04-29_085310.zip 	new file:   hardware/INA-3.1/INA-3.1-backups/INA-3.1-2026-04-30_110843.zip 	new file:   hardware/INA-3.1/INA-3.1-backups/INA-3.1-2026-04-30_111401.zip 	new file:   hardware/INA-3.1/INA-3.1-backups/INA-3.1-2026-04-30_111913.zip 	new file:   hardware/INA-3.1/INA-3.1-backups/INA-3.1-2026-04-30_112649.zip 	new file:   hardware/INA-3.1/INA-3.1-backups/INA-3.1-2026-04-30_113258.zip 	modified:   hardware/INA-3.1/INA-3.1.kicad_pcb 	modified:   hardware/INA-3.1/INA-3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
Parts:
- added C8: 100nF, Capacitor_SMD:C_0805_2012Metric_Pad1.18x1.45mm_HandSolder, F.Cu at (119.1, 54.1)
- added R9: 10kΩ, Resistor_SMD:R_0805_2012Metric_Pad1.20x1.40mm_HandSolder, F.Cu at (117.2, 54.1)
- R1: value 6.8kΩ -> 5.1kΩ
Connections:
- R6 pad 2: /OUT -> Net-(R6-Pad2)
- U3 pad 1: /OUT -> Net-(R6-Pad2)
Routing:
- net /OUT: track 16.5 -> 0.48 mm
- net Net-(R6-Pad2): track 0.00 -> 12.1 mm
- net /IN: track 18.0 -> 20.6 mm
- net 1V8: track 11.4 -> 9.05 mm
- added copper zone on F.Cu, net /OUT
