File: hardware/INA-3.1/INA-3.1.kicad_sch (KiCad schematic)
At the start: 20 parts, among them J1 Conn_01x05, U1 OPA365, U2 OPA365, U3 OPA365, U4 AMS1117-1.8

Commit message: modified:   .DS_Store 	new file:   hardware/INA-3.1/INA-3-backups/INA-3-2026-04-16_161548.zip 	new file:   hardware/INA-3.1/INA-3-backups/INA-3-2026-04-16_162307.zip 	new file:   hardware/INA-3.1/INA-3-backups/INA-3-2026-04-16_163207.zip 	new file:   hardware/INA-3.1/INA-3-backups/INA-3-2026-04-17_160528.zip 	new file:   hardware/INA-3.1/INA-3-backups/INA-3-2026-04-17_161450.zip 	new file:   hardware/INA-3.1/INA-3-backups/INA-3-2026-04-17_162010.zip 	new file:   hardware/INA-3.1/INA-3-backups/INA-3-2026-04-17_162549.zip 	new file:   hardware/INA-3.1/INA-3-backups/INA-3-2026-04-17_163140.zip 	renamed:    hardware/INA-3/INA-3-backups/INA-3-2026-04-20_085258.zip -> hardware/INA-3.1/INA-3-backups/INA-3-2026-04-20_085258.zip 	new file:   hardware/INA-3.1/INA-3-backups/INA-3-2026-04-20_085822.zip 	new file:   hardware/INA-3.1/INA-3-backups/INA-3-2026-04-20_090419.zip 	new file:   hardware/INA-3.1/INA-3-backups/INA-3-2026-04-20_091140.zip 	new file:   hardware/INA-3.1/INA-3-backups/INA-3-2026-04-20_092653.zip 	new file:   hardware/INA-3.1/INA-3-backups/INA-3-2026-04-20_144439.zip 	new file:   hardware/INA-3.1/INA-3.1-backups/INA-3.1-2026-04-20_160434.zip 	new file:   hardware/INA-3.1/INA-3.1-backups/INA-3.1-2026-04-20_161047.zip 	new file:   hardware/INA-3.1/INA-3.1-backups/INA-3.1-2026-04-20_161551.zip 	new file:   hardware/INA-3.1/INA-3.1-backups/INA-3.1-2026-04-20_162147.zip 	new file:   hardware/INA-3.1/INA-3.1-backups/INA-3.1-2026-04-20_163149.zip 	new file:   hardware/INA-3.1/INA-3.1-backups/INA-3.1-2026-04-21_104126.zip 	new file:   hardware/INA-3.1/INA-3.1-backups/INA-3.1-2026-04-21_105025.zip 	new file:   hardware/INA-3.1/INA-3.1-backups/INA-3.1-2026-04-21_105750.zip 	new file:   hardware/INA-3.1/INA-3.1-backups/INA-3.1-2026-04-21_110437.zip 	new file:   hardware/INA-3.1/INA-3.1-backups/INA-3.1-2026-04-21_143841.zip 	new file:   hardware/INA-3.1/INA-3.1-backups/INA-3.1-2026-04-21_154136.zip 	renamed:    hardware/INA-3/_autosave-INA-3.kicad_pcb -> hardware/INA-3.1/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
Parts:
- C7: value 100nF -> 470pF
Connections:
- net GND: no longer J1.2 (Pin_2)
- net IN: now also J1.2 (Pin_2); no longer J1.3 (Pin_3)
- net 1V8: now reaches C5.1, C6.1, U1.3 (+), U4.2 (VO)
Changed lines of the file:
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@@
-	)
-	(junction
-		(at 31.75 140.97)
-		(diameter 0)
-		(color 0 0 0 0)
 	)
 	(junction
@@
 	(wire
 		(pts
-			(xy 29.21 140.97) (xy 31.75 140.97)
-		)
-		(stroke
-			(width 0)
-			(type default)
-		)
-	)
-	(wire
-		(pts
 			(xy 45.72 40.64) (xy 45.72 43.18)
 		)
@@
 	(wire
 		(pts
+			(xy 55.88 38.1) (xy 55.88 40.64)
+		)
+		(stroke
+			(width 0)
+			(type default)
+		)
+	)
+	(wire
+		(pts
 			(xy 63.5 142.24) (xy 63.5 139.7)
 		)
@@
 	(wire
 		(pts
-			(xy 31.75 135.89) (xy 31.75 140.97)
-		)
-		(stroke
-			(width 0)
-			(type default)
-		)
-	)
-	(wire
-		(pts
 			(xy 66.04 45.72) (xy 66.04 49.53)
 		)
@@
 	(wire
 		(pts
-			(xy 31.75 140.97) (xy 31.75 146.05)
+			(xy 31.75 135.89) (xy 31.75 146.05)
 		)
 		(stroke
@@
 	(wire
 		(pts
-			(xy 29.21 138.43) (xy 39.37 138.43)
+			(xy 29.21 140.97) (xy 39.37 140.97)
 		)
 		(stroke
@@
 		)
 	)
-	(label "OUT"
-		(at 121.92 55.88 0)
+	(label "IN"
+		(at 35.56 140.97 0)
 		(fields_autoplaced yes)
 		(effects
@@
 		)
 	)
-	(label "IN"
-		(at 35.56 138.43 0)
+	(label "OUT"
+		(at 121.92 55.88 0)
 		(fields_autoplaced yes)
 		(effects
@@
 	)
 	(symbol
+		(lib_id "power:+5V")
+		(at 55.88 38.1 0)
+		(unit 1)
+		(exclude_from_sim no)
+		(in_bom yes)
+		(on_board yes)
+		(dnp no)
+		(property "Reference" "#PWR09"
+			(at 55.88 41.91 0)
+			(effects
+				(font
+					(size 1.27 1.27)
+				)
+				(hide yes)
+			)
+		)
+		(property "Value" "1V8"
+			(at 55.88 34.544 0)
+			(effects
+				(font
+					(size 1 1)
+				)
+			)
+		)
+		(property "Footprint" ""
+			(at 55.88 38.1 0)
+			(effects
+				(font
+					(size 1.27 1.27)
+				)
+				(hide yes)
+			)
+		)
+		(property "Datasheet" ""
+			(at 55.88 38.1 0)
+			(effects
+				(font
+					(size 1.27 1.27)
+				)
+				(hide yes)
+			)
+		)
+		(property "Description" "Power symbol creates a global label with name \"+5V\""
+			(at 55.88 38.1 0)
+			(effects
+				(font
+					(size 1.27 1.27)
+				)
+				(hide yes)
+			)
+		)
+		(pin "1"
+		)
+		(instances
+			(project "INA-3.1"
+				(path "/012ecf8f-e59d-4b86-a3cc-27fec600e7df"
+					(reference "#PWR09")
+					(unit 1)
+				)
+			)
+		)
+	)
+	(symbol
 		(lib_id "Amplifier_Operational:OPA365xxDBV")
 		(at 76.2 68.58 0)
@@
 			)
 		)
-		(property "Value" "100nF"
+		(property "Value" "470pF"
 			(at 56.134 79.502 0)
 			(effects

Commit message: modified:   .DS_Store 	new file:   archive/Payment 20260424.pdf 	new file:   archive/Purchase 20260424.docx 	new file:   archive/REM_OUTPUT.xlsx 	modified:   firmware/ESP32-S3 PWM/include/config.h 	modified:   firmware/ESP32-S3 PWM/src/hardware_control.cpp 	deleted:    hardware/CTL-5.0/CTL-5.0-backups/CTL-5.0-2026-02-20_154251.zip 	deleted:    hardware/CTL-5.0/CTL-5.0-backups/CTL-5.0-2026-02-20_184343.zip 	deleted:    hardware/CTL-5.0/CTL-5.0-backups/CTL-5.0-2026-02-26_100701.zip 	deleted:    hardware/CTL-5.0/CTL-5.0-backups/CTL-5.0-2026-02-26_102054.zip 	deleted:    hardware/CTL-5.0/CTL-5.0-backups/CTL-5.0-2026-02-26_102605.zip 	deleted:    hardware/CTL-5.0/CTL-5.0-backups/CTL-5.0-2026-02-26_103340.zip 	deleted:    hardware/CTL-5.0/CTL-5.0-backups/CTL-5.0-2026-02-26_153650.zip 	new file:   hardware/CTL-5.0/CTL-5.0-backups/CTL-5.0-2026-04-30_153803.zip 	new file:   hardware/CTL-5.0/CTL-5.0-backups/CTL-5.0-2026-04-30_154828.zip 	new file:   hardware/CTL-5.0/CTL-5.0-backups/CTL-5.0-2026-04-30_160225.zip 	new file:   hardware/CTL-5.0/CTL-5.0-backups/CTL-5.0-2026-04-30_161241.zip 	new file:   hardware/CTL-5.0/CTL-5.0-backups/CTL-5.0-2026-04-30_162225.zip 	new file:   hardware/CTL-5.0/CTL-5.0-backups/CTL-5.0-2026-04-30_162925.zip 	modified:   hardware/CTL-5.0/CTL-5.0.kicad_pcb 	modified:   hardware/CTL-5.0/CTL-5.0.kicad_sch 	modified:   hardware/CTL-5.0/fp-info-cache 	deleted:    hardware/INA-3.1/INA-3.1-backups/INA-3.1-2026-04-21_104126.zip 	new file:   hardware/INA-3.1/INA-3.1-backups/INA-3.1-2026-04-29_085310.zip 	new file:   hardware/INA-3.1/INA-3.1-backups/INA-3.1-2026-04-30_110843.zip 	new file:   hardware/INA-3.1/INA-3.1-backups/INA-3.1-2026-04-30_111401.zip 	new file:   hardware/INA-3.1/INA-3.1-backups/INA-3.1-2026-04-30_111913.zip 	new file:   hardware/INA-3.1/INA-3.1-backups/INA-3.1-2026-04-30_112649.zip 	new file:   hardware/INA-3.1/INA-3.1-backups/INA-3.1-2026-04-30_113258.zip 	modified:   hardware/INA-3.1/INA-3.1.kicad_pcb 	modified:   hardware/INA-3.1/INA-3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
Parts:
- added C8: 100nF, Capacitor_SMD:C_0805_2012Metric_Pad1.18x1.45mm_HandSolder, symbol Device:C
- added R9: 10kΩ, Resistor_SMD:R_0805_2012Metric_Pad1.20x1.40mm_HandSolder, symbol Device:R
- R1: value 6.8kΩ -> 5.1kΩ
Connections:
- net GND: now also C8.2
- net OUT: now also C8.1, R9.2; no longer R6.2, U3.1
- new net: R6.2, R9.1, U3.1
Changed lines of the file:
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@@
+	)
+	(junction
+		(at 132.08 55.88)
+		(diameter 0)
+		(color 0 0 0 0)
 	)
 	(junction
@@
 	(wire
 		(pts
-			(xy 119.38 55.88) (xy 127 55.88)
+			(xy 119.38 55.88) (xy 121.92 55.88)
 		)
 		(stroke
@@
 	(wire
 		(pts
+			(xy 129.54 55.88) (xy 132.08 55.88)
+		)
+		(stroke
+			(width 0)
+			(type default)
+		)
+	)
+	(wire
+		(pts
 			(xy 29.21 143.51) (xy 39.37 143.51)
 		)
@@
 	(wire
 		(pts
+			(xy 132.08 55.88) (xy 132.08 58.42)
+		)
+		(stroke
+			(width 0)
+			(type default)
+		)
+	)
+	(wire
+		(pts
 			(xy 68.58 45.72) (xy 66.04 45.72)
 		)
@@
 	(wire
 		(pts
+			(xy 132.08 55.88) (xy 139.7 55.88)
+		)
+		(stroke
+			(width 0)
+			(type default)
+		)
+	)
+	(wire
+		(pts
 			(xy 68.58 124.46) (xy 63.5 124.46)
 		)
@@
 			(width 0)
 			(type default)
+		)
+	)
+	(label "OUT"
+		(at 138.43 55.88 180)
+		(fields_autoplaced yes)
+		(effects
+			(font
+				(size 1 1)
+			)
+			(justify right bottom)
 		)
 	)
@@
 		)
 	)
-	(label "OUT"
-		(at 121.92 55.88 0)
-		(fields_autoplaced yes)
-		(effects
-			(font
-				(size 1 1)
-			)
-			(justify left bottom)
-		)
-	)
 	(label "IN"
 		(at 36.83 71.12 0)
@@
 			)
 		)
-		(property "Value" "6.8kΩ"
+		(property "Value" "5.1kΩ"
 			(at 67.818 56.896 0)
 			(effects
@@
 	)
 	(symbol
+		(lib_id "Device:R")
+		(at 125.73 55.88 90)
+		(unit 1)
+		(exclude_from_sim no)
+		(in_bom yes)
+		(on_board yes)
+		(dnp no)
+		(property "Reference" "R9"
+			(at 125.73 53.594 90)
+			(effects
+				(font
+					(size 1 1)
+				)
+			)
+		)
+		(property "Value" "10kΩ"
+			(at 125.73 58.166 90)
+			(effects
+				(font
+					(size 1 1)
+				)
+			)
+		)
+		(property "Footprint" "Resistor_SMD:R_0805_2012Metric_Pad1.20x1.40mm_HandSolder"
+			(at 125.73 57.658 90)
+			(effects
+				(font
+					(size 1.27 1.27)
+				)
+				(hide yes)
+			)
+		)
+		(property "Datasheet" "~"
+			(at 125.73 55.88 0)
+			(effects
+				(font
+					(size 1.27 1.27)
+				)
+				(hide yes)
+			)
+		)
+		(property "Description" "Resistor"
+			(at 125.73 55.88 0)
+			(effects
+				(font
+					(size 1.27 1.27)
+				)
+				(hide yes)
+			)
+		)
+		(pin "2"
+		)
+		(pin "1"
+		)
+		(instances
+			(project "INA-3.1"
+				(path "/012ecf8f-e59d-4b86-a3cc-27fec600e7df"
+					(reference "R9")
+					(unit 1)
+				)
+			)
+		)
+	)
+	(symbol
+		(lib_id "Device:C")
+		(at 132.08 62.23 0)
+		(unit 1)
+		(exclude_from_sim no)
+		(in_bom yes)
+		(on_board yes)
+		(dnp no)
+		(property "Reference" "C8"
+			(at 132.334 60.198 0)
+			(effects
+				(font
+					(size 1 1)
+				)
+				(justify left)
+			)
+		)
+		(property "Value" "100nF"
+			(at 132.334 64.262 0)
+			(effects
+				(font
+					(size 1 1)
+				)
+				(justify left)
+			)
+		)
+		(property "Footprint" "Capacitor_SMD:C_0805_2012Metric_Pad1.18x1.45mm_HandSolder"
+			(at 133.0452 66.04 0)
+			(effects
+				(font
+					(size 1.27 1.27)
+				)
+				(hide yes)
+			)
+		)
+		(property "Datasheet" "~"
+			(at 132.08 62.23 0)
+			(effects
+				(font
+					(size 1.27 1.27)
+				)
+				(hide yes)
+			)
+		)
+		(property "Description" "Unpolarized capacitor"
+			(at 132.08 62.23 0)
+			(effects
+				(font
+					(size 1.27 1.27)
+				)
+				(hide yes)
+			)
+		)
+		(pin "1"
+		)
+		(pin "2"
+		)
+		(instances
+			(project "INA-3.1"
+				(path "/012ecf8f-e59d-4b86-a3cc-27fec600e7df"
+					(reference "C8")
+					(unit 1)
+				)
+			)
+		)
+	)
+	(symbol
 		(lib_id "power:+5V")
 		(at 55.88 38.1 0)
@@
 					(unit 1)
 				)
+			)
+		)
+	)
+	(symbol
+		(lib_id "power:GND")
+		(at 132.08 66.04 0)
+		(unit 1)
+		(exclude_from_sim no)
+		(in_bom yes)
+		(on_board yes)
+		(dnp no)
+		(fields_autoplaced yes)
+		(property "Reference" "#PWR010"
+			(at 132.08 72.39 0)
+			(effects
+				(font
+					(size 1.27 1.27)
+				)
+				(hide yes)
+			)
+		)
+		(property "Value" "GND"
+			(at 132.08 71.12 0)
+			(effects
+				(font
+					(size 1.27 1.27)
+				)
+				(hide yes)
+			)
+		)
+		(property "Footprint" ""
+			(at 132.08 66.04 0)
+			(effects
+				(font
+					(size 1.27 1.27)
+				)
+				(hide yes)
+			)
+		)
+		(property "Datasheet" ""
+			(at 132.08 66.04 0)
+			(effects
+				(font
+					(size 1.27 1.27)
+				)
+				(hide yes)
+			)
+		)
+		(property "Description" "Power symbol creates a global label with name \"GND\" , ground"
+			(at 132.08 66.04 0)
+			(effects
+				(font
+					(size 1.27 1.27)
+				)
+				(hide yes)
+			)
+		)
+		(pin "1"
+		)
+		(instances
+			(project "INA-3.1"
+				(path "/012ecf8f-e59d-4b86-a3cc-27fec600e7df"
+					(reference "#PWR010")
+					(unit 1)
+				)
