File: hardware/REM-5.0/_autosave-REM-5.0.kicad_pcb (KiCad board)
At the start: 2 copper layers, 98.4 x 44.5 mm, 35 parts, among them J1 PinHeader_2.54mm 02x04 Horizo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, J2 PinHeader_2.54mm 02x05 Horizo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, Q1 IRLB3034PbF, Q2 BCX56, Q3 BCX53, U2 74LVC1G14

Commit message: new file:   hardware/INA-3.1/INA-3.1-backups/INA-3.1-2026-06-03_154006.zip 	new file:   hardware/INA-3/INA-3-backups/INA-3-2026-06-03_161017.zip 	new file:   hardware/INA-3/INA-3-backups/INA-3-2026-06-03_161951.zip 	new file:   hardware/INA-4.0/INA-4.0-backups/INA-4.0-2026-06-03_153924.zip 	deleted:    hardware/REM-5.0/REM-5.0-backups/REM-5.0-2026-05-13_154048.zip 	deleted:    hardware/REM-5.0/REM-5.0-backups/REM-5.0-2026-05-13_155631.zip 	deleted:    hardware/REM-5.0/REM-5.0-backups/REM-5.0-2026-05-13_161956.zip 	deleted:    hardware/REM-5.0/REM-5.0-backups/REM-5.0-2026-05-13_162957.zip 	deleted:    hardware/REM-5.0/REM-5.0-backups/REM-5.0-2026-05-18_092511.zip 	deleted:    hardware/REM-5.0/REM-5.0-backups/REM-5.0-2026-05-18_093513.zip 	new file:   hardware/REM-5.0/REM-5.0-backups/REM-5.0-2026-06-04_102738.zip 	new file:   hardware/REM-5.0/REM-5.0-backups/REM-5.0-2026-06-04_103505.zip 	new file:   hardware/REM-5.0/REM-5.0-backups/REM-5.0-2026-06-04_104754.zip 	new file:   hardware/REM-5.0/REM-5.0-backups/REM-5.0-2026-06-04_164037.zip 	new file:   hardware/REM-5.0/REM-5.0-backups/REM-5.0-2026-06-05_111411.zip 	new file:   hardware/REM-5.0/REM-5.0-backups/REM-5.0-2026-06-05_115032.zip 	modified:   hardware/REM-5.0/REM-5.0.kicad_pcb 	modified:   hardware/REM-5.0/REM-5.0.kicad_prl 	modified:   hardware/REM-5.0/REM-5.0.kicad_sch 	new file:   hardware/REM-5.0/SHIELD.dxf 	new file:   hardware/REM-5.0/_autosave-REM-5.0.kicad_pcb 	new file:   hardware/REM-5.0/~REM-5.0.kicad_sch.lck 	new file:   hardware/REM-5.0/~_autosave-REM-5.0.kicad_pcb.lck
Changed lines of the file:
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@@
 		)
+	)
+	(gr_line
+		(start 107.6325 107.95)
+		(end 107.6325 111.91875)
+		(stroke
+			(width 0.1)
+			(type default)
+		)
+		(layer "F.SilkS")
+	)
+	(gr_line
+		(start 107.6325 111.91875)
+		(end 96.8375 111.91875)
+		(stroke
+			(width 0.1)
+			(type default)
+		)
+		(layer "F.SilkS")
+	)
+	(gr_line
+		(start 107.315 107.95)
+		(end 107.6325 107.95)
+		(stroke
+			(width 0.1)
+			(type default)
+		)
+		(layer "F.SilkS")
 	)
 	(gr_circle
