File: hardware/REM-5.0/REM-5.0.kicad_pcb (KiCad board)
At the start: 2 copper layers, 98.4 x 44.5 mm, 35 parts, among them J1 PinHeader_2.54mm 02x04 Horizo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, J2 PinHeader_2.54mm 02x05 Horizo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, Q1 IRLB3034PbF, Q2 BCX56, Q3 BCX53, U2 74LVC1G14

Commit message: deleted:    hardware/CTL-6.0/CTL-6.0-backups/CTL-6.0-2026-05-05_105851.zip 	new file:   hardware/CTL-6.0/CTL-6.0-backups/CTL-6.0-2026-05-21_155839.zip 	modified:   hardware/CTL-6.0/CTL-6.0.kicad_pcb 	new file:   hardware/CTL-6.1/CTL-6.0-backups/CTL-6.0-2026-05-04_160013.zip 	new file:   hardware/CTL-6.1/CTL-6.0-backups/CTL-6.0-2026-05-04_160854.zip 	new file:   hardware/CTL-6.1/CTL-6.0-backups/CTL-6.0-2026-05-04_161354.zip 	new file:   hardware/CTL-6.1/CTL-6.0-backups/CTL-6.0-2026-05-04_161937.zip 	new file:   hardware/CTL-6.1/CTL-6.0-backups/CTL-6.0-2026-05-04_162757.zip 	new file:   hardware/CTL-6.1/CTL-6.0-backups/CTL-6.0-2026-05-05_110550.zip 	new file:   hardware/CTL-6.1/CTL-6.0-backups/CTL-6.0-2026-05-05_111755.zip 	new file:   hardware/CTL-6.1/CTL-6.0-backups/CTL-6.0-2026-05-05_114939.zip 	new file:   hardware/CTL-6.1/CTL-6.0-backups/CTL-6.0-2026-05-05_155039.zip 	new file:   hardware/CTL-6.1/CTL-6.0-backups/CTL-6.0-2026-05-05_204356.zip 	new file:   hardware/CTL-6.1/CTL-6.0-backups/CTL-6.0-2026-05-21_155839.zip 	new file:   hardware/CTL-6.1/CTL-6.1-backups/CTL-6.1-2026-05-21_160708.zip 	new file:   hardware/CTL-6.1/CTL-6.1-backups/CTL-6.1-2026-05-21_163235.zip 	new file:   hardware/CTL-6.1/CTL-6.1.FCStd 	new file:   hardware/CTL-6.1/CTL-6.1.iges 	new file:   hardware/CTL-6.1/CTL-6.1.kicad_pcb 	new file:   hardware/CTL-6.1/CTL-6.1.kicad_prl 	new file:   hardware/CTL-6.1/CTL-6.1.kicad_pro 	new file:   hardware/CTL-6.1/CTL-6.1.kicad_sch 	new file:   hardware/CTL-6.1/CTL-6.1.png 	new file:   hardware/CTL-6.1/CTL-6.1.step 	new file:   hardware/CTL-6.1/CTL-6.1.xlsx 	new file:   hardware/CTL-6.1/bom/ibom.html 	new file:   hardware/CTL-6.1/fabrication-output/CTL-4.3-B_Cu.pdf 	new file:   hardware/CTL-6.1/fabrication-output/CTL-4.3-B_Mask.pdf 	new file:   hardware/CTL-6.1/fabrication-output/CTL-4.3-B_Paste.pdf 	new file:   hardware/CTL-6.1/fabrication-output/CTL-4.3-B_Silkscreen.pdf 	new file:   hardware/CTL-6.1/fabrication-output/CTL-4.3-Edge_Cuts.pdf 	new file:   h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
Parts:
- R1, R2, R6, R7: value 1kΩ -> ~
Routing:
- net Net-(Q1-D): track 23.1 -> 25.9 mm
Changed lines of the file:
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@@
 			)
 		)
-		(property "Value" "1kΩ"
+		(property "Value" "~"
 			(at 0 1.65 0)
 			(layer "F.Fab")
@@
 		(pad "1" thru_hole circle
 			(at -5.079999 0 90)
-			(size 3.81 3.81)
-			(drill 2)
+			(size 1.905 3.81)
+			(drill 1)
 			(layers "*.Cu" "*.Mask")
 			(remove_unused_layers no)
@@
 		(pad "2" thru_hole circle
 			(at 5.079999 0 90)
-			(size 3.81 3.81)
-			(drill 2)
+			(size 1.905 3.81)
+			(drill 1)
 			(layers "*.Cu" "*.Mask")
 			(remove_unused_layers no)
@@
 			)
 		)
-		(property "Value" "1kΩ"
+		(property "Value" "~"
 			(at 0 1.65 0)
 			(layer "F.Fab")
@@
 			)
 		)
-		(property "Value" "1kΩ"
+		(property "Value" "~"
 			(at 0 1.65 0)
 			(layer "F.Fab")
@@
 		(tags "Potentiometer vertical Bourns 3296W")
 		(property "Reference" "RV1"
-			(at 0 -3.66 0)
+			(at 0 -3.66 360)
 			(layer "F.SilkS")
 			(hide yes)
@@
 		)
 		(property "Value" "5kΩ"
-			(at 0 3.67 0)
+			(at 0 3.67 360)
 			(layer "F.Fab")
 			(effects
@@
 		)
 		(fp_text user "${REFERENCE}"
-			(at -0.635 0.005 0)
+			(at -0.635 0.005 360)
 			(layer "F.Fab")
 			(effects
@@
 			)
 		)
-		(property "Value" "1kΩ"
+		(property "Value" "~"
 			(at 0 1.65 0)
 			(layer "F.Fab")
@@
 	)
 	(segment
-		(start 128.42875 84.455)
+		(start 132.08 79.375001)
+		(end 132.08 80.80375)
+		(width 1.905)
+		(layer "B.Cu")
+		(net 4)
+	)
+	(segment
+		(start 132.08 80.80375)
 		(end 133.50875 79.375)
 		(width 1.905)
@@
 		(width 1.905)
 		(layer "B.Cu")
+		(net 4)
+	)
+	(segment
+		(start 128.42875 84.455)
+		(end 132.08 80.80375)
+		(width 1.905)
+		(layer "B.Cu")
+		(net 4)
+	)
+	(segment
+		(start 133.50875 79.375)
+		(end 132.080001 79.375)
+		(width 1.905)
+		(layer "B.Cu")
+		(net 4)
+	)
+	(segment
+		(start 132.080001 79.375)
+		(end 132.08 79.375001)
+		(width 1.905)
+		(layer "B.Cu")

Commit message: modified:   .DS_Store 	new file:   hardware/REM-5.0/#auto_saved_files# 	deleted:    hardware/REM-5.0/REM-5.0-backups/REM-5.0-2026-05-12_155759.zip 	deleted:    hardware/REM-5.0/REM-5.0-backups/REM-5.0-2026-05-12_160527.zip 	deleted:    hardware/REM-5.0/REM-5.0-backups/REM-5.0-2026-05-21_105350.zip 	new file:   hardware/REM-5.0/REM-5.0-backups/REM-5.0-2026-05-29_114350.zip 	new file:   hardware/REM-5.0/REM-5.0-backups/REM-5.0-2026-05-29_130144.zip 	new file:   hardware/REM-5.0/REM-5.0-backups/REM-5.0-2026-05-29_130807.zip 	new file:   hardware/REM-5.0/REM-5.0-backups/REM-5.0-2026-05-29_131841.zip 	new file:   hardware/REM-5.0/REM-5.0-backups/REM-5.0-2026-05-29_144946.zip 	new file:   hardware/REM-5.0/REM-5.0-backups/REM-5.0-2026-05-29_155445.zip 	modified:   hardware/REM-5.0/REM-5.0.kicad_pcb 	modified:   hardware/REM-5.0/REM-5.0.kicad_prl 	modified:   hardware/REM-5.0/REM-5.0.kicad_sch 	modified:   hardware/REM-5.0/fabrication-output/REM-5.0-B_Cu.dxf 	modified:   hardware/REM-5.0/fabrication-output/REM-5.0-F_Cu.dxf 	new file:   hardware/REM-5.0/fabrication-output/REM-5.0-job.gbrjob 	modified:   hardware/REM-5.0/fabrication-output/TRACE_BOT.dxf 	modified:   hardware/REM-5.0/fabrication-output/TRACE_TOP.dwg 	modified:   hardware/REM-5.0/fabrication-output/TRACE_TOP.dxf 	modified:   hardware/REM-5.0/fp-info-cache 	new file:   hardware/REM-5.0/~REM-5.0.kicad_pcb.lck 	new file:   hardware/REM-5.0/~REM-5.0.kicad_sch.lck
Parts:
- C7: value 470uF 50V -> 470uF 16V; footprint Capacitor_SMD:CP_Elec_10x10 -> Capacitor_Tantalum_SMD:CP_EIA-7343-15_Kemet-W_Pad2.25x2.55mm_HandSolder
- moved C12 11.1 mm to (179.4, 84.5)
- moved R9 11.1 mm to (179.4, 79.4)
- moved C11 11.1 mm to (179.4, 94.6)
- moved R8 11.1 mm to (179.4, 89.5)
- moved L1 3.49 mm to (152.4, 84.5)
- moved C3 3.49 mm to (135.6, 84.5)
- moved C7 1.21 mm to (102.4, 97.2), turned to 180 degrees
- moved Q1 0.64 mm to (128.1, 87.0)
- moved R13 0.64 mm to (128.1, 96.4)
- moved C1 0.64 mm to (105.9, 81.0)
- moved C2 0.64 mm to (105.9, 85.9)
- moved C4 0.64 mm to (119.7, 75.4)
- moved C5 0.64 mm to (109.9, 69.8)
- moved C6 0.64 mm to (109.9, 71.8)
- moved C8 0.64 mm to (118.7, 96.4)
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Connections:
- C11 pad 2: Net-(J2-Pin_1) -> Net-(J2-Pin_3)
- C12 pad 1: Net-(J2-Pin_1) -> Net-(J2-Pin_2)
- C12 pad 2: Net-(J2-Pin_1) -> Net-(J2-Pin_3)
- J2 pad 2: Net-(J2-Pin_1) -> Net-(J2-Pin_2)
- J2 pad 3: Net-(J2-Pin_1) -> Net-(J2-Pin_3)
- R9 pad 1: Net-(J2-Pin_1) -> Net-(J2-Pin_2)
Routing:
- net Net-(J2-Pin_1): track 73.8 -> 21.2 mm
- net Net-(J2-Pin_2): track 0.00 -> 33.5 mm
- net Net-(J2-Pin_3): track 0.00 -> 24.2 mm
- net +5V: track 68.6 -> 45.7 mm

Commit message: new file:   firmware/ESP32-S3 PWM/.cache/clangd/index/Alignment.hpp.726B1D6F8AC0E5FC.idx 	new file:   firmware/ESP32-S3 PWM/.cache/clangd/index/ArduinoJson.h.11C8086DC5DC1D39.idx 	new file:   firmware/ESP32-S3 PWM/.cache/clangd/index/ArduinoJson.hpp.7FAD813322DCFBBA.idx 	new file:   firmware/ESP32-S3 PWM/.cache/clangd/index/ArduinoStreamReader.hpp.6A6C10A39AA283AA.idx 	new file:   firmware/ESP32-S3 PWM/.cache/clangd/index/ArduinoStringReader.hpp.4194E32BF9D83CDF.idx 	new file:   firmware/ESP32-S3 PWM/.cache/clangd/index/ArduinoStringWriter.hpp.B2A9673B221215CD.idx 	new file:   firmware/ESP32-S3 PWM/.cache/clangd/index/BasicJsonDocument.hpp.FF9A72F18774339B.idx 	new file:   firmware/ESP32-S3 PWM/.cache/clangd/index/CollectionData.hpp.D0A6E066F6D81A3D.idx 	new file:   firmware/ESP32-S3 PWM/.cache/clangd/index/CollectionImpl.hpp.9A8E7E970CC61A36.idx 	new file:   firmware/ESP32-S3 PWM/.cache/clangd/index/Configuration.hpp.709A1F7F02EFA908.idx 	new file:   firmware/ESP32-S3 PWM/.cache/clangd/index/Converter.hpp.2991290B38DAAF2D.idx 	new file:   firmware/ESP32-S3 PWM/.cache/clangd/index/ConverterImpl.hpp.2B62C8A86CE75E37.idx 	new file:   firmware/ESP32-S3 PWM/.cache/clangd/index/CountingDecorator.hpp.4110D54BC05F9B43.idx 	new file:   firmware/ESP32-S3 PWM/.cache/clangd/index/DeserializationError.hpp.EFFDB4C051A5880A.idx 	new file:   firmware/ESP32-S3 PWM/.cache/clangd/index/DeserializationOptions.hpp.D0990CE9A84F0543.idx 	new file:   firmware/ESP32-S3 PWM/.cache/clangd/index/DummyWriter.hpp.436C5532B841A3A4.idx 	new file:   firmware/ESP32-S3 PWM/.cache/clangd/index/DynamicJsonDocument.hpp.DEEADBD70694B4BE.idx 	new file:   firmware/ESP32-S3 PWM/.cache/clangd/index/ElementProxy.hpp.209B2FA01DA5C38D.idx 	new file:   firmware/ESP32-S3 PWM/.cache/clangd/index/EscapeSequence.hpp.0E535D59050D1B63.idx 	new file:   firmware/ESP32-S3 PWM/.cache/clangd/index/Filter.hpp.2866D748202E02C1.idx 	new file:   firmware/ESP32-S3 PWM/.cache/clangd/index/FlashReader.hpp.A4CB3621CFAD50BE.idx 	n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
Routing:
- net Net-(L1-Pad4): track 3.17 -> 4.13 mm
- net Net-(L1-Pad3): track 3.17 -> 4.13 mm
Changed lines of the file:
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@@
 		)
 		(property "Value" "0.01µF 1000"
-			(at 4.999999 3.75 360)
+			(at 4.999999 3.75 0)
 			(layer "F.Fab")
 			(effects
@@
 		)
 		(fp_text user "${REFERENCE}"
-			(at 5 0 360)
+			(at 5 0 0)
 			(layer "F.Fab")
 			(effects
@@
 	)
 	(footprint "Connector_PinHeader_2.54mm:PinHeader_1x03_P5.08mm_Horizontal_2"
+		(locked yes)
 		(layer "F.Cu")
 		(at 180.0225 104.29875 -90)
@@
 		(tags "Resistor Axial_DIN0414 series Axial Horizontal pin pitch 20.32mm 2W length 11.9mm diameter 4.5mm")
 		(property "Reference" "R9"
-			(at 0 -3.37 360)
+			(at 0 -3.37 0)
 			(layer "F.SilkS")
 			(hide yes)
@@
 		)
 		(property "Value" "33Ω 2W"
-			(at 0 3.37 360)
+			(at 0 3.37 0)
 			(layer "F.Fab")
 			(effects
@@
 		)
 		(fp_text user "${REFERENCE}"
-			(at 0 0 360)
+			(at 0 0 0)
 			(layer "F.Fab")
 			(effects
@@
 		)
 		(property "Value" "0.01µF 1000"
-			(at 4.999999 3.75 360)
+			(at 4.999999 3.75 0)
 			(layer "F.Fab")
 			(effects
@@
 		)
 		(fp_text user "${REFERENCE}"
-			(at 5 0 360)
+			(at 5 0 0)
 			(layer "F.Fab")
 			(effects
@@
 		(tags "capacitor tantalum")
 		(property "Reference" "C7"
-			(at 0 -3.1 360)
+			(at 0 -3.1 0)
 			(layer "F.SilkS")
 			(hide yes)
@@
 		)
 		(property "Value" "470uF 16V"
-			(at 0 3.1 360)
+			(at 0 3.1 0)
 			(layer "F.Fab")
 			(effects
@@
 		)
 		(fp_text user "${REFERENCE}"
-			(at 0 0 360)
+			(at 0 0 0)
 			(layer "F.Fab")
 			(effects
@@
 	(segment
 		(start 169.2275 79.375001)
-		(end 166.0525 79.375001)
+		(end 165.1 79.375001)
 		(width 2.8575)
 		(layer "B.Cu")
@@
 	(segment
 		(start 169.2275 89.535001)
-		(end 166.0525 89.535001)
+		(end 165.1 89.535001)
 		(width 2.8575)
 		(layer "B.Cu")
