File: hardware/REM-5.0/REM-5.0.kicad_pcb (KiCad board)
At the start: 2 copper layers, 98.4 x 44.5 mm, 35 parts, among them J1 PinHeader_2.54mm 02x04 Horizo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, J2 PinHeader_2.54mm 02x05 Horizo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, Q1 IRLB3034PbF, Q2 BCX56, Q3 BCX53, U2 74LVC1G14

Commit message: modified:   firmware/ESU_V1/include/config.h 	modified:   firmware/ESU_V1/src/hardware_control.cpp 	new file:   hardware/REM-4.0/.history 	new file:   hardware/REM-5.0/.history 	modified:   hardware/REM-5.0/REM-5.0.kicad_pcb 	modified:   hardware/REM-5.0/REM-5.0.kicad_prl 	modified:   hardware/REM-5.0/REM-5.0.kicad_pro 	modified:   hardware/REM-5.0/REM-5.0.kicad_sch 	modified:   hardware/REM-5.0/fabrication-output/REM-5.0-B_Cu.dxf 	new file:   hardware/REM-5.0/fabrication-output/REM-5.0-B_Cu.pdf 	modified:   hardware/REM-5.0/fabrication-output/REM-5.0-F_Cu.dxf 	new file:   hardware/REM-5.0/fabrication-output/REM-5.0-F_Cu.pdf 	new file:   hardware/REM-5.0/fabrication-output/TRACE_BOT_2.dwg 	new file:   hardware/REM-6.0/.history 	new file:   hardware/REM-6.0/REM-6.0.kicad_pcb 	new file:   hardware/REM-6.0/REM-6.0.kicad_prl 	new file:   hardware/REM-6.0/REM-6.0.kicad_pro 	new file:   hardware/REM-6.0/REM-6.0.kicad_sch 	new file:   hardware/REM-6.0/REM-6.asc 	new file:   hardware/REM-6.0/fabrication-output/MARK_B.dxf 	new file:   hardware/REM-6.0/fabrication-output/MARK_F.dxf 	new file:   hardware/REM-6.0/fabrication-output/REM-6.0-B_Cu.dxf 	new file:   hardware/REM-6.0/fabrication-output/REM-6.0-B_Cu.pdf 	new file:   hardware/REM-6.0/fabrication-output/REM-6.0-F_Cu.dxf 	new file:   hardware/REM-6.0/fabrication-output/REM-6.0-F_Cu.pdf 	new file:   hardware/REM-6.0/~REM-6.0.kicad_pcb.lck 	new file:   hardware/REM-6.0/~REM-6.0.kicad_pro.lck 	new file:   hardware/REM-6B/.history 	new file:   hardware/REM-6B/REM-6B.kicad_pcb 	new file:   hardware/REM-6B/REM-6B.kicad_prl 	new file:   hardware/REM-6B/REM-6B.kicad_pro 	new file:   hardware/REM-6B/REM-6B.kicad_sch
Parts:
- added TP1: ~, TestPoint:TestPoint_Bridge_Pitch2.54mm_Drill1.0mm, F.Cu at (125.6, 91.8)
- added TP2: ~, TestPoint:TestPoint_Bridge_Pitch2.54mm_Drill1.0mm, F.Cu at (134.3, 75.6)
Connections:
- C3 pad 1: Net-(C3-Pad1) -> +5V
- L1 pad 2: Net-(C3-Pad1) -> +5V
- R8 pad 2: Net-(L1-Pad4) -> Net-(L1-Pad3)
- R9 pad 2: Net-(L1-Pad3) -> Net-(L1-Pad4)
Routing:
- net +5V: track 45.7 -> 68.3 mm
- net Net-(Q1-D): track 25.7 -> 34.3 mm
- net Net-(C3-Pad1): track 4.13 -> 0.00 mm
- net Net-(Q1-G): track 9.92 -> 12.5 mm
