File: hardware/REM-5.0/REM-5.0.kicad_sch (KiCad schematic)
At the start: 39 parts, among them J1 PinHeader_2.54mm 02x04 Horizo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, J2 PinHeader_2.54mm 02x05 Horizo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, Q1 IRLB3034PbF, Q2 BCX56, Q3 BCX53, U2 74LVC1G14

Commit message: deleted:    hardware/CTL-6.0/CTL-6.0-backups/CTL-6.0-2026-05-05_105851.zip 	new file:   hardware/CTL-6.0/CTL-6.0-backups/CTL-6.0-2026-05-21_155839.zip 	modified:   hardware/CTL-6.0/CTL-6.0.kicad_pcb 	new file:   hardware/CTL-6.1/CTL-6.0-backups/CTL-6.0-2026-05-04_160013.zip 	new file:   hardware/CTL-6.1/CTL-6.0-backups/CTL-6.0-2026-05-04_160854.zip 	new file:   hardware/CTL-6.1/CTL-6.0-backups/CTL-6.0-2026-05-04_161354.zip 	new file:   hardware/CTL-6.1/CTL-6.0-backups/CTL-6.0-2026-05-04_161937.zip 	new file:   hardware/CTL-6.1/CTL-6.0-backups/CTL-6.0-2026-05-04_162757.zip 	new file:   hardware/CTL-6.1/CTL-6.0-backups/CTL-6.0-2026-05-05_110550.zip 	new file:   hardware/CTL-6.1/CTL-6.0-backups/CTL-6.0-2026-05-05_111755.zip 	new file:   hardware/CTL-6.1/CTL-6.0-backups/CTL-6.0-2026-05-05_114939.zip 	new file:   hardware/CTL-6.1/CTL-6.0-backups/CTL-6.0-2026-05-05_155039.zip 	new file:   hardware/CTL-6.1/CTL-6.0-backups/CTL-6.0-2026-05-05_204356.zip 	new file:   hardware/CTL-6.1/CTL-6.0-backups/CTL-6.0-2026-05-21_155839.zip 	new file:   hardware/CTL-6.1/CTL-6.1-backups/CTL-6.1-2026-05-21_160708.zip 	new file:   hardware/CTL-6.1/CTL-6.1-backups/CTL-6.1-2026-05-21_163235.zip 	new file:   hardware/CTL-6.1/CTL-6.1.FCStd 	new file:   hardware/CTL-6.1/CTL-6.1.iges 	new file:   hardware/CTL-6.1/CTL-6.1.kicad_pcb 	new file:   hardware/CTL-6.1/CTL-6.1.kicad_prl 	new file:   hardware/CTL-6.1/CTL-6.1.kicad_pro 	new file:   hardware/CTL-6.1/CTL-6.1.kicad_sch 	new file:   hardware/CTL-6.1/CTL-6.1.png 	new file:   hardware/CTL-6.1/CTL-6.1.step 	new file:   hardware/CTL-6.1/CTL-6.1.xlsx 	new file:   hardware/CTL-6.1/bom/ibom.html 	new file:   hardware/CTL-6.1/fabrication-output/CTL-4.3-B_Cu.pdf 	new file:   hardware/CTL-6.1/fabrication-output/CTL-4.3-B_Mask.pdf 	new file:   hardware/CTL-6.1/fabrication-output/CTL-4.3-B_Paste.pdf 	new file:   hardware/CTL-6.1/fabrication-output/CTL-4.3-B_Silkscreen.pdf 	new file:   hardware/CTL-6.1/fabrication-output/CTL-4.3-Edge_Cuts.pdf 	new file:   h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
Parts:
- R1, R2, R6, R7: value 1kΩ -> ~
Changed lines of the file:
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@@
 			)
 		)
-		(property "Value" "1kΩ"
+		(property "Value" "~"
 			(at 136.398 90.17 90)
 			(effects
@@
 			)
 		)
-		(property "Value" "1kΩ"
+		(property "Value" "~"
 			(at 158.75 103.632 90)
 			(effects
@@
 			)
 		)
-		(property "Value" "1kΩ"
+		(property "Value" "~"
 			(at 103.632 54.61 90)
 			(effects
@@
 			)
 		)
-		(property "Value" "1kΩ"
+		(property "Value" "~"
 			(at 136.398 97.79 90)
 			(effects

Commit message: modified:   .DS_Store 	new file:   hardware/REM-5.0/#auto_saved_files# 	deleted:    hardware/REM-5.0/REM-5.0-backups/REM-5.0-2026-05-12_155759.zip 	deleted:    hardware/REM-5.0/REM-5.0-backups/REM-5.0-2026-05-12_160527.zip 	deleted:    hardware/REM-5.0/REM-5.0-backups/REM-5.0-2026-05-21_105350.zip 	new file:   hardware/REM-5.0/REM-5.0-backups/REM-5.0-2026-05-29_114350.zip 	new file:   hardware/REM-5.0/REM-5.0-backups/REM-5.0-2026-05-29_130144.zip 	new file:   hardware/REM-5.0/REM-5.0-backups/REM-5.0-2026-05-29_130807.zip 	new file:   hardware/REM-5.0/REM-5.0-backups/REM-5.0-2026-05-29_131841.zip 	new file:   hardware/REM-5.0/REM-5.0-backups/REM-5.0-2026-05-29_144946.zip 	new file:   hardware/REM-5.0/REM-5.0-backups/REM-5.0-2026-05-29_155445.zip 	modified:   hardware/REM-5.0/REM-5.0.kicad_pcb 	modified:   hardware/REM-5.0/REM-5.0.kicad_prl 	modified:   hardware/REM-5.0/REM-5.0.kicad_sch 	modified:   hardware/REM-5.0/fabrication-output/REM-5.0-B_Cu.dxf 	modified:   hardware/REM-5.0/fabrication-output/REM-5.0-F_Cu.dxf 	new file:   hardware/REM-5.0/fabrication-output/REM-5.0-job.gbrjob 	modified:   hardware/REM-5.0/fabrication-output/TRACE_BOT.dxf 	modified:   hardware/REM-5.0/fabrication-output/TRACE_TOP.dwg 	modified:   hardware/REM-5.0/fabrication-output/TRACE_TOP.dxf 	modified:   hardware/REM-5.0/fp-info-cache 	new file:   hardware/REM-5.0/~REM-5.0.kicad_pcb.lck 	new file:   hardware/REM-5.0/~REM-5.0.kicad_sch.lck
Parts:
- C7: value 470uF 50V -> 470uF 16V; footprint Capacitor_SMD:CP_Elec_10x10 -> Capacitor_Tantalum_SMD:CP_EIA-7343-15_Kemet-W_Pad2.25x2.55mm_HandSolder
Connections:
- new net: C11.1, J2.1 (Pin_1), R8.1
- new net: C12.1, J2.2 (Pin_2), R9.1
- new net: C11.2, C12.2, J2.3 (Pin_3)
Changed lines of the file:
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@@
 	)
 	(junction
-		(at 279.4 83.82)
-		(diameter 0)
-		(color 0 0 0 0)
-	)
-	(junction
 		(at 132.08 101.6)
 		(diameter 0)
@@
 		(color 0 0 0 0)
 	)
-	(junction
-		(at 279.4 86.36)
-		(diameter 0)
-		(color 0 0 0 0)
-	)
 	(wire
 		(pts
@@
 	(wire
 		(pts
-			(xy 276.86 81.28) (xy 276.86 114.3)
+			(xy 276.86 88.9) (xy 276.86 114.3)
 		)
 		(stroke
@@
 	(wire
 		(pts
-			(xy 279.4 81.28) (xy 279.4 83.82)
-		)
-		(stroke
-			(width 0)
-			(type default)
-		)
-	)
-	(wire
-		(pts
 			(xy 187.96 96.52) (xy 190.5 96.52)
 		)
@@
 	(wire
 		(pts
-			(xy 279.4 86.36) (xy 279.4 88.9)
-		)
-		(stroke
-			(width 0)
-			(type default)
-		)
-	)
-	(wire
-		(pts
 			(xy 81.28 30.48) (xy 81.28 36.83)
 		)
@@
 	(wire
 		(pts
-			(xy 279.4 81.28) (xy 276.86 81.28)
+			(xy 279.4 88.9) (xy 276.86 88.9)
 		)
 		(stroke
@@
 	(wire
 		(pts
-			(xy 279.4 83.82) (xy 279.4 86.36)
-		)
-		(stroke
-			(width 0)
-			(type default)
-		)
-	)
-	(wire
-		(pts
 			(xy 129.54 86.36) (xy 132.08 86.36)
 		)
@@
 		(lib_id "Connector_Generic:Conn_01x03")
 		(at 284.48 86.36 0)
-		(mirror x)
 		(unit 1)
 		(exclude_from_sim no)
@@
 		)
 		(property "Value" "PinHeader_2.54mm 02x05 Horizontal"
-			(at 287.02 85.0901 0)
+			(at 287.02 87.6299 0)
 			(effects
 				(font
@@
 			)
 		)
-		(property "Value" "470uF 50V"
+		(property "Value" "470uF 16V"
 			(at 95.758 119.38 90)
 			(effects
@@
 			)
 		)
-		(property "Footprint" "Capacitor_SMD:CP_Elec_10x10"
+		(property "Footprint" "Capacitor_Tantalum_SMD:CP_EIA-7343-15_Kemet-W_Pad2.25x2.55mm_HandSolder"
 			(at 100.0252 123.19 0)
 			(effects
@@
 			)
 		)
-		(property "Description" "Polarized capacitor"
+		(property "Description" "Tantalum capacitor"
 			(at 99.06 119.38 0)
 			(effects

Commit message: new file:   firmware/ESP32-S3 PWM/.cache/clangd/index/Alignment.hpp.726B1D6F8AC0E5FC.idx 	new file:   firmware/ESP32-S3 PWM/.cache/clangd/index/ArduinoJson.h.11C8086DC5DC1D39.idx 	new file:   firmware/ESP32-S3 PWM/.cache/clangd/index/ArduinoJson.hpp.7FAD813322DCFBBA.idx 	new file:   firmware/ESP32-S3 PWM/.cache/clangd/index/ArduinoStreamReader.hpp.6A6C10A39AA283AA.idx 	new file:   firmware/ESP32-S3 PWM/.cache/clangd/index/ArduinoStringReader.hpp.4194E32BF9D83CDF.idx 	new file:   firmware/ESP32-S3 PWM/.cache/clangd/index/ArduinoStringWriter.hpp.B2A9673B221215CD.idx 	new file:   firmware/ESP32-S3 PWM/.cache/clangd/index/BasicJsonDocument.hpp.FF9A72F18774339B.idx 	new file:   firmware/ESP32-S3 PWM/.cache/clangd/index/CollectionData.hpp.D0A6E066F6D81A3D.idx 	new file:   firmware/ESP32-S3 PWM/.cache/clangd/index/CollectionImpl.hpp.9A8E7E970CC61A36.idx 	new file:   firmware/ESP32-S3 PWM/.cache/clangd/index/Configuration.hpp.709A1F7F02EFA908.idx 	new file:   firmware/ESP32-S3 PWM/.cache/clangd/index/Converter.hpp.2991290B38DAAF2D.idx 	new file:   firmware/ESP32-S3 PWM/.cache/clangd/index/ConverterImpl.hpp.2B62C8A86CE75E37.idx 	new file:   firmware/ESP32-S3 PWM/.cache/clangd/index/CountingDecorator.hpp.4110D54BC05F9B43.idx 	new file:   firmware/ESP32-S3 PWM/.cache/clangd/index/DeserializationError.hpp.EFFDB4C051A5880A.idx 	new file:   firmware/ESP32-S3 PWM/.cache/clangd/index/DeserializationOptions.hpp.D0990CE9A84F0543.idx 	new file:   firmware/ESP32-S3 PWM/.cache/clangd/index/DummyWriter.hpp.436C5532B841A3A4.idx 	new file:   firmware/ESP32-S3 PWM/.cache/clangd/index/DynamicJsonDocument.hpp.DEEADBD70694B4BE.idx 	new file:   firmware/ESP32-S3 PWM/.cache/clangd/index/ElementProxy.hpp.209B2FA01DA5C38D.idx 	new file:   firmware/ESP32-S3 PWM/.cache/clangd/index/EscapeSequence.hpp.0E535D59050D1B63.idx 	new file:   firmware/ESP32-S3 PWM/.cache/clangd/index/Filter.hpp.2866D748202E02C1.idx 	new file:   firmware/ESP32-S3 PWM/.cache/clangd/index/FlashReader.hpp.A4CB3621CFAD50BE.idx 	n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
Other:
- moved on the sheet: C1, C11, C12, C2, C3, C4, C5, C6, C7, C8, D4, D5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

Commit message: new file:   hardware/INA-3.1/INA-3.1-backups/INA-3.1-2026-06-03_154006.zip 	new file:   hardware/INA-3/INA-3-backups/INA-3-2026-06-03_161017.zip 	new file:   hardware/INA-3/INA-3-backups/INA-3-2026-06-03_161951.zip 	new file:   hardware/INA-4.0/INA-4.0-backups/INA-4.0-2026-06-03_153924.zip 	deleted:    hardware/REM-5.0/REM-5.0-backups/REM-5.0-2026-05-13_154048.zip 	deleted:    hardware/REM-5.0/REM-5.0-backups/REM-5.0-2026-05-13_155631.zip 	deleted:    hardware/REM-5.0/REM-5.0-backups/REM-5.0-2026-05-13_161956.zip 	deleted:    hardware/REM-5.0/REM-5.0-backups/REM-5.0-2026-05-13_162957.zip 	deleted:    hardware/REM-5.0/REM-5.0-backups/REM-5.0-2026-05-18_092511.zip 	deleted:    hardware/REM-5.0/REM-5.0-backups/REM-5.0-2026-05-18_093513.zip 	new file:   hardware/REM-5.0/REM-5.0-backups/REM-5.0-2026-06-04_102738.zip 	new file:   hardware/REM-5.0/REM-5.0-backups/REM-5.0-2026-06-04_103505.zip 	new file:   hardware/REM-5.0/REM-5.0-backups/REM-5.0-2026-06-04_104754.zip 	new file:   hardware/REM-5.0/REM-5.0-backups/REM-5.0-2026-06-04_164037.zip 	new file:   hardware/REM-5.0/REM-5.0-backups/REM-5.0-2026-06-05_111411.zip 	new file:   hardware/REM-5.0/REM-5.0-backups/REM-5.0-2026-06-05_115032.zip 	modified:   hardware/REM-5.0/REM-5.0.kicad_pcb 	modified:   hardware/REM-5.0/REM-5.0.kicad_prl 	modified:   hardware/REM-5.0/REM-5.0.kicad_sch 	new file:   hardware/REM-5.0/SHIELD.dxf 	new file:   hardware/REM-5.0/_autosave-REM-5.0.kicad_pcb 	new file:   hardware/REM-5.0/~REM-5.0.kicad_sch.lck 	new file:   hardware/REM-5.0/~_autosave-REM-5.0.kicad_pcb.lck
Parts:
- L1: symbol Device:L_Coupled -> Device:L_Coupled_1243
Connections:
- net at L1.3: now also R8.2; no longer R9.2
- net at L1.4: now also R9.2; no longer R8.2
Changed lines of the file:
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@@
 	)
 	(symbol
-		(lib_id "Device:L_Coupled")
+		(lib_id "Device:L_Coupled_1243")
 		(at 209.55 95.25 90)
 		(unit 1)

Commit message: modified:   firmware/ESU_V1/include/config.h 	modified:   firmware/ESU_V1/src/hardware_control.cpp 	new file:   hardware/REM-4.0/.history 	new file:   hardware/REM-5.0/.history 	modified:   hardware/REM-5.0/REM-5.0.kicad_pcb 	modified:   hardware/REM-5.0/REM-5.0.kicad_prl 	modified:   hardware/REM-5.0/REM-5.0.kicad_pro 	modified:   hardware/REM-5.0/REM-5.0.kicad_sch 	modified:   hardware/REM-5.0/fabrication-output/REM-5.0-B_Cu.dxf 	new file:   hardware/REM-5.0/fabrication-output/REM-5.0-B_Cu.pdf 	modified:   hardware/REM-5.0/fabrication-output/REM-5.0-F_Cu.dxf 	new file:   hardware/REM-5.0/fabrication-output/REM-5.0-F_Cu.pdf 	new file:   hardware/REM-5.0/fabrication-output/TRACE_BOT_2.dwg 	new file:   hardware/REM-6.0/.history 	new file:   hardware/REM-6.0/REM-6.0.kicad_pcb 	new file:   hardware/REM-6.0/REM-6.0.kicad_prl 	new file:   hardware/REM-6.0/REM-6.0.kicad_pro 	new file:   hardware/REM-6.0/REM-6.0.kicad_sch 	new file:   hardware/REM-6.0/REM-6.asc 	new file:   hardware/REM-6.0/fabrication-output/MARK_B.dxf 	new file:   hardware/REM-6.0/fabrication-output/MARK_F.dxf 	new file:   hardware/REM-6.0/fabrication-output/REM-6.0-B_Cu.dxf 	new file:   hardware/REM-6.0/fabrication-output/REM-6.0-B_Cu.pdf 	new file:   hardware/REM-6.0/fabrication-output/REM-6.0-F_Cu.dxf 	new file:   hardware/REM-6.0/fabrication-output/REM-6.0-F_Cu.pdf 	new file:   hardware/REM-6.0/~REM-6.0.kicad_pcb.lck 	new file:   hardware/REM-6.0/~REM-6.0.kicad_pro.lck 	new file:   hardware/REM-6B/.history 	new file:   hardware/REM-6B/REM-6B.kicad_pcb 	new file:   hardware/REM-6B/REM-6B.kicad_prl 	new file:   hardware/REM-6B/REM-6B.kicad_pro 	new file:   hardware/REM-6B/REM-6B.kicad_sch
Parts:
- removed TP5, TP7: ~, TestPoint:TestPoint_Bridge_Pitch2.54mm_Drill1.0mm, symbol Connector:TestPoint
- R1, R2, R6, R7, TP1, TP2: value ~ -> (none)
Connections:
- net +5V: now also C3.1, L1.2
- net at Q1.1 (G), R13.2, R3.2: now also TP1.1
- net REM: now reaches C6.1, J1.1 (Pin_1), R5.2, R7.1, RV1.3
