File: hardware/INA-3/INA-3.kicad_sch (KiCad schematic)
At the start: 20 parts, among them J1 Conn_01x05, U1 OPA365, U2 OPA365, U3 OPA365, U4 AMS1117-1.8

Commit message: modified:   .DS_Store 	new file:   archive/Payment 20260424.pdf 	new file:   archive/Purchase 20260424.docx 	new file:   archive/REM_OUTPUT.xlsx 	modified:   firmware/ESP32-S3 PWM/include/config.h 	modified:   firmware/ESP32-S3 PWM/src/hardware_control.cpp 	deleted:    hardware/CTL-5.0/CTL-5.0-backups/CTL-5.0-2026-02-20_154251.zip 	deleted:    hardware/CTL-5.0/CTL-5.0-backups/CTL-5.0-2026-02-20_184343.zip 	deleted:    hardware/CTL-5.0/CTL-5.0-backups/CTL-5.0-2026-02-26_100701.zip 	deleted:    hardware/CTL-5.0/CTL-5.0-backups/CTL-5.0-2026-02-26_102054.zip 	deleted:    hardware/CTL-5.0/CTL-5.0-backups/CTL-5.0-2026-02-26_102605.zip 	deleted:    hardware/CTL-5.0/CTL-5.0-backups/CTL-5.0-2026-02-26_103340.zip 	deleted:    hardware/CTL-5.0/CTL-5.0-backups/CTL-5.0-2026-02-26_153650.zip 	new file:   hardware/CTL-5.0/CTL-5.0-backups/CTL-5.0-2026-04-30_153803.zip 	new file:   hardware/CTL-5.0/CTL-5.0-backups/CTL-5.0-2026-04-30_154828.zip 	new file:   hardware/CTL-5.0/CTL-5.0-backups/CTL-5.0-2026-04-30_160225.zip 	new file:   hardware/CTL-5.0/CTL-5.0-backups/CTL-5.0-2026-04-30_161241.zip 	new file:   hardware/CTL-5.0/CTL-5.0-backups/CTL-5.0-2026-04-30_162225.zip 	new file:   hardware/CTL-5.0/CTL-5.0-backups/CTL-5.0-2026-04-30_162925.zip 	modified:   hardware/CTL-5.0/CTL-5.0.kicad_pcb 	modified:   hardware/CTL-5.0/CTL-5.0.kicad_sch 	modified:   hardware/CTL-5.0/fp-info-cache 	deleted:    hardware/INA-3.1/INA-3.1-backups/INA-3.1-2026-04-21_104126.zip 	new file:   hardware/INA-3.1/INA-3.1-backups/INA-3.1-2026-04-29_085310.zip 	new file:   hardware/INA-3.1/INA-3.1-backups/INA-3.1-2026-04-30_110843.zip 	new file:   hardware/INA-3.1/INA-3.1-backups/INA-3.1-2026-04-30_111401.zip 	new file:   hardware/INA-3.1/INA-3.1-backups/INA-3.1-2026-04-30_111913.zip 	new file:   hardware/INA-3.1/INA-3.1-backups/INA-3.1-2026-04-30_112649.zip 	new file:   hardware/INA-3.1/INA-3.1-backups/INA-3.1-2026-04-30_113258.zip 	modified:   hardware/INA-3.1/INA-3.1.kicad_pcb 	modified:   hardware/INA-3.1/INA-3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
Parts:
- added C8: 100nF, Capacitor_SMD:C_0805_2012Metric_Pad1.18x1.45mm_HandSolder, symbol Device:C
- added R9: 10kΩ, Resistor_SMD:R_0805_2012Metric_Pad1.20x1.40mm_HandSolder, symbol Device:R
- R1: value 6.8kΩ -> 5.1kΩ
Connections:
- net GND: now also C8.2
- net OUT: now also C8.1, R9.2; no longer R6.2, U3.1
- new net: R6.2, R9.1, U3.1
Changed lines of the file:
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@@
+	)
+	(junction
+		(at 132.08 55.88)
+		(diameter 0)
+		(color 0 0 0 0)
 	)
 	(junction
@@
 	(wire
 		(pts
+			(xy 129.54 55.88) (xy 132.08 55.88)
+		)
+		(stroke
+			(width 0)
+			(type default)
+		)
+	)
+	(wire
+		(pts
+			(xy 132.08 55.88) (xy 139.7 55.88)
+		)
+		(stroke
+			(width 0)
+			(type default)
+		)
+	)
+	(wire
+		(pts
 			(xy 68.58 137.16) (xy 68.58 142.24)
 		)
@@
 	(wire
 		(pts
-			(xy 119.38 55.88) (xy 127 55.88)
+			(xy 119.38 55.88) (xy 121.92 55.88)
 		)
 		(stroke
@@
 	(wire
 		(pts
+			(xy 132.08 55.88) (xy 132.08 58.42)
+		)
+		(stroke
+			(width 0)
+			(type default)
+		)
+	)
+	(wire
+		(pts
 			(xy 68.58 124.46) (xy 63.5 124.46)
 		)
@@
 			(width 0)
 			(type default)
-		)
-	)
-	(label "OUT"
-		(at 121.92 55.88 0)
-		(fields_autoplaced yes)
-		(effects
-			(font
-				(size 1 1)
-			)
-			(justify left bottom)
 		)
 	)
@@
 		)
 	)
+	(label "OUT"
+		(at 134.62 55.88 0)
+		(fields_autoplaced yes)
+		(effects
+			(font
+				(size 1 1)
+			)
+			(justify left bottom)
+		)
+	)
 	(label "IN"
 		(at 36.83 71.12 0)
@@
 			)
 		)
-		(property "Value" "6.8kΩ"
+		(property "Value" "5.1kΩ"
 			(at 67.818 56.896 0)
 			(effects
@@
 				(path "/012ecf8f-e59d-4b86-a3cc-27fec600e7df"
 					(reference "#PWR07")
+					(unit 1)
+				)
+			)
+		)
+	)
+	(symbol
+		(lib_id "Device:C")
+		(at 132.08 62.23 0)
+		(unit 1)
+		(exclude_from_sim no)
+		(in_bom yes)
+		(on_board yes)
+		(dnp no)
+		(property "Reference" "C8"
+			(at 132.334 60.198 0)
+			(effects
+				(font
+					(size 1 1)
+				)
+				(justify left)
+			)
+		)
+		(property "Value" "100nF"
+			(at 132.334 64.262 0)
+			(effects
+				(font
+					(size 1 1)
+				)
+				(justify left)
+			)
+		)
+		(property "Footprint" "Capacitor_SMD:C_0805_2012Metric_Pad1.18x1.45mm_HandSolder"
+			(at 133.0452 66.04 0)
+			(effects
+				(font
+					(size 1.27 1.27)
+				)
+				(hide yes)
+			)
+		)
+		(property "Datasheet" "~"
+			(at 132.08 62.23 0)
+			(effects
+				(font
+					(size 1.27 1.27)
+				)
+				(hide yes)
+			)
+		)
+		(property "Description" "Unpolarized capacitor"
+			(at 132.08 62.23 0)
+			(effects
+				(font
+					(size 1.27 1.27)
+				)
+				(hide yes)
+			)
+		)
+		(pin "1"
+		)
+		(pin "2"
+		)
+		(instances
+			(project "INA-3"
+				(path "/012ecf8f-e59d-4b86-a3cc-27fec600e7df"
+					(reference "C8")
 					(unit 1)
 				)
@@
 	(symbol
 		(lib_id "Device:R")
+		(at 125.73 55.88 90)
+		(unit 1)
+		(exclude_from_sim no)
+		(in_bom yes)
+		(on_board yes)
+		(dnp no)
+		(property "Reference" "R9"
+			(at 125.73 53.594 90)
+			(effects
+				(font
+					(size 1 1)
+				)
+			)
+		)
+		(property "Value" "10kΩ"
+			(at 125.73 58.166 90)
+			(effects
+				(font
+					(size 1 1)
+				)
+			)
+		)
+		(property "Footprint" "Resistor_SMD:R_0805_2012Metric_Pad1.20x1.40mm_HandSolder"
+			(at 125.73 57.658 90)
+			(effects
+				(font
+					(size 1.27 1.27)
+				)
+				(hide yes)
+			)
+		)
+		(property "Datasheet" "~"
+			(at 125.73 55.88 0)
+			(effects
+				(font
+					(size 1.27 1.27)
+				)
+				(hide yes)
+			)
+		)
+		(property "Description" "Resistor"
+			(at 125.73 55.88 0)
+			(effects
+				(font
+					(size 1.27 1.27)
+				)
+				(hide yes)
+			)
+		)
+		(pin "2"
+		)
+		(pin "1"
+		)
+		(instances
+			(project "INA-3"
+				(path "/012ecf8f-e59d-4b86-a3cc-27fec600e7df"
+					(reference "R9")
+					(unit 1)
+				)
+			)
+		)
+	)
+	(symbol
+		(lib_id "Device:R")
 		(at 92.71 62.23 90)
 		(unit 1)
@@
 					(unit 1)
 				)
+			)
+		)
+	)
+	(symbol
+		(lib_id "power:GND")
+		(at 132.08 66.04 0)
+		(unit 1)
+		(exclude_from_sim no)
+		(in_bom yes)
+		(on_board yes)
+		(dnp no)
+		(fields_autoplaced yes)
+		(property "Reference" "#PWR09"
+			(at 132.08 72.39 0)
+			(effects
+				(font
+					(size 1.27 1.27)
+				)
+				(hide yes)
+			)
+		)
+		(property "Value" "GND"
+			(at 132.08 71.12 0)
+			(effects
+				(font
+					(size 1.27 1.27)
+				)
+				(hide yes)
+			)
+		)
+		(property "Footprint" ""
+			(at 132.08 66.04 0)
+			(effects
+				(font
+					(size 1.27 1.27)
+				)
+				(hide yes)
+			)
+		)
+		(property "Datasheet" ""
+			(at 132.08 66.04 0)
+			(effects
+				(font
+					(size 1.27 1.27)
+				)
+				(hide yes)
+			)
+		)
+		(property "Description" "Power symbol creates a global label with name \"GND\" , ground"
+			(at 132.08 66.04 0)
+			(effects
+				(font
+					(size 1.27 1.27)
+				)
+				(hide yes)
+			)
+		)
+		(pin "1"
+		)
+		(instances
+			(project "INA-3"
+				(path "/012ecf8f-e59d-4b86-a3cc-27fec600e7df"
+					(reference "#PWR09")
+					(unit 1)
+				)

Commit message: modified:   firmware/ESU_V1/include/data_manager.h 	modified:   firmware/ESU_V1/include/hardware_control.h 	modified:   firmware/ESU_V1/src/hardware_control.cpp 	modified:   firmware/ESU_V1/src/main.cpp 	modified:   hardware/CTL-6.1/CTL-6.1.kicad_pcb 	modified:   hardware/CTL-6.1/CTL-6.1.kicad_prl 	modified:   hardware/CTL-6.1/CTL-6.1.kicad_pro 	modified:   hardware/INA-3/INA-3.kicad_pcb 	modified:   hardware/INA-3/INA-3.kicad_prl 	modified:   hardware/INA-3/INA-3.kicad_pro 	modified:   hardware/INA-3/INA-3.kicad_sch 	renamed:    hardware/INA-3/fabrication-outputs/INA-3-TRACE.dxf -> hardware/INA-3/fabrication-outputs/EDGE.dxf 	deleted:    hardware/INA-3/fabrication-outputs/INA-3-Edge_Cuts.dxf 	modified:   hardware/INA-3/fabrication-outputs/INA-3-F_Cu.dxf 	new file:   hardware/INA-3/fabrication-outputs/INA-3-F_Cu.pdf 	deleted:    hardware/INA-3/fabrication-outputs/INA-3-NPTH-drl_map.dxf 	deleted:    hardware/INA-3/fabrication-outputs/INA-3-PTH-drl_map.dxf 	new file:   hardware/INA-3/fabrication-outputs/TRACE.dxf 	deleted:    hardware/INA-3/fp-info-cache 	new file:   hardware/REM-5.0/.history 	modified:   hardware/REM-5.0/REM-5.0.kicad_pcb 	modified:   hardware/REM-5.0/REM-5.0.kicad_prl 	modified:   hardware/REM-5.0/REM-5.0.kicad_pro
Parts:
- added C9: 100nF, Capacitor_SMD:C_0805_2012Metric_Pad1.18x1.45mm_HandSolder, symbol Device:C
- added R10, R11: 10kΩ, Resistor_SMD:R_0805_2012Metric_Pad1.20x1.40mm_HandSolder, symbol Device:R
Connections:
- net GND: now also C9.2, R11.2
- net OUT: now also C9.1, R10.2, R11.1; no longer C8.1, R9.2
- new net: C8.1, R10.1, R9.2
