File: hardware/INA-3/INA-3.kicad_pcb (KiCad board)
At the start: 2 copper layers, 29.5 x 24.4 mm, 20 parts, among them J1 Conn_01x05, U1 OPA365, U2 OPA365, U3 OPA365, U4 AMS1117-1.8

Commit message: modified:   .DS_Store 	new file:   archive/Payment 20260424.pdf 	new file:   archive/Purchase 20260424.docx 	new file:   archive/REM_OUTPUT.xlsx 	modified:   firmware/ESP32-S3 PWM/include/config.h 	modified:   firmware/ESP32-S3 PWM/src/hardware_control.cpp 	deleted:    hardware/CTL-5.0/CTL-5.0-backups/CTL-5.0-2026-02-20_154251.zip 	deleted:    hardware/CTL-5.0/CTL-5.0-backups/CTL-5.0-2026-02-20_184343.zip 	deleted:    hardware/CTL-5.0/CTL-5.0-backups/CTL-5.0-2026-02-26_100701.zip 	deleted:    hardware/CTL-5.0/CTL-5.0-backups/CTL-5.0-2026-02-26_102054.zip 	deleted:    hardware/CTL-5.0/CTL-5.0-backups/CTL-5.0-2026-02-26_102605.zip 	deleted:    hardware/CTL-5.0/CTL-5.0-backups/CTL-5.0-2026-02-26_103340.zip 	deleted:    hardware/CTL-5.0/CTL-5.0-backups/CTL-5.0-2026-02-26_153650.zip 	new file:   hardware/CTL-5.0/CTL-5.0-backups/CTL-5.0-2026-04-30_153803.zip 	new file:   hardware/CTL-5.0/CTL-5.0-backups/CTL-5.0-2026-04-30_154828.zip 	new file:   hardware/CTL-5.0/CTL-5.0-backups/CTL-5.0-2026-04-30_160225.zip 	new file:   hardware/CTL-5.0/CTL-5.0-backups/CTL-5.0-2026-04-30_161241.zip 	new file:   hardware/CTL-5.0/CTL-5.0-backups/CTL-5.0-2026-04-30_162225.zip 	new file:   hardware/CTL-5.0/CTL-5.0-backups/CTL-5.0-2026-04-30_162925.zip 	modified:   hardware/CTL-5.0/CTL-5.0.kicad_pcb 	modified:   hardware/CTL-5.0/CTL-5.0.kicad_sch 	modified:   hardware/CTL-5.0/fp-info-cache 	deleted:    hardware/INA-3.1/INA-3.1-backups/INA-3.1-2026-04-21_104126.zip 	new file:   hardware/INA-3.1/INA-3.1-backups/INA-3.1-2026-04-29_085310.zip 	new file:   hardware/INA-3.1/INA-3.1-backups/INA-3.1-2026-04-30_110843.zip 	new file:   hardware/INA-3.1/INA-3.1-backups/INA-3.1-2026-04-30_111401.zip 	new file:   hardware/INA-3.1/INA-3.1-backups/INA-3.1-2026-04-30_111913.zip 	new file:   hardware/INA-3.1/INA-3.1-backups/INA-3.1-2026-04-30_112649.zip 	new file:   hardware/INA-3.1/INA-3.1-backups/INA-3.1-2026-04-30_113258.zip 	modified:   hardware/INA-3.1/INA-3.1.kicad_pcb 	modified:   hardware/INA-3.1/INA-3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
Parts:
- added C8: 100nF, Capacitor_SMD:C_0805_2012Metric_Pad1.18x1.45mm_HandSolder, F.Cu at (118.1, 57.5)
- added R9: 10kΩ, Resistor_SMD:R_0805_2012Metric_Pad1.20x1.40mm_HandSolder, F.Cu at (115.4, 54.8)
- C7: value 470pF -> 100nF
- R1: value 6.8kΩ -> 5.1kΩ
Connections:
- R6 pad 2: /OUT -> Net-(R6-Pad2)
- U3 pad 1: /OUT -> Net-(R6-Pad2)
Routing:
- added copper zone on F.Cu, net Net-(R6-Pad2)

Commit message: modified:   firmware/ESU_V1/include/data_manager.h 	modified:   firmware/ESU_V1/include/hardware_control.h 	modified:   firmware/ESU_V1/src/hardware_control.cpp 	modified:   firmware/ESU_V1/src/main.cpp 	modified:   hardware/CTL-6.1/CTL-6.1.kicad_pcb 	modified:   hardware/CTL-6.1/CTL-6.1.kicad_prl 	modified:   hardware/CTL-6.1/CTL-6.1.kicad_pro 	modified:   hardware/INA-3/INA-3.kicad_pcb 	modified:   hardware/INA-3/INA-3.kicad_prl 	modified:   hardware/INA-3/INA-3.kicad_pro 	modified:   hardware/INA-3/INA-3.kicad_sch 	renamed:    hardware/INA-3/fabrication-outputs/INA-3-TRACE.dxf -> hardware/INA-3/fabrication-outputs/EDGE.dxf 	deleted:    hardware/INA-3/fabrication-outputs/INA-3-Edge_Cuts.dxf 	modified:   hardware/INA-3/fabrication-outputs/INA-3-F_Cu.dxf 	new file:   hardware/INA-3/fabrication-outputs/INA-3-F_Cu.pdf 	deleted:    hardware/INA-3/fabrication-outputs/INA-3-NPTH-drl_map.dxf 	deleted:    hardware/INA-3/fabrication-outputs/INA-3-PTH-drl_map.dxf 	new file:   hardware/INA-3/fabrication-outputs/TRACE.dxf 	deleted:    hardware/INA-3/fp-info-cache 	new file:   hardware/REM-5.0/.history 	modified:   hardware/REM-5.0/REM-5.0.kicad_pcb 	modified:   hardware/REM-5.0/REM-5.0.kicad_prl 	modified:   hardware/REM-5.0/REM-5.0.kicad_pro
Parts:
- added C9: 100nF, Capacitor_SMD:C_0805_2012Metric_Pad1.18x1.45mm_HandSolder, F.Cu at (122.9, 57.3)
- added R10: 10kΩ, Resistor_SMD:R_0805_2012Metric_Pad1.20x1.40mm_HandSolder, F.Cu at (119.1, 55.4)
- added R11: 10kΩ, Resistor_SMD:R_0805_2012Metric_Pad1.20x1.40mm_HandSolder, F.Cu at (122.9, 55.4)
- moved C8 4.70 mm to (119.1, 52.9)
- moved R9 1.91 mm to (115.3, 52.9), turned to 0 degrees
- moved C1 0.16 mm to (102.6, 57.9)
- moved R3 0.16 mm to (102.6, 63.7)
- moved R5 0.16 mm to (102.6, 55.4)
- moved R7 0.16 mm to (102.6, 52.9)
- moved U2 0.16 mm to (102.6, 60.8)
- moved C2 0.16 mm to (111.4, 63.7)
- moved C3 0.16 mm to (107.0, 57.9)
- moved C4 0.16 mm to (98.1, 72.5)
- moved C5 0.16 mm to (98.1, 69.4)
- moved C6 0.16 mm to (98.1, 66.7)
- moved C7 0.16 mm to (98.1, 61.8)
- moved R1 0.16 mm to (107.0, 60.8)
- moved R2 0.16 mm to (111.4, 57.9)
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Connections:
- C8 pad 1: /OUT -> Net-(C8-Pad1)
- R9 pad 2: /OUT -> Net-(C8-Pad1)
Routing:
- net Net-(C8-Pad1): track 0.00 -> 3.81 mm
- net +5V: track 8.41 -> 11.3 mm

Commit message: new file:   hardware/INA-3/.history 	modified:   hardware/INA-3/INA-3.kicad_pcb 	modified:   hardware/INA-3/INA-3.kicad_prl 	modified:   hardware/INA-3/INA-3.kicad_pro 	modified:   hardware/INA-3/fabrication-outputs/EDGE.dxf 	modified:   hardware/INA-3/fabrication-outputs/TRACE.dxf 	new file:   hardware/INA-3/~INA-3.kicad_pcb.lck 	new file:   hardware/INA-3/~INA-3.kicad_pro.lck
Routing:
- net Net-(C8-Pad1): track 3.81 -> 0.00 mm
- added copper zone on F.Cu, net Net-(C8-Pad1)
Changed lines of the file:
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@@
 		(layer "Edge.Cuts")
-	)
-	(segment
-		(start 117.95125 52.86375)
-		(end 117.95125 55.40375)
-		(width 0.9525)
-		(layer "F.Cu")
-		(net "Net-(C8-Pad1)")
-	)
-	(segment
-		(start 116.5225 52.86375)
-		(end 117.7925 52.86375)
-		(width 1.27)
-		(layer "F.Cu")
-		(net "Net-(C8-Pad1)")
 	)
 	(via
@@
 			)
 		)
+	)
+	(zone
+		(net "Net-(C8-Pad1)")
+		(layer "F.Cu")
+		(hatch none 0.5)
+		(priority 1)
+		(connect_pads yes
+			(clearance 0)
+		)
+		(min_thickness 0.03175)
+		(fill yes
+			(thermal_gap 0.5)
+			(thermal_bridge_width 0.5)
+			(island_removal_mode 0)
+		)
+		(polygon
+			(pts
+				(xy 115.8875 52.22875) (xy 118.4275 52.22875) (xy 118.4275 56.03875) (xy 117.475 56.03875) (xy 117.475 53.49875)
+				(xy 115.8875 53.49875)
+			)
+		)
