File: hardware/CTL-6.1/CTL-6.1.kicad_sch (KiCad schematic)
At the start: 80 parts, among them J1 Conn_02x16_Top_Bottom, J3 Conn_01x03, J4 Conn_01x03, J5 Conn_02x06_Odd_Even, J6 Conn_01x04, J7 Conn_01x04, J8 Conn_01x04, K1 G5V-1, Q1 BCX56, Q2 BCX56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

Commit message: new file:   hardware/CTL-6.0/CTL-6.0-backups/CTL-6.0-2026-06-11_110233.zip 	modified:   hardware/CTL-6.0/CTL-6.0.kicad_prl 	modified:   hardware/CTL-6.0/CTL-6.0.kicad_pro 	deleted:    hardware/CTL-6.1/CTL-6.1-backups/CTL-6.1-2026-05-21_160708.zip 	deleted:    hardware/CTL-6.1/CTL-6.1-backups/CTL-6.1-2026-05-21_163235.zip 	deleted:    hardware/CTL-6.1/CTL-6.1-backups/CTL-6.1-2026-05-22_160447.zip 	deleted:    hardware/CTL-6.1/CTL-6.1-backups/CTL-6.1-2026-05-22_160956.zip 	deleted:    hardware/CTL-6.1/CTL-6.1-backups/CTL-6.1-2026-05-22_162109.zip 	deleted:    hardware/CTL-6.1/CTL-6.1-backups/CTL-6.1-2026-05-22_163223.zip 	deleted:    hardware/CTL-6.1/CTL-6.1-backups/CTL-6.1-2026-05-22_210324.zip 	deleted:    hardware/CTL-6.1/CTL-6.1-backups/CTL-6.1-2026-05-25_112244.zip 	new file:   hardware/CTL-6.1/CTL-6.1-backups/CTL-6.1-2026-06-11_110530.zip 	new file:   hardware/CTL-6.1/CTL-6.1-backups/CTL-6.1-2026-06-11_110702.zip 	new file:   hardware/CTL-6.1/CTL-6.1-backups/CTL-6.1-2026-06-11_111015.zip 	new file:   hardware/CTL-6.1/CTL-6.1-backups/CTL-6.1-2026-06-11_111525.zip 	new file:   hardware/CTL-6.1/CTL-6.1-backups/CTL-6.1-2026-06-11_112032.zip 	new file:   hardware/CTL-6.1/CTL-6.1-backups/CTL-6.1-2026-06-11_112817.zip 	new file:   hardware/CTL-6.1/CTL-6.1-backups/CTL-6.1-2026-06-11_113247.zip 	new file:   hardware/CTL-6.1/CTL-6.1-backups/CTL-6.1-2026-06-11_115705.zip 	new file:   hardware/CTL-6.1/CTL-6.1-backups/CTL-6.1-2026-06-11_115856.zip 	modified:   hardware/CTL-6.1/CTL-6.1.kicad_pcb 	modified:   hardware/CTL-6.1/CTL-6.1.kicad_prl 	modified:   hardware/CTL-6.1/CTL-6.1.kicad_pro 	modified:   hardware/CTL-6.1/CTL-6.1.kicad_sch 	new file:   hardware/CTL-6.1/~CTL-6.1.kicad_pcb.lck 	new file:   hardware/CTL-6.1/~CTL-6.1.kicad_pro.lck 	new file:   hardware/CTL-6.1/~CTL-6.1.kicad_sch.lck
Parts:
- added R30: 3.3kΩ, Resistor_SMD:R_0805_2012Metric_Pad1.20x1.40mm_HandSolder, symbol Device:R
- J2, U4: value ~ -> (none)
- R29: value 10kΩ -> 1.8kΩ
Connections:
- net GND: now also R30.2
- net REM: now also R30.1
Other:
- note added: "INA equivalent: OPA365 OPA364 OPA320 OPA376"
