File: hardware/REM-7.0/REM-7.0.kicad_sch (KiCad schematic)
At the start: 22 parts, among them J1 Conn_01x04, J2 Conn_01x05, Q1 MMBT3904, T1 Transformer_1P_1S

Commit message: modified:   hardware/REM-7.0/REM-7.0.kicad_sch
Parts:
- RV1: value R_Potentiometer -> 20k
Changed lines of the file:
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@@
-	(wire
-		(pts
-			(xy 114.3 58.42) (xy 114.3 63.5)
-		)
-		(stroke
-			(width 0)
-			(type default)
-		)
-	)
 	(wire
 		(pts
@@
 			)
 		)
-		(property "Value" "R_Potentiometer"
+		(property "Value" "20k"
 			(at 73.66 58.42 0)
 			(show_name no)
