File: hardware/REM-7.0/REM-7.0.kicad_pcb (KiCad board)
At the start: 2 copper layers, 98.4 x 31.8 mm, 21 parts, among them J1 Conn_01x04, J2 Conn_01x05, Q1 MMBT3904

Commit message: modified:   CHANGELOG.md 	modified:   archive/REM - Vsense.xlsx 	modified:   archive/REM_OUTPUT.xlsx 	modified:   hardware/REM-7.0/REM-7.0.kicad_pcb 	modified:   hardware/REM-7.0/REM-7.0.kicad_prl 	modified:   hardware/REM-7.0/REM-7.0.kicad_pro 	modified:   hardware/REM-7.0/REM-7.0.kicad_sch 	modified:   hardware/REM-7.0/REM-7.op.raw 	modified:   hardware/REM-7.0/REM-7.raw 	new file:   hardware/REM-7.0/pabrication output/REM-7.0-B_Cu.dxf 	modified:   hardware/REM-7.0/pabrication output/REM-7.0-B_Cu.pdf 	new file:   hardware/REM-7.0/pabrication output/REM-7.0-Edge_Cuts.dxf 	modified:   hardware/REM-7.0/pabrication output/REM-7.0-Edge_Cuts.pdf 	new file:   hardware/REM-7.0/pabrication output/REM-7.0-F_Cu.dxf 	modified:   hardware/REM-7.0/pabrication output/REM-7.0-F_Cu.pdf 	modified:   hardware/REM-7.0/pabrication output/TRACE_BOT.dxf 	new file:   hardware/REM-7.0/pabrication output/TRACE_TOP.dxf.dwg
Parts:
- added RV_ALT1: R, Resistor_SMD:R_0805_2012Metric_Pad1.20x1.40mm_HandSolder, F.Cu at (87.0, 126.0)
- added T1: Transformer_1P_1S, Transformer_THT:Transformer_EP13_1423, F.Cu at (126.2, 130.3)
- R3: value R -> 4.7k
- RV1: value R_Potentiometer -> 20k
Connections:
- R6 pad 1: unconnected-(R6-Pad1) -> Net-(T1-SB)
- R7 pad 1: unconnected-(R7-Pad1) -> Net-(T1-SA)
Routing:
- net Net-(T1-SB): track 0.00 -> 22.5 mm
- net Net-(Q1-C): track 16.0 -> 38.1 mm, vias 2 -> 1
- net Net-(T1-SA): track 0.00 -> 21.3 mm
- net +5V: track 16.0 -> 28.3 mm, vias 3 -> 2
- net unconnected-(R7-Pad1): track 4.29 -> 0.00 mm, vias 1 -> 0
- net unconnected-(R6-Pad1): track 4.29 -> 0.00 mm, vias 1 -> 0
- net (no net): vias 1 -> 0

Commit message: new file:   archive/Peripheral Migration ESP32S3-STM32H7.md 	new file:   archive/datasheets/STM32H750VBT6_STM32H7XX_M-2.jpg 	new file:   archive/datasheets/original-schematic-STM32H7XX-M.pdf 	new file:   archive/datasheets/stm32h750ib.pdf 	new file:   hardware/CTL-7.0/CTL-7.0.kicad_pcb 	new file:   hardware/CTL-7.0/CTL-7.0.kicad_prl 	new file:   hardware/CTL-7.0/CTL-7.0.kicad_pro 	new file:   hardware/CTL-7.0/CTL-7.0.kicad_sch 	modified:   hardware/REM-7.0/REM-7.0.kicad_pcb 	modified:   hardware/REM-7.0/REM-7.0.kicad_prl 	modified:   hardware/REM-7.0/REM-7.0.kicad_pro 	modified:   hardware/REM-7.0/REM-7.0.kicad_sch
Parts:
- removed J1: Conn_01x04, Connector_PinHeader_2.54mm:PinHeader_1x04_P2.54mm_Horizontal
- removed J2: Conn_01x05, Connector_PinHeader_2.54mm:PinHeader_1x05_P2.54mm_Horizontal
- moved RV_ALT1 10.2 mm to (77.8, 130.5)
- moved R3 2.98 mm to (80.6, 127.8), turned to 0 degrees
- moved C2 2.22 mm to (79.7, 130.5)
- moved RV1 0.64 mm to (83.2, 125.4)
- moved C23 0.35 mm to (81.6, 135.1)
- moved C4 0.32 mm to (94.9, 134.9)
- moved C5 0.32 mm to (94.9, 130.5)
- moved Q1 0.32 mm to (92.1, 130.5)
- moved R2 0.32 mm to (93.0, 134.9)
- moved C1 0.32 mm to (87.3, 134.9)
- moved C3 0.32 mm to (81.6, 130.5)
- moved C6 0.32 mm to (89.2, 130.5), turned to -90 degrees
- moved C7 0.32 mm to (91.1, 134.9)
- moved D1 0.32 mm to (84.5, 130.5)
- moved R4 0.32 mm to (89.2, 134.9)
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Connections:
- C6 pad 1: Net-(D1-COM) -> Net-(Q1-C)
- C6 pad 2: Net-(Q1-C) -> Net-(D1-COM)
- RV1 pad 1: /REM -> GND
- RV1 pad 2: /REM -> GND
- RV1 pad 3: GND -> /REM
Routing:
- net /REM: track 20.1 -> 16.8 mm, vias 1 -> 2
- net +5V: track 28.3 -> 28.1 mm, vias 2 -> 3
- net GND: vias 2 -> 17
- net Net-(J2-Pin_5): vias 1 -> 2
- net Net-(J2-Pin_3): vias 1 -> 2
- net Net-(J2-Pin_1): vias 1 -> 2
